File: Kicad/A1K Adaptor Board/A1K Adaptor Board.kicad_sch (KiCad schematic)
At the start: 0 parts

Commit message: e
e
Changed lines of the file:
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@@
 	(paper "A4")
 	(sheet
-		(at 24.13 59.69)
-		(size 22.86 80.01)
+		(at 66.04 60.96)
+		(size 16.51 48.26)
 		(exclude_from_sim no)
 		(in_bom yes)
@@
 		)
 		(property "Sheetname" "Toolhead_Board"
-			(at 24.13 58.9784 0)
+			(at 66.04 60.2484 0)
 			(effects
 				(font
@@
 		)
 		(property "Sheetfile" "Toolhead_Board.kicad_sch"
-			(at 24.13 140.2846 0)
+			(at 66.04 109.8046 0)
 			(effects
 				(font
@@
 		)
 		(instances
-			(project "A1K Board"
-				(path "/2c6f0d05-350a-4e4e-887e-c97bc5a9b57b"
-					(page "12")
+			(project "A1K Adaptor Board"
+				(path "/763e8f8f-9e52-4f06-9d68-06c79d355bec"
+					(page "2")
 				)
 			)
