File: Kicad/A1K_CM/rpi-cm4-base-carrier/rpi-cm4-base-carrier.kicad_pcb (KiCad board)
At the start: 2 copper layers, 115 x 64.5 mm, 14 parts, among them J1 X_MOTOR_JST, J2 RJ45, J3 USB3_A, J4 USB_A_Stacked, J5 Y_MOTOR_JST, J6 Z_MOTOR_JST, J7 S_MOTOR_JST, J8 Micro_SD_Card, J9 HDMI_A_1.4, U3 X_TMC2209, U4 X_TMC2209, U5 X_TMC2209, U6 X_TMC2209

Commit message: e
e
Parts:
- removed U3, U4, U5, U6: X_TMC2209, TMC2209:MODULE_TMC2209_SILENTSTEPSTICK
- added J10: Bus_PCI_Express_x1, Connector_PCBEdge:BUS_PCIexpress_x1, F.Cu at (176.5, 91.0)
- added J11: Conn_02x03_Odd_Even, Connector_PinHeader_2.54mm:PinHeader_2x03_P2.54mm_Vertical, F.Cu at (118.7, 119.0)
- added J13: Conn_02x03_Odd_Even, Connector_PinSocket_2.54mm:PinSocket_2x03_P2.54mm_Vertical, F.Cu at (137.5, 119.0)
- added J15: Conn_02x03_Odd_Even, Connector_PinSocket_2.54mm:PinSocket_2x03_P2.54mm_Vertical, F.Cu at (151.0, 118.9)
- added J17: Conn_02x03_Odd_Even, Connector_PinSocket_2.54mm:PinSocket_2x03_P2.54mm_Vertical, F.Cu at (167.5, 118.9)
- added M2: TMC2209 Breakout, TMC2209:MODULE_TMC2209_SILENTSTEPSTICK, F.Cu at (118.0, 117.6)
- added M3: TMC2209 Breakout, TMC2209:MODULE_TMC2209_SILENTSTEPSTICK, F.Cu at (134.0, 117.7)
- added M4: TMC2209 Breakout, TMC2209:MODULE_TMC2209_SILENTSTEPSTICK, F.Cu at (150.0, 117.7)
- added M5: TMC2209 Breakout, TMC2209:MODULE_TMC2209_SILENTSTEPSTICK, F.Cu at (166.3, 117.7)
- added R3: 10kΩ, Resistor_THT:R_Axial_DIN0207_L6.3mm_D2.5mm_P10.16mm_Horizontal, F.Cu at (112.9, 105.0)
- added R4: 10kΩ, Resistor_THT:R_Axial_DIN0207_L6.3mm_D2.5mm_P10.16mm_Horizontal, F.Cu at (128.9, 105.0)
- added R5: 10kΩ, Resistor_THT:R_Axial_DIN0207_L6.3mm_D2.5mm_P10.16mm_Horizontal, F.Cu at (144.9, 105.0)
- added R6: 10kΩ, Resistor_THT:R_Axial_DIN0207_L6.3mm_D2.5mm_P10.16mm_Horizontal, F.Cu at (161.4, 105.2)
- moved J8 93.3 mm to (73.5, 65.5)
- moved J9 12.6 mm to (110.0, 63.8)
- moved J2 12.6 mm to (123.8, 60.0)
- moved J4 12.6 mm to (168.4, 69.6)
- moved J3 12.6 mm to (143.8, 61.7)
Other:
- board size 115 x 64.5 mm -> 115 x 79 mm
