File: Kicad/A1K_CM/rpi-cm4-base-carrier/tmc_modules.kicad_sch (KiCad schematic)
At the start: 24 parts, among them J11 Conn_02x03_Odd_Even, J12 Conn_01x04, J13 Conn_02x03_Odd_Even, J14 Conn_01x04, J15 Conn_02x03_Odd_Even, J16 Conn_01x04, J17 Conn_02x03_Odd_Even, J18 Conn_01x04, M2 TMC2209 Breakout, M3 TMC2209 Breakout, M4 TMC2209 Breakout, M5 TMC2209 Breakout

Commit message: e
e
Parts:
- J13, J15, J17: footprint Connector_PinHeader_2.54mm:PinHeader_2x03_P2.54mm_Vertical -> Connector_PinSocket_2.54mm:PinSocket_2x03_P2.54mm_Vertical
- M2, M3, M4, M5: footprint CustomFootprints:TMC2209 Footprint -> TMC2209:MODULE_TMC2209_SILENTSTEPSTICK
Changed lines of the file:
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@@
 			)
 		)
-		(property "Footprint" "CustomFootprints:TMC2209 Footprint"
+		(property "Footprint" "TMC2209:MODULE_TMC2209_SILENTSTEPSTICK"
 			(at 182.245 140.97 0)
 			(effects
@@
 			)
 		)
-		(property "Footprint" "CustomFootprints:TMC2209 Footprint"
+		(property "Footprint" "TMC2209:MODULE_TMC2209_SILENTSTEPSTICK"
 			(at 182.245 176.53 0)
 			(effects
@@
 			)
 		)
-		(property "Footprint" "CustomFootprints:TMC2209 Footprint"
+		(property "Footprint" "TMC2209:MODULE_TMC2209_SILENTSTEPSTICK"
 			(at 182.245 74.93 0)
 			(effects
@@
 			)
 		)
-		(property "Footprint" "Connector_PinHeader_2.54mm:PinHeader_2x03_P2.54mm_Vertical"
+		(property "Footprint" "Connector_PinSocket_2.54mm:PinSocket_2x03_P2.54mm_Vertical"
 			(at 123.19 143.51 0)
 			(effects
@@
 			)
 		)
-		(property "Footprint" "CustomFootprints:TMC2209 Footprint"
+		(property "Footprint" "TMC2209:MODULE_TMC2209_SILENTSTEPSTICK"
 			(at 182.245 107.95 0)
 			(effects
@@
 			)
 		)
-		(property "Footprint" "Connector_PinHeader_2.54mm:PinHeader_2x03_P2.54mm_Vertical"
+		(property "Footprint" "Connector_PinSocket_2.54mm:PinSocket_2x03_P2.54mm_Vertical"
 			(at 123.19 107.95 0)
 			(effects
@@
 			)
 		)
-		(property "Footprint" "Connector_PinHeader_2.54mm:PinHeader_2x03_P2.54mm_Vertical"
+		(property "Footprint" "Connector_PinSocket_2.54mm:PinSocket_2x03_P2.54mm_Vertical"
 			(at 123.19 74.93 0)
 			(effects
