File: A1_AMS/A1_AMS.kicad_pcb (KiCad board)
At the start: 2 copper layers, 60 x 60 mm, 19 parts, among them J1 Screw_Terminal_01x02, J2 Servo, J3 9-10-11-14-15, J4 Conn_01x04, J5 16-17-18-19-20, J6 21-22-26-27-28, J7 Conn_01x04, J8 5-5-3.3-G-G, M1 StepperMotor, M2 StepperMotor, U1 Pico

Commit message: e
e
Routing:
- net GND: track 303.8 -> 0.00 mm, vias 1 -> 0
- net /5V: track 2.54 -> 50.2 mm, vias 0 -> 1
- net /G19: track 29.2 -> 0.00 mm, vias 1 -> 0
- net /M_UART: track 93.2 -> 67.7 mm, vias 1 -> 0
- net /G15: track 19.5 -> 0.00 mm
- net /SV_SIG: track 51.7 -> 60.5 mm, vias 3 -> 1
- net /MS_STEP: track 32.1 -> 26.1 mm
- net /MS_EN: track 28.3 -> 33.8 mm, vias 0 -> 1
- net /MS_DIR: track 33.5 -> 30.1 mm
- net /G14: track 12.4 -> 9.65 mm
- net /G16: track 33.1 -> 30.5 mm, vias 1 -> 0
- net /MD_EN: track 59.9 -> 57.7 mm
- net /G10: track 16.1 -> 14.7 mm
- net /G17: track 30.8 -> 29.6 mm, vias 1 -> 0
- net /G21: track 25.8 -> 25.1 mm, vias 1 -> 0
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- added copper zone on B.Cu, net GND
- added copper zone on F.Cu, net GND

Commit message: l
Parts:
- added C1: 100uF 63V, OpenA1K:Cap63V100UF, F.Cu at (140.5, 73.5)
- added C2: 100uF 63V, OpenA1K:Cap63V100UF, F.Cu at (140.5, 47.0)
- added J9: Servo2, Connector_PinHeader_2.54mm:PinHeader_1x03_P2.54mm_Vertical, F.Cu at (123.2, 65.0)
- J2: value Servo -> Servo1; footprint Connector_PinSocket_2.54mm:PinSocket_1x03_P2.54mm_Vertical -> Connector_PinHeader_2.54mm:PinHeader_1x03_P2.54mm_Vertical
- J3: value 9-10-11-14-15 -> G-10-11-14-15; footprint Connector_PinSocket_2.54mm:PinSocket_1x05_P2.54mm_Vertical -> Connector_PinHeader_2.54mm:PinHeader_1x05_P2.54mm_Vertical
- J5, J6, J8: footprint Connector_PinSocket_2.54mm:PinSocket_1x05_P2.54mm_Vertical -> Connector_PinHeader_2.54mm:PinHeader_1x05_P2.54mm_Vertical
- moved J2 34.9 mm to (123.5, 74.0), turned to 180 degrees
- moved M2 30.0 mm to (140.3, 66.7), turned to 90 degrees
- moved H5 29.2 mm to (132.5, 77.5)
- moved J6 25.5 mm to (147.5, 39.0), turned to -90 degrees
- moved R3 24.1 mm to (143.0, 63.5), turned to 0 degrees
- moved M1 17.8 mm to (140.5, 93.3), turned to 90 degrees
- moved R2 12.1 mm to (143.0, 90.5), turned to 0 degrees
- moved J4 10.7 mm to (156.5, 76.0), turned to 180 degrees
- moved J8 8.23 mm to (123.5, 45.8)
- moved J5 5.64 mm to (123.5, 39.0), turned to 90 degrees
- moved J3 4.19 mm to (123.5, 41.5), turned to 90 degrees
- moved J7 1.57 mm to (156.5, 49.0), turned to 180 degrees
Connections:
- net /SV_SIG renamed /SV_SIG1
- J3 pad 1: /G9 -> GND
- U1 pad 12: /G9 -> /SV_SIG2
Routing:
- net /SV_SIG1: track 60.5 -> 11.1 mm, vias 1 -> 0
- net /G19: track 0.00 -> 39.4 mm
- net /G28: track 27.2 -> 64.6 mm, vias 0 -> 1
- net /G27: track 26.2 -> 63.0 mm, vias 0 -> 1
- net /G22: track 25.1 -> 57.2 mm, vias 0 -> 1
- net /G26: track 26.2 -> 57.0 mm, vias 0 -> 1
- net /G17: track 29.6 -> 0.00 mm
- net /MD_EN: track 57.7 -> 28.9 mm
- net /G21: track 25.1 -> 51.6 mm
- net /G9: track 23.8 -> 0.00 mm
- net /MD_DIR: track 23.2 -> 43.9 mm, vias 0 -> 2
- net /5V: track 50.2 -> 29.6 mm, vias 1 -> 0
- net /MS_STEP: track 26.1 -> 45.7 mm
- net /M_VBUS: track 85.9 -> 68.3 mm
- net /MS_DIR: track 30.1 -> 47.5 mm
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Other:
- board text added: "5V"
- board text added: "DriverStepper"
- board text added: "GND"
- board text added: "HEAD OF PICO PI"
- board text added: "SIG"
- board text added: "VIN"
- board text added: "m1.5"

Commit message: e
e
Parts:
- removed H3, H6: M1.5, OpenA1K:Mountinghole_m1.5
- removed U1: Pico, OpenA1K:Socketed MCU - Pico (No Text)
- added C3: 470uF, OpenA1K:Cap ~ 12.5, 2.5mm-7.5mm pitch, F.Cu at (235.5, 131.5)
- added C4: 470uF, OpenA1K:Cap ~ 12.5, 2.5mm-7.5mm pitch, F.Cu at (235.0, 68.0)
- added H2: M1.5, OpenA1K:Mountinghole_m1.5, F.Cu at (266.2, 91.1)
- added H4: M1.5, OpenA1K:Mountinghole_m1.5, F.Cu at (169.0, 193.0)
- added J10: Screw_Terminal_01x02, OpenA1K:1x2 Terminal Block, F.Cu at (193.4, 115.5)
- added J11: M1, Connector_JST:JST_XH_B2B-XH-AM_1x02_P2.50mm_Vertical, F.Cu at (117.9, 76.5)
- added J12: M2, Connector_JST:JST_XH_B2B-XH-AM_1x02_P2.50mm_Vertical, F.Cu at (117.9, 69.5)
- added J13: Conn_01x04, Connector_JST:JST_XH_B4B-XH-A_1x04_P2.50mm_Vertical, F.Cu at (114.1, 131.0)
- added J14: M4, Connector_JST:JST_XH_B2B-XH-AM_1x02_P2.50mm_Vertical, F.Cu at (118.0, 55.5)
- added J15: M3, Connector_JST:JST_XH_B2B-XH-AM_1x02_P2.50mm_Vertical, F.Cu at (117.9, 62.5)
- added J16: Conn_01x04, Connector_JST:JST_XH_B4B-XH-A_1x04_P2.50mm_Vertical, F.Cu at (140.5, 131.0)
- added J17: LED2, Connector_JST:JST_XH_B3B-XH-A_1x03_P2.50mm_Vertical, F.Cu at (178.5, 69.5)
- added J18: LED3, Connector_JST:JST_XH_B3B-XH-A_1x03_P2.50mm_Vertical, F.Cu at (178.5, 62.5)
- added J19: Conn_01x04, Connector_JST:JST_XH_B4B-XH-A_1x04_P2.50mm_Vertical, F.Cu at (167.3, 130.5)
- added J20: LED4, Connector_JST:JST_XH_B3B-XH-A_1x03_P2.50mm_Vertical, F.Cu at (178.5, 55.5)
- added J21: SW1, Connector_JST:JST_XH_B2B-XH-AM_1x02_P2.50mm_Vertical, F.Cu at (164.3, 76.6)
- added J22: Conn_01x04, Connector_JST:JST_XH_B4B-XH-A_1x04_P2.50mm_Vertical, F.Cu at (193.5, 130.5)
- added J23: SW2, Connector_JST:JST_XH_B2B-XH-AM_1x02_P2.50mm_Vertical, F.Cu at (164.3, 69.4)
- added J24: SW3, Connector_JST:JST_XH_B2B-XH-AM_1x02_P2.50mm_Vertical, F.Cu at (164.3, 62.6)
- added J25: MSHUB1, Connector_JST:JST_XH_B2B-XH-AM_1x02_P2.50mm_Vertical, F.Cu at (109.5, 62.5)
- added J26: MSHUB2, Connector_JST:JST_XH_B2B-XH-AM_1x02_P2.50mm_Vertical, F.Cu at (109.5, 69.5)
- added J27: MSBYPASS, Connector_JST:JST_XH_B2B-XH-AM_1x02_P2.50mm_Vertical, F.Cu at (109.5, 76.5)
- added J29: T1, Connector_JST:JST_XH_B2B-XH-AM_1x02_P2.50mm_Vertical, F.Cu at (187.0, 76.5)
- added J30: T2, Connector_JST:JST_XH_B2B-XH-AM_1x02_P2.50mm_Vertical, F.Cu at (187.0, 69.5)
- added J31: T3, Connector_JST:JST_XH_B2B-XH-AM_1x02_P2.50mm_Vertical, F.Cu at (187.0, 62.5)
- added JS4: SW4, Connector_JST:JST_XH_B2B-XH-AM_1x02_P2.50mm_Vertical, F.Cu at (164.5, 55.6)
- added JS5: T4, Connector_JST:JST_XH_B2B-XH-AM_1x02_P2.50mm_Vertical, F.Cu at (187.0, 55.5)
- added JS6: HT1, Connector_JST:JST_XH_B2B-XH-AM_1x02_P2.50mm_Vertical, F.Cu at (154.5, 76.5)
- added JS7: HT2, Connector_JST:JST_XH_B2B-XH-AM_1x02_P2.50mm_Vertical, F.Cu at (154.6, 69.5)
- added M3: TMC2209 Breakout, OpenA1K:TMC2209 Footprint, F.Cu at (154.8, 148.2)
- added M4: TMC2209 Breakout, OpenA1K:TMC2209 Footprint, F.Cu at (180.6, 148.1)
- added R4: 10kΩ, Resistor_THT:R_Axial_DIN0207_L6.3mm_D2.5mm_P10.16mm_Horizontal, F.Cu at (239.5, 99.0)
- added R5: 10kΩ, Resistor_THT:R_Axial_DIN0207_L6.3mm_D2.5mm_P10.16mm_Horizontal, F.Cu at (240.0, 78.1)
- added U2: ~, OpenA1K:Socketed MCU STM32 64P, F.Cu at (168.4, 117.0)
- C1, C2: value 100uF 63V -> 470uF; footprint OpenA1K:Cap63V100UF -> OpenA1K:Cap ~ 12.5, 2.5mm-7.5mm pitch
- F1: value M_ATO_FUSE -> Mini ATO Fuse
- J1: value Screw_Terminal_01x02 -> 1A; footprint OpenA1K:1x2 Terminal Block -> Connector_JST:JST_XH_B2B-XH-AM_1x02_P2.50mm_Vertical
- J2: value Servo1 -> 2A; footprint Connector_PinHeader_2.54mm:PinHeader_1x03_P2.54mm_Vertical -> Connector_JST:JST_XH_B2B-XH-AM_1x02_P2.50mm_Vertical
- J3: value G-10-11-14-15 -> 3A; footprint Connector_PinHeader_2.54mm:PinHeader_1x05_P2.54mm_Vertical -> Connector_JST:JST_XH_B2B-XH-AM_1x02_P2.50mm_Vertical
- J4: value Conn_01x04 -> 4A; footprint Connector_JST:JST_XH_B4B-XH-A_1x04_P2.50mm_Vertical -> Connector_JST:JST_XH_B2B-XH-AM_1x02_P2.50mm_Vertical
- J5: value 16-17-18-19-20 -> LED1; footprint Connector_PinHeader_2.54mm:PinHeader_1x05_P2.54mm_Vertical -> Connector_JST:JST_XH_B3B-XH-A_1x03_P2.50mm_Vertical
- J6: value 21-22-26-27-28 -> 1B; footprint Connector_PinHeader_2.54mm:PinHeader_1x05_P2.54mm_Vertical -> Connector_JST:JST_XH_B2B-XH-AM_1x02_P2.50mm_Vertical
- J7: value Conn_01x04 -> 2B; footprint Connector_JST:JST_XH_B4B-XH-A_1x04_P2.50mm_Vertical -> Connector_JST:JST_XH_B2B-XH-AM_1x02_P2.50mm_Vertical
- J8: value 5-5-3.3-G-G -> 3B; footprint Connector_PinHeader_2.54mm:PinHeader_1x05_P2.54mm_Vertical -> Connector_JST:JST_XH_B2B-XH-AM_1x02_P2.50mm_Vertical
- J9: value Servo2 -> 4B; footprint Connector_PinHeader_2.54mm:PinHeader_1x03_P2.54mm_Vertical -> Connector_JST:JST_XH_B2B-XH-AM_1x02_P2.50mm_Vertical
- M1, M2: value StepperMotor -> TMC2209 Breakout
- moved C2 116.2 mm to (236.5, 112.5)
- moved R3 111.9 mm to (239.5, 120.1), turned to 90 degrees
- moved R1 110.4 mm to (204.5, 105.5), turned to 90 degrees
- moved R2 109.0 mm to (239.5, 141.1), turned to 90 degrees
- moved C1 94.9 mm to (234.0, 90.0)
- moved M2 82.3 mm to (128.1, 148.1)
- moved H5 69.6 mm to (197.5, 52.5)
- moved F1 68.5 mm to (179.5, 120.5)
- moved M1 67.1 mm to (101.6, 148.1)
- moved J5 66.6 mm to (178.5, 76.5), turned to 180 degrees
- moved H1 57.0 mm to (102.5, 52.5)
- moved J6 40.8 mm to (131.5, 76.5), turned to 180 degrees
- moved J7 32.3 mm to (131.5, 69.5)
- moved J3 26.7 mm to (140.0, 62.5), turned to 180 degrees
- moved J4 26.3 mm to (140.0, 55.5)
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Connections:
- net /MD_EN renamed /MB_EN
- net /MS_EN renamed /MA_EN
- F1 pad 2: Net-(J1-Pin_2) -> /VIN
- J1 pad 1: GND -> /MS_1A
- J1 pad 2: Net-(J1-Pin_2) -> GND
- J2 pad 1: GND -> /MS_2A
- J2 pad 2: /5V -> GND
- J3 pad 1: GND -> /MS_3A
- J3 pad 2: /G10 -> GND
- J4 pad 1: /SelectorMotor/B2 -> /MS_4A
- J4 pad 2: /SelectorMotor/B1 -> GND
- J5 pad 1: /G16 -> GND
- J5 pad 2: /G17 -> /LED_1
- J5 pad 3: /G18 -> /5V
- J6 pad 1: /G21 -> /MS_1B
- J6 pad 2: /G22 -> GND
- J7 pad 1: /DriveMotor/B2 -> /MS_2B
- J7 pad 2: /DriveMotor/B1 -> GND
- J8 pad 1: /5V -> /MS_3B
- J8 pad 2: /5V -> GND
- J9 pad 1: GND -> /MS_4B
- J9 pad 2: /5V -> GND
- M1 pad 11: /SelectorMotor/B2 -> /AMotor/B2
- M1 pad 12: /SelectorMotor/B1 -> /AMotor/B1
- M1 pad 13: /SelectorMotor/A1 -> /AMotor/A1
- M1 pad 14: /SelectorMotor/A2 -> /AMotor/A2
- M1 pad 7: /MS_STEP -> /MA_STEP
- M1 pad 8: /MS_DIR -> /MA_DIR
- M2 pad 11: /DriveMotor/B2 -> /BMotor/B2
- M2 pad 12: /DriveMotor/B1 -> /BMotor/B1
- M2 pad 13: /DriveMotor/A1 -> /BMotor/A1
- M2 pad 14: /DriveMotor/A2 -> /BMotor/A2
- M2 pad 2: GND -> /3V3
- M2 pad 3: /3V3 -> GND
- M2 pad 7: /MD_STEP -> /MB_STEP
- M2 pad 8: /MD_DIR -> /MB_DIR
Routing:
- net GND: track 14.2 -> 231.6 mm
- net +3V3: track 111.0 -> 0.00 mm, vias 1 -> 0
- net /M_UART: track 76.0 -> 0.00 mm, vias 1 -> 0
- net /M_VBUS: track 68.3 -> 0.00 mm
- net /G28: track 64.6 -> 0.00 mm, vias 1 -> 0
- net /G27: track 63.0 -> 0.00 mm, vias 1 -> 0
- net /G22: track 57.2 -> 0.00 mm, vias 1 -> 0
- net /MS_HUB2: track 0.00 -> 57.2 mm
- net /G26: track 57.0 -> 0.00 mm, vias 1 -> 0
- net /MS_HUB1: track 0.00 -> 54.1 mm
- net /G21: track 51.6 -> 0.00 mm
- net /MS_DIR: track 47.5 -> 0.00 mm, vias 1 -> 0
- net /MS_4B: track 0.00 -> 47.5 mm, vias 0 -> 1
- net /MS_STEP: track 45.7 -> 0.00 mm, vias 1 -> 0
- net /MS_BYPASS: track 0.00 -> 45.3 mm
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- removed copper zone on B.Cu, net GND
- removed copper zone on F.Cu, net GND
Other:
- board outline removed
- board text removed: "5V"
- board text removed: "DriverStepper"
- board text removed: "GND"
- board text removed: "HEAD OF PICO PI"
- board text removed: "OpenA1K AMS Board By Cyclonekitten"
- board text removed: "SIG"
- board text removed: "SelectorStepper"
- board text removed: "VIN"
- board text removed: "m1.5"
