File: A1_AMS/A1_AMS.kicad_sch (KiCad schematic)
At the start: 13 parts, among them J1 Screw_Terminal_01x02, J2 Servo, J3 9-10-11-14-15, J5 16-17-18-19-20, J6 21-22-26-27-28, J8 5-5-3.3-G-G, U1 Pico

Commit message: l
Parts:
- added J9: Servo2, Connector_PinHeader_2.54mm:PinHeader_1x03_P2.54mm_Vertical, symbol Connector_Generic:Conn_01x03
- J2: value Servo -> Servo1; footprint Connector_PinSocket_2.54mm:PinSocket_1x03_P2.54mm_Vertical -> Connector_PinHeader_2.54mm:PinHeader_1x03_P2.54mm_Vertical
- J3: value 9-10-11-14-15 -> G-10-11-14-15; footprint Connector_PinSocket_2.54mm:PinSocket_1x05_P2.54mm_Vertical -> Connector_PinHeader_2.54mm:PinHeader_1x05_P2.54mm_Vertical
- J5, J6, J8: footprint Connector_PinSocket_2.54mm:PinSocket_1x05_P2.54mm_Vertical -> Connector_PinHeader_2.54mm:PinHeader_1x05_P2.54mm_Vertical
Connections:
- net 5V: now also J9.2 (Pin_2)
- net GND: now also J3.1 (Pin_1), J9.1 (Pin_1)
- net G9 renamed SV_SIG2
- net SV_SIG2: now also J9.3 (Pin_3); no longer J3.1 (Pin_1)
- net SV_SIG renamed SV_SIG1
Changed lines of the file:
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@@
 		)
 	)
-	(hierarchical_label "G9"
+	(hierarchical_label "GND"
 		(shape input)
 		(at 91.44 17.78 0)
@@
 		)
 	)
-	(hierarchical_label "SV_SIG"
+	(hierarchical_label "SV_SIG1"
 		(shape input)
 		(at 22.86 40.64 180)
@@
 		)
 	)
-	(hierarchical_label "SV_SIG"
+	(hierarchical_label "SV_SIG1"
 		(shape input)
 		(at 21.59 146.05 180)
@@
 		)
 	)
+	(hierarchical_label "SV_SIG2"
+		(shape input)
+		(at 21.59 154.94 180)
+		(effects
+			(font
+				(size 1.27 1.27)
+			)
+			(justify right)
+		)
+	)
+	(hierarchical_label "GND"
+		(shape input)
+		(at 21.59 149.86 180)
+		(effects
+			(font
+				(size 1.27 1.27)
+			)
+			(justify right)
+		)
+	)
 	(hierarchical_label "G10"
 		(shape input)
@@
 		)
 	)
+	(hierarchical_label "5V"
+		(shape input)
+		(at 21.59 152.4 180)
+		(effects
+			(font
+				(size 1.27 1.27)
+			)
+			(justify right)
+		)
+	)
 	(hierarchical_label "G27"
 		(shape input)
@@
 		)
 	)
-	(hierarchical_label "G9"
+	(hierarchical_label "SV_SIG2"
 		(shape input)
 		(at 22.86 43.18 180)
@@
 	)
 	(symbol
+		(lib_id "Connector_Generic:Conn_01x03")
+		(at 26.67 152.4 0)
+		(unit 1)
+		(exclude_from_sim no)
+		(in_bom yes)
+		(on_board yes)
+		(dnp no)
+		(fields_autoplaced yes)
+		(property "Reference" "J9"
+			(at 29.21 151.1299 0)
+			(effects
+				(font
+					(size 1.27 1.27)
+				)
+				(justify left)
+			)
+		)
+		(property "Value" "Servo2"
+			(at 29.21 153.6699 0)
+			(effects
+				(font
+					(size 1.27 1.27)
+				)
+				(justify left)
+			)
+		)
+		(property "Footprint" "Connector_PinHeader_2.54mm:PinHeader_1x03_P2.54mm_Vertical"
+			(at 26.67 152.4 0)
+			(effects
+				(font
+					(size 1.27 1.27)
+				)
+				(hide yes)
+			)
+		)
+		(property "Datasheet" "~"
+			(at 26.67 152.4 0)
+			(effects
+				(font
+					(size 1.27 1.27)
+				)
+				(hide yes)
+			)
+		)
+		(property "Description" "Generic connector, single row, 01x03, script generated (kicad-library-utils/schlib/autogen/connector/)"
+			(at 26.67 152.4 0)
+			(effects
+				(font
+					(size 1.27 1.27)
+				)
+				(hide yes)
+			)
+		)
+		(pin "1"
+		)
+		(pin "2"
+		)
+		(pin "3"
+		)
+		(instances
+			(project "A1_AMS"
+				(path "/989d6d42-19bd-451f-8ed3-d8ee079df240"
+					(reference "J9")
+					(unit 1)
+				)
+			)
+		)
+	)
+	(symbol
 		(lib_id "Connector:Conn_01x05_Pin")
 		(at 85.09 44.45 0)
@@
 			)
 		)
-		(property "Footprint" "Connector_PinSocket_2.54mm:PinSocket_1x05_P2.54mm_Vertical"
+		(property "Footprint" "Connector_PinHeader_2.54mm:PinHeader_1x05_P2.54mm_Vertical"
 			(at 85.09 44.45 0)
 			(effects
@@
 			)
 		)
-		(property "Value" "Servo"
+		(property "Value" "Servo1"
 			(at 29.21 144.7799 0)
 			(effects
@@
 			)
 		)
-		(property "Footprint" "Connector_PinSocket_2.54mm:PinSocket_1x03_P2.54mm_Vertical"
+		(property "Footprint" "Connector_PinHeader_2.54mm:PinHeader_1x03_P2.54mm_Vertical"
 			(at 26.67 143.51 0)
 			(effects
@@
 			)
 		)
-		(property "Value" "9-10-11-14-15"
+		(property "Value" "G-10-11-14-15"
 			(at 86.995 15.24 0)
 			(effects
@@
 			)
 		)
-		(property "Footprint" "Connector_PinSocket_2.54mm:PinSocket_1x05_P2.54mm_Vertical"
+		(property "Footprint" "Connector_PinHeader_2.54mm:PinHeader_1x05_P2.54mm_Vertical"
 			(at 86.36 22.86 0)
 			(effects
@@
 			)
 		)
-		(property "Footprint" "Connector_PinSocket_2.54mm:PinSocket_1x05_P2.54mm_Vertical"
+		(property "Footprint" "Connector_PinHeader_2.54mm:PinHeader_1x05_P2.54mm_Vertical"
 			(at 85.09 62.23 0)
 			(effects
@@
 			)
 		)
-		(property "Footprint" "Connector_PinSocket_2.54mm:PinSocket_1x05_P2.54mm_Vertical"
+		(property "Footprint" "Connector_PinHeader_2.54mm:PinHeader_1x05_P2.54mm_Vertical"
 			(at 85.09 80.01 0)
 			(effects

Commit message: e
e
Parts:
- removed H6: M1.5, OpenA1K:Mountinghole_m1.5, symbol Mechanical:MountingHole_Pad
- removed J2: Servo1, Connector_PinHeader_2.54mm:PinHeader_1x03_P2.54mm_Vertical, symbol Connector_Generic:Conn_01x03
- removed J3: G-10-11-14-15, Connector_PinHeader_2.54mm:PinHeader_1x05_P2.54mm_Vertical, symbol Connector:Conn_01x05_Pin
- removed J5: 16-17-18-19-20, Connector_PinHeader_2.54mm:PinHeader_1x05_P2.54mm_Vertical, symbol Connector:Conn_01x05_Pin
- removed J6: 21-22-26-27-28, Connector_PinHeader_2.54mm:PinHeader_1x05_P2.54mm_Vertical, symbol Connector:Conn_01x05_Pin
- removed J8: 5-5-3.3-G-G, Connector_PinHeader_2.54mm:PinHeader_1x05_P2.54mm_Vertical, symbol Connector:Conn_01x05_Pin
- removed J9: Servo2, Connector_PinHeader_2.54mm:PinHeader_1x03_P2.54mm_Vertical, symbol Connector_Generic:Conn_01x03
- removed U1: Pico, OpenA1K:Socketed MCU - Pico (No Text), symbol MCU_RaspberryPi_and_Boards:Pico
- added H2, H4: M1.5, OpenA1K:Mountinghole_m1.5, symbol Mechanical:MountingHole_Pad
- added J1: 1A, Connector_JST:JST_XH_B2B-XH-AM_1x02_P2.50mm_Vertical, symbol Connector:Conn_01x02_Pin
- added J11: M1, Connector_JST:JST_XH_B2B-XH-AM_1x02_P2.50mm_Vertical, symbol Connector:Conn_01x02_Pin
- added J12: M2, Connector_JST:JST_XH_B2B-XH-AM_1x02_P2.50mm_Vertical, symbol Connector:Conn_01x02_Pin
- added J14: M4, Connector_JST:JST_XH_B2B-XH-AM_1x02_P2.50mm_Vertical, symbol Connector:Conn_01x02_Pin
- added J15: M3, Connector_JST:JST_XH_B2B-XH-AM_1x02_P2.50mm_Vertical, symbol Connector:Conn_01x02_Pin
- added J17: LED2, Connector_JST:JST_XH_B3B-XH-A_1x03_P2.50mm_Vertical, symbol Connector:Conn_01x03_Pin
- added J18: LED3, Connector_JST:JST_XH_B3B-XH-A_1x03_P2.50mm_Vertical, symbol Connector:Conn_01x03_Pin
- added J2: 2A, Connector_JST:JST_XH_B2B-XH-AM_1x02_P2.50mm_Vertical, symbol Connector:Conn_01x02_Pin
- added J20: LED4, Connector_JST:JST_XH_B3B-XH-A_1x03_P2.50mm_Vertical, symbol Connector:Conn_01x03_Pin
- added J21: SW1, Connector_JST:JST_XH_B2B-XH-AM_1x02_P2.50mm_Vertical, symbol Connector:Conn_01x02_Pin
- added J23: SW2, Connector_JST:JST_XH_B2B-XH-AM_1x02_P2.50mm_Vertical, symbol Connector:Conn_01x02_Pin
- added J24: SW3, Connector_JST:JST_XH_B2B-XH-AM_1x02_P2.50mm_Vertical, symbol Connector:Conn_01x02_Pin
- added J25: MSHUB1, Connector_JST:JST_XH_B2B-XH-AM_1x02_P2.50mm_Vertical, symbol Connector:Conn_01x02_Pin
- added J26: MSHUB2, Connector_JST:JST_XH_B2B-XH-AM_1x02_P2.50mm_Vertical, symbol Connector:Conn_01x02_Pin
- added J27: MSBYPASS, Connector_JST:JST_XH_B2B-XH-AM_1x02_P2.50mm_Vertical, symbol Connector:Conn_01x02_Pin
- added J28: Conn_01x04, symbol Connector_Generic:Conn_01x04
- added J29: T1, Connector_JST:JST_XH_B2B-XH-AM_1x02_P2.50mm_Vertical, symbol Connector:Conn_01x02_Pin
- added J3: 3A, Connector_JST:JST_XH_B2B-XH-AM_1x02_P2.50mm_Vertical, symbol Connector:Conn_01x02_Pin
- added J30: T2, Connector_JST:JST_XH_B2B-XH-AM_1x02_P2.50mm_Vertical, symbol Connector:Conn_01x02_Pin
- added J31: T3, Connector_JST:JST_XH_B2B-XH-AM_1x02_P2.50mm_Vertical, symbol Connector:Conn_01x02_Pin
- added J4: 4A, Connector_JST:JST_XH_B2B-XH-AM_1x02_P2.50mm_Vertical, symbol Connector:Conn_01x02_Pin
- added J5: LED1, Connector_JST:JST_XH_B3B-XH-A_1x03_P2.50mm_Vertical, symbol Connector:Conn_01x03_Pin
- added J6: 1B, Connector_JST:JST_XH_B2B-XH-AM_1x02_P2.50mm_Vertical, symbol Connector:Conn_01x02_Pin
- added J7: 2B, Connector_JST:JST_XH_B2B-XH-AM_1x02_P2.50mm_Vertical, symbol Connector:Conn_01x02_Pin
- added J8: 3B, Connector_JST:JST_XH_B2B-XH-AM_1x02_P2.50mm_Vertical, symbol Connector:Conn_01x02_Pin
- added J9: 4B, Connector_JST:JST_XH_B2B-XH-AM_1x02_P2.50mm_Vertical, symbol Connector:Conn_01x02_Pin
- added JS4: SW4, Connector_JST:JST_XH_B2B-XH-AM_1x02_P2.50mm_Vertical, symbol Connector:Conn_01x02_Pin
- added JS5: T4, Connector_JST:JST_XH_B2B-XH-AM_1x02_P2.50mm_Vertical, symbol Connector:Conn_01x02_Pin
- added JS6: HT1, Connector_JST:JST_XH_B2B-XH-AM_1x02_P2.50mm_Vertical, symbol Connector:Conn_01x02_Pin
- added JS7: HT2, Connector_JST:JST_XH_B2B-XH-AM_1x02_P2.50mm_Vertical, symbol Connector:Conn_01x02_Pin
- added U2: ~, OpenA1K:Socketed MCU STM32 64P, symbol OpenA1KSymbols:STM32_64P_Thingo
- F1: value M_ATO_FUSE -> Mini ATO Fuse
- renumbered J1 to J10
Connections:
- net 5V: now also J17.3 (Pin_3), J18.3 (Pin_3), J20.3 (Pin_3), J5.3 (Pin_3)
- net GND: now also H2.1, H4.1, J1.2 (Pin_2), J11.2 (Pin_2), J12.2 (Pin_2), J14.2 (Pin_2), J15.2 (Pin_2), J17.1 (Pin_1), J18.1 (Pin_1), J2.2 (Pin_2), J20.1 (Pin_1), J21.2 (Pin_2), J23.2 (Pin_2), J24.2 (Pin_2), J25.2 (Pin_2), J26.2 (Pin_2), J27.2 (Pin_2), J29.2 (Pin_2), J3.2 (Pin_2), J30.2 (Pin_2), J31.2 (Pin_2), J4.2 (Pin_2), J5.1 (Pin_1), J6.2 (Pin_2), J7.2 (Pin_2), J8.2 (Pin_2), J9.2 (Pin_2), JS4.2 (Pin_2), JS5.2 (Pin_2), JS6.2 (Pin_2), JS7.2 (Pin_2)
- net MD_DIAG: now also U2.18 (PA7)
- net MD_DIR: now also U2.14 (PA3)
- net MD_EN: now also U2.12 (PA1)
- net MD_STEP: now also U2.13 (PA4)
- net VIN: now reaches F1.2, J10.2 (Pin_2)
- new net DC_1: J11.1 (Pin_1)
- new net DC_2: J12.1 (Pin_1)
- new net DC_3: J15.1 (Pin_1)
- new net DC_4: J14.1 (Pin_1)
- new net HT_C1: JS6.1 (Pin_1), U2.43 (PA12)
- new net HT_C2: JS7.1 (Pin_1), U2.44 (PA15)
- new net LED_1: J5.2 (Pin_2), U2.49 (PC8)
- new net LED_2: J17.2 (Pin_2), U2.50 (PC9)
- new net LED_3: J18.2 (Pin_2), U2.51 (PC6)
- new net LED_4: J20.2 (Pin_2), U2.52 (PC7)
- new net MA_DIAG: U2.15 (PA6)
- new net MA_DIR: U2.5 (PC0)
- new net MA_EN: U2.3 (PC14)
- new net MA_STEP: U2.4 (PC13)
- new net MB_DIAG: U2.16 (PA5)
- new net MB_DIR: U2.8 (PC1)
- new net MB_EN: U2.6 (PC15)
- new net MB_STEP: U2.7 (PC2)
- new net MC_DIAG: U2.17 (PC4)
- new net MC_DIR: U2.11 (PA2)
- new net MC_EN: U2.9 (PA0)
- new net MC_STEP: U2.10 (PC3)
- new net MS_1A: J1.1 (Pin_1), U2.31 (PB9)
- new net MS_1B: J6.1 (Pin_1), U2.33 (PB7)
- new net MS_2A: J2.1 (Pin_1), U2.34 (PB8)
- new net MS_2B: J7.1 (Pin_1), U2.35 (PB5)
- new net MS_3A: J3.1 (Pin_1), U2.36 (PB6)
- new net MS_3B: J8.1 (Pin_1), U2.37 (PB3)
- new net MS_4A: J4.1 (Pin_1), U2.38 (PB4)
- new net MS_4B: J9.1 (Pin_1), U2.39 (PC12)
- new net MS_BYPASS: J27.1 (Pin_1), U2.42 (PC11)
- new net MS_HUB1: J25.1 (Pin_1), U2.40 (PD2)
- new net MS_HUB2: J26.1 (Pin_1), U2.41 (PC10)
- new net SP1: J28.1 (Pin_1), U2.19 (PB0)
- new net SP2: J28.2 (Pin_2), U2.20 (PC5)
- new net SP3: J28.3 (Pin_3), U2.21 (PB2)
- new net SP4: J28.4 (Pin_4), U2.22 (PB1)
- new net SW_1: J21.1 (Pin_1), U2.45 (PA10)
- new net SW_2: J23.1 (Pin_1), U2.46 (PA11)
- new net SW_3: J24.1 (Pin_1), U2.47 (PA8)
- new net SW_4: JS4.1 (Pin_1), U2.48 (PA9)
- new net THM_1: J29.1 (Pin_1), U2.53 (PB14)
- new net THM_2: J30.1 (Pin_1), U2.54 (PB15)
- new net THM_3: J31.1 (Pin_1), U2.55 (PB12)
- new net THM_4: JS5.1 (Pin_1), U2.56 (PB13)
- no-connect marks 8 -> 0
Other:
- sheet DriveMotor renamed DMotor
- sheet SelectorMotor renamed CMotor
- added sheet AMotor (DriverSlot.kicad_sch)
- added sheet BMotor (DriverSlot.kicad_sch)
- sheet DMotor ports: added A1, A2, B1, B2; removed none
- note added: "Motors"
- note added: "POWER INPUT"
- note added: "STEPPER UART"
- note added: "USB"
- note removed: "AMS Motors"
- note removed: "Holes IG"
- moved on the sheet: F1, H1, H3, H5, J10, R1
