File: A1_AMS/DriverSlot.kicad_sch (KiCad schematic)
At the start: 3 parts, among them J4 Conn_01x04, M1 StepperMotor

Commit message: l
Parts:
- added C1: 100uF 63V, OpenA1K:Cap63V100UF, symbol Device:C_Polarized
Connections:
- net GND: now also C1.2
- net VIN: now also C1.1
Changed lines of the file:
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@@
 	(paper "A4")
+	(junction
+		(at 176.53 83.82)
+		(diameter 0)
+		(color 0 0 0 0)
+	)
 	(junction
 		(at 175.26 93.98)
@@
 	)
 	(junction
+		(at 168.91 81.28)
+		(diameter 0)
+		(color 0 0 0 0)
+	)
+	(junction
 		(at 175.26 96.52)
 		(diameter 0)
@@
 	(wire
 		(pts
-			(xy 168.91 78.105) (xy 168.91 83.82)
+			(xy 168.91 78.105) (xy 168.91 81.28)
 		)
 		(stroke
@@
 	(wire
 		(pts
+			(xy 168.91 81.28) (xy 168.91 83.82)
+		)
+		(stroke
+			(width 0)
+			(type default)
+		)
+	)
+	(wire
+		(pts
 			(xy 175.26 96.52) (xy 177.8 96.52)
 		)
@@
 		(pts
 			(xy 168.91 88.9) (xy 175.26 88.9)
+		)
+		(stroke
+			(width 0)
+			(type default)
+		)
+	)
+	(wire
+		(pts
+			(xy 176.53 81.28) (xy 176.53 83.82)
 		)
 		(stroke
@@
 					(unit 1)
 				)
+			)
+		)
+	)
+	(symbol
+		(lib_id "Device:C_Polarized")
+		(at 172.72 81.28 90)
+		(unit 1)
+		(exclude_from_sim no)
+		(in_bom yes)
+		(on_board yes)
+		(dnp no)
+		(fields_autoplaced yes)
+		(property "Reference" "C1"
+			(at 171.831 73.66 90)
+			(effects
+				(font
+					(size 1.27 1.27)
+				)
+			)
+		)
+		(property "Value" "100uF 63V"
+			(at 171.831 76.2 90)
+			(effects
+				(font
+					(size 1.27 1.27)
+				)
+			)
+		)
+		(property "Footprint" "OpenA1K:Cap63V100UF"
+			(at 176.53 80.3148 0)
+			(effects
+				(font
+					(size 1.27 1.27)
+				)
+				(hide yes)
+			)
+		)
+		(property "Datasheet" "~"
+			(at 172.72 81.28 0)
+			(effects
+				(font
+					(size 1.27 1.27)
+				)
+				(hide yes)
+			)
+		)
+		(property "Description" "Polarized capacitor"
+			(at 172.72 81.28 0)
+			(effects
+				(font
+					(size 1.27 1.27)
+				)
+				(hide yes)
+			)
+		)
+		(pin "1"
+		)
+		(pin "2"
+		)
+		(instances
+			(project ""
+				(path "/989d6d42-19bd-451f-8ed3-d8ee079df240/2a25a3b1-37eb-4dde-897c-41aa70453add"
+					(reference "C2")
+					(unit 1)
+				)
+				(path "/989d6d42-19bd-451f-8ed3-d8ee079df240/da5b7a11-adf7-487a-b63f-2d36df684954"
+					(reference "C1")
+					(unit 1)
+				)

Commit message: e
e
Parts:
- C1: value 100uF 63V -> 470uF; footprint OpenA1K:Cap63V100UF -> OpenA1K:Cap ~ 12.5, 2.5mm-7.5mm pitch
- M1: value StepperMotor -> TMC2209 Breakout
- renumbered J4 to J13
Other:
- note added: "Enstop"
- note added: "Sensorless Homing"
