File: A1_THB/ExtruderDriver.kicad_sch (KiCad schematic)
At the start: 4 parts, among them M1 StepperMotor

Commit message: e
e
Connections:
- net EN renamed ENABLE
Changed lines of the file:
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@@
 		)
 	)
-	(hierarchical_label "EN"
+	(hierarchical_label "ENABLE"
 		(shape input)
 		(at 127 88.9 180)
