File: A1_THB/A1_THB.kicad_pcb (KiCad board)
At the start: 2 copper layers, 12 parts, among them J10 SFS, J11 Probe, J12 Hotend, J3 Pico Conn1, J4 Pico Conn2, J5 Pico Conn3, J6 Thermister, J7 Conn_02x04_Odd_Even, J8 PCF, J9 EXF

Commit message: e
e
Parts:
- removed J10: SFS, Connector_PinHeader_2.54mm:PinHeader_1x05_P2.54mm_Vertical
- removed J11: Probe, Connector_PinHeader_2.54mm:PinHeader_1x05_P2.54mm_Vertical
- removed J12: Hotend, Connector_JST:JST_XH_B2B-XH-AM_1x02_P2.50mm_Vertical
- removed J9: EXF, Connector_JST:JST_XH_B5B-XH-AM_1x05_P2.50mm_Vertical
- added C1: 100uF 63V, OpenA1K:Cap63V100UF, F.Cu at (87.5, 108.5)
- added J2: Conn_01x04, Connector_JST:JST_XH_B4B-XH-A_1x04_P2.50mm_Vertical, F.Cu at (53.0, 120.5)
- added M1: StepperMotor, OpenA1K:TMC2209 Footprint, F.Cu at (84.0, 115.7)
- added R2: 10kΩ, Resistor_THT:R_Axial_DIN0207_L6.3mm_D2.5mm_P10.16mm_Horizontal, F.Cu at (93.5, 118.9)
- added U1: RP2040-ZERO, Libraries:RP2040-ZERO, F.Cu at (73.0, 114.5)
- ExtruderMotor1: footprint Connector_JST:JST_XH_B4B-XH-AM_1x04_P2.50mm_Vertical -> Connector_JST:JST_XH_B4B-XH-A_1x04_P2.50mm_Vertical
- J3: value Pico Conn1 -> Probe; footprint Connector_PinHeader_2.54mm:PinHeader_1x06_P2.54mm_Vertical -> Connector_PinHeader_2.54mm:PinHeader_1x05_P2.54mm_Vertical
- J4: value Pico Conn2 -> Molex 2x02; footprint Connector_PinHeader_2.54mm:PinHeader_1x06_P2.54mm_Vertical -> Connector_PinSocket_2.54mm:PinSocket_2x02_P2.54mm_Vertical
- J5: value Pico Conn3 -> PCF; footprint Connector_PinHeader_2.54mm:PinHeader_1x06_P2.54mm_Vertical -> Connector_JST:JST_XH_B4B-XH-AM_1x04_P2.50mm_Vertical
- J6: value Thermister -> EXF; footprint Connector_JST:JST_XH_B2B-XH-AM_1x02_P2.50mm_Vertical -> Connector_JST:JST_XH_B5B-XH-AM_1x05_P2.50mm_Vertical
- J7: value Conn_02x04_Odd_Even -> Thermister; footprint Connector_Molex:Molex_Micro-Fit_3.0_43045-0818_2x04-1MP_P3.00mm_Vertical -> Connector_JST:JST_XH_B2B-XH-AM_1x02_P2.50mm_Vertical
- J8: value PCF -> Hotend; footprint Connector_JST:JST_XH_B4B-XH-AM_1x04_P2.50mm_Vertical -> OpenA1K:1x2 Terminal Block
- moved J7 109.6 mm to (66.8, 130.0)
- moved J8 87.8 mm to (56.5, 127.5), turned to -90 degrees
- moved J5 79.9 mm to (85.5, 140.0)
- moved J3 71.8 mm to (52.0, 105.3)
- moved J6 69.3 mm to (69.5, 140.0)
- moved J4 67.4 mm to (61.5, 105.0)
- moved ExtruderMotor1 52.2 mm to (96.0, 111.0), turned to 90 degrees
- moved R1 36.8 mm to (77.5, 109.4), turned to -90 degrees
Connections:
- ExtruderMotor1 pad 1: /COIL-B2 -> /ExtruderDriver/B2
- ExtruderMotor1 pad 2: /COIL-B1 -> /ExtruderDriver/B1
- ExtruderMotor1 pad 3: /COIL-A1 -> /ExtruderDriver/A1
- ExtruderMotor1 pad 4: /COIL-A2 -> /ExtruderDriver/A2
- J3 pad 1: /SFS_SW -> /GND_LV
- J3 pad 2: /HT_CT -> /5V
- J3 pad 3: /BL_PR -> /BL_SV
- J3 pad 4: /BL_SV -> /GND_LV
- J3 pad 5: /PCF_PWM -> /BL_PR
- J4 pad 1: /SFS_OP -> /24v
- J4 pad 2: /EXF_SG -> /GND
- J4 pad 3: /PCF_SG -> /D-
- J4 pad 4: /THM_SG -> /D+
- J5 pad 1: /GND_LV -> /GND
- J5 pad 2: /GND_LV -> /24V
- J5 pad 3: /3V3 -> /PCF_SG
- J5 pad 4: /5V -> /EXF_PWM
- J6 pad 1: /3V3 -> unconnected-(J6-Pin_1-Pad1)
- J6 pad 2: /THM_SG -> /GND_LV
- J7 pad 1: /24v -> /3V3
- J7 pad 2: /COIL-A2 -> /THM_SG
- J8 pad 1: /GND -> Net-(D1-A)

Commit message: e
e
Parts:
- added D1: D, Diode_THT:D_5KPW_P12.70mm_Horizontal, F.Cu at (116.8, 123.5)
Other:
- board outline added: 50 x 44 mm

Commit message: e
e
Parts:
- J8: footprint OpenA1K:1x2 Terminal Block -> Libraries:CUI_TB004-508-05BE
- moved D1 92.2 mm to (28.6, 150.5)
- moved J8 22.6 mm to (34.0, 124.8)

Commit message: e
e
Parts:
- removed D1: D, Diode_THT:D_5KPW_P12.70mm_Horizontal
- added D2: D, A1_THB:DIOAD1036W78L470D235, F.Cu at (75.0, 135.5)
- added D3: D, A1_THB:DIOAD1036W78L470D235, F.Cu at (87.8, 135.5)
- added J1: Conn_01x02, Connector_JST:JST_XH_B2B-XH-AM_1x02_P2.50mm_Vertical, F.Cu at (54.5, 106.5)
- J4: value Molex 2x02 -> MolexS1; footprint Connector_PinSocket_2.54mm:PinSocket_2x02_P2.54mm_Vertical -> OpenA1K:ScrewTerminal 7mm x 7mm
- J7: value Thermister -> Molex S2; footprint Connector_JST:JST_XH_B2B-XH-AM_1x02_P2.50mm_Vertical -> OpenA1K:ScrewTerminal 7mm x 7mm
- J8: footprint Libraries:CUI_TB004-508-05BE -> OpenA1K:ScrewTerminal 7mm x 7mm
- R1: value 10kO -> 1k
- moved J4 25.9 mm to (67.8, 130.1), turned to 90 degrees
- moved J8 19.8 mm to (53.7, 122.9)
- moved J7 19.4 mm to (54.3, 115.1), turned to 90 degrees
- moved J3 14.2 mm to (61.5, 115.8)
- moved J2 11.0 mm to (53.0, 131.5)
- moved C1 1.50 mm to (87.5, 107.0)
- moved R1 1.50 mm to (77.5, 107.9)
- moved M1 0.93 mm to (84.0, 114.8)
- moved ExtruderMotor1 0.71 mm to (95.5, 110.5)
Connections:
- C1 pad 1: /ExtruderDriver/VIN -> /24V
- J2 pad 1: unconnected-(J2-Pin_1-Pad1) -> /GND_LV
- J2 pad 3: unconnected-(J2-Pin_3-Pad3) -> /3V3
- J4 pad 1: /24v -> /24V
- J4 pad 2: /GND -> GND
- J5 pad 1: /GND -> /24V
- J5 pad 2: /24V -> GND
- J5 pad 4: /EXF_PWM -> unconnected-(J5-Pin_4-Pad4)
- J6 pad 2: /GND_LV -> /5V
- J6 pad 3: /5V -> /GND_LV
- J6 pad 5: /EXF_PWM -> unconnected-(J6-Pin_5-Pad5)
- J7 pad 1: /3V3 -> /HT1
- J7 pad 2: /THM_SG -> /HT2
- J8 pad 1: Net-(D1-A) -> /HT1
- J8 pad 2: /24V -> /HT2
- M1 pad 1: /ExtruderDriver/EN -> /ExtruderDriver/ENABLE
- M1 pad 16: /ExtruderDriver/VIN -> /24V
- M1 pad 2: /GND -> GND
- M1 pad 3: /GND -> GND
- R1 pad 1: /HT_CT -> /ExtruderDriver/UART
- R1 pad 2: Net-(Q1-G) -> Net-(U1-GP4)
- R2 pad 1: /ExtruderDriver/EN -> /ExtruderDriver/ENABLE
- U1 pad 1: /SFS_SW -> unconnected-(U1-GP0-Pad1)
- U1 pad 13: /ENABLE -> /ExtruderDriver/ENABLE
- U1 pad 14: /ExtruderDriver/UART -> unconnected-(U1-GP13-Pad14)
- U1 pad 15: /PCF_CT -> /PCF_SG
- U1 pad 16: /PCF_SG -> /EXF_SG
- U1 pad 17: /EXF_CT -> /SFS_SW
- U1 pad 18: /EXF_SG -> /SFS_ENC
- U1 pad 2: /SFS_ENC -> unconnected-(U1-GP1-Pad2)
- U1 pad 21: unconnected-(U1-3V3-Pad21) -> /3V3
- U1 pad 22: unconnected-(U1-GND-Pad22) -> /GND_LV
- U1 pad 23: unconnected-(U1-5V-Pad23) -> /5V
- U1 pad 4: /HT_CT -> /ExtruderDriver/UART
- U1 pad 5: unconnected-(U1-GP4-Pad5) -> Net-(U1-GP4)
Routing:
- net GND: track 0.00 -> 98.4 mm
- net /GND_LV: track 0.00 -> 79.4 mm
- net /24V: track 0.00 -> 71.0 mm
- net /5V: track 0.00 -> 55.6 mm
- net /ExtruderDriver/ENABLE: track 0.00 -> 48.0 mm, vias 0 -> 1
- net /3V3: track 0.00 -> 43.5 mm
- net /EXF_SG: track 0.00 -> 35.4 mm, vias 0 -> 1
- net /THM_SG: track 0.00 -> 26.8 mm
- net /ExtruderDriver/UART: track 0.00 -> 25.1 mm, vias 0 -> 2
- net /ExtruderDriver/DIR: track 0.00 -> 23.8 mm, vias 0 -> 1
- net /ExtruderDriver/B1: track 0.00 -> 22.4 mm, vias 0 -> 1
- net /ExtruderDriver/STEP: track 0.00 -> 21.7 mm, vias 0 -> 3
- net /SFS_ENC: track 0.00 -> 19.8 mm
- net /ExtruderDriver/B2: track 0.00 -> 18.8 mm
- net /ExtruderDriver/A2: track 0.00 -> 18.8 mm
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- added copper zone on B.Cu, net GND
- added copper zone on F.Cu, net GND
Other:
- outline, holes or cut-outs redrawn
- board text added: "A"
- board text added: "C"

Commit message: e
e
Parts:
- added R3: 10k, Resistor_THT:R_Axial_DIN0207_L6.3mm_D2.5mm_P10.16mm_Horizontal, F.Cu at (67.9, 104.5)
- added R4: 10k, Resistor_THT:R_Axial_DIN0207_L6.3mm_D2.5mm_P10.16mm_Horizontal, F.Cu at (68.5, 111.9)
- added R5: 10k, Resistor_THT:R_Axial_DIN0207_L6.3mm_D2.5mm_P10.16mm_Horizontal, F.Cu at (73.0, 111.9)
- J8: value Hotend -> e
- moved R1 4.00 mm to (77.5, 111.9)
- moved PROBE 1.00 mm to (61.5, 116.8)
- moved J4 1.00 mm to (66.8, 130.3)
- moved J2 0.50 mm to (53.0, 132.0)
- renumbered J3 to PROBE
Connections:
- net /24V renamed +24V
- net /5V renamed +5V
- net /ExtruderDriver/UART renamed /M_UART
- net /HT1 renamed Net-(J7-Pin_1)
- net /HT2 renamed Net-(J7-Pin_2)
- D2 pad 2: /GND_LV -> GND
- J5 pad 4: unconnected-(J5-Pin_4-Pad4) -> Net-(J5-Pin_4)
- J6 pad 3: /GND_LV -> GND
- J6 pad 5: unconnected-(J6-Pin_5-Pad5) -> Net-(J6-Pin_5)
- PROBE pad 1: /GND_LV -> GND
- PROBE pad 4: /GND_LV -> GND
- U1 pad 11: /ExtruderDriver/STEP -> /M_STEP
- U1 pad 12: /ExtruderDriver/DIR -> /M_DIR
- U1 pad 13: /ExtruderDriver/ENABLE -> /M_EN
- U1 pad 21: /3V3 -> +3V3
- U1 pad 22: /GND_LV -> GND
Routing:
- net (no net): track 0.00 -> 86.2 mm
- net +24V: track 71.0 -> 10.00 mm
- net /M_UART: track 25.1 -> 0.00 mm
Other:
- board text added: "+24V"
- board text added: "GND"

Commit message: e
e
Parts:
- J2: value Conn_01x04 -> SFS
- J8: value e -> Hotend
- R1: value 1k -> 1kΩ
- R4, R5: value 10k -> 10kΩ
- renumbered PROBE to J3
Other:
- board text removed: "A"
- board text removed: "C"
Changed lines of the file:
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@@
 		(descr "Through hole straight pin header, 1x05, 2.54mm pitch, single row")
 		(tags "Through hole pin header THT 1x05 2.54mm single row")
-		(property "Reference" "PROBE"
+		(property "Reference" "J3"
 			(at 0 -2.33 0)
 			(layer "F.SilkS")
@@
 		(tags "Resistor Axial_DIN0207 series Axial Horizontal pin pitch 10.16mm 0.25W = 1/4W length 6.3mm diameter 2.5mm")
 		(property "Reference" "R2"
-			(at 5.08 -2.37 90)
-			(layer "B.SilkS")
+			(at 5.08 0 90)
+			(layer "F.SilkS")
 			(effects
 				(font
@@
 			)
 		)
-		(property "Value" "10k"
+		(property "Value" "10kΩ"
 			(at 5.08 0 90)
 			(layer "F.SilkS")
@@
 			)
 		)
-		(property "Value" "e"
+		(property "Value" "Hotend"
 			(at -0.0814 2.8956 270)
 			(unlocked yes)
@@
 			)
 		)
-		(property "Value" "10k"
+		(property "Value" "10kΩ"
 			(at 5.08 0 90)
 			(layer "F.SilkS")
@@
 		)
 		(property "Value" "EXF"
-			(at 5 4.6 0)
-			(layer "F.Fab")
+			(at -10 2 0)
+			(layer "F.SilkS")
 			(effects
 				(font
@@
 			)
 		)
-		(property "Value" "Conn_01x04"
+		(property "Value" "SFS"
 			(at 3.75 4.6 0)
-			(layer "F.Fab")
+			(layer "F.SilkS")
 			(effects
 				(font
 					(size 1 1)
-					(thickness 0.15)
+					(thickness 0.125)
 				)
 			)
@@
 			)
 		)
-		(property "Value" "1k"
+		(property "Value" "1kΩ"
 			(at 7.08 0 90)
 			(layer "F.SilkS")
@@
 		(tags "connector JST XH vertical boss")
 		(property "Reference" "J5"
-			(at 16.5 0.525 0)
+			(at -0.5 3.5 0)
 			(layer "F.SilkS")
 			(effects
@@
 		(layer "Edge.Cuts")
 	)
-	(gr_text "A"
-		(at 118 146.5 0)
-		(layer "F.SilkS")
-		(effects
-			(font
-				(size 1 1)
-				(thickness 0.15)
-			)
-		)
-	)
 	(gr_text "+24V"
 		(at 70 132.5 0)
@@
 		)
 	)
-	(gr_text "C"
-		(at 103 146.5 0)
-		(layer "F.SilkS")
-		(effects
-			(font
-				(size 1 1)
-				(thickness 0.15)
-			)
-		)
-	)
 	(gr_text "GND"
 		(at 70.5 130 0)
@@
 	)
 	(zone
-		(net 32)
-		(net_name "Net-(J7-Pin_2)")
+		(net 19)
+		(net_name "Net-(J7-Pin_1)")
 		(layer "B.Cu")
 		(name "$teardrop_padvia$")
 		(hatch full 0.1)
-		(priority 30001)
+		(priority 30000)
 		(attr
 			(teardrop
@@
 		(polygon
 			(pts
-				(xy 51.774737 124.052077) (xy 51.891173 124.161673) (xy 51.999654 124.250557) (xy 52.099758 124.32032)
-				(xy 52.194675 124.37523) (xy 52.382468 124.453487) (xy 52.635756 124.516431) (xy 52.806115 124.554901)
-				(xy 52.992321 124.611608) (xy 53.202413 124.703135) (xy 53.44443 124.84607) (xy 54.000707 124.015307)
-				(xy 53.80491 123.033815) (xy 53.604564 123.0914) (xy 53.40551 123.18306) (xy 53.298308 123.24248)
-				(xy 53.130234 123.331011) (xy 53.051014 123.360219) (xy 52.972345 123.374318) (xy 52.89223 123.369504)
-				(xy 52.808676 123.341973) (xy 52.719686 123.287923) (xy 52.623264 123.20355)
+				(xy 53.4 119.519215) (xy 53.395169 119.745871) (xy 53.381356 119.934664) (xy 53.360735 120.087108)
+				(xy 53.333745 120.219835) (xy 53.256169 120.4783) (xy 53.227974 120.558746) (xy 53.125981 120.86715)
+				(xy 53.072536 121.064488) (xy 53.019215 121.30491) (xy 54 121.501) (xy 54.980785 121.30491) (xy 54.882937 120.897704)
+				(xy 54.772026 120.558748) (xy 54.703827 120.356813) (xy 54.649284 120.141845) (xy 54.613106 119.875445)
+				(xy 54.6 119.519215)
 			)
 		)
@@
 	)
 	(zone
-		(net 19)
-		(net_name "Net-(J7-Pin_1)")
+		(net 32)
+		(net_name "Net-(J7-Pin_2)")
 		(layer "B.Cu")
 		(name "$teardrop_padvia$")
 		(hatch full 0.1)
-		(priority 30000)
+		(priority 30001)
 		(attr
 			(teardrop
@@
 		(polygon
 			(pts
-				(xy 53.4 119.519215) (xy 53.395169 119.745871) (xy 53.381356 119.934664) (xy 53.360735 120.087108)
-				(xy 53.333745 120.219835) (xy 53.256169 120.4783) (xy 53.227974 120.558746) (xy 53.125981 120.86715)
-				(xy 53.072536 121.064488) (xy 53.019215 121.30491) (xy 54 121.501) (xy 54.980785 121.30491) (xy 54.882937 120.897704)
-				(xy 54.772026 120.558748) (xy 54.703827 120.356813) (xy 54.649284 120.141845) (xy 54.613106 119.875445)
-				(xy 54.6 119.519215)
+				(xy 51.774737 124.052077) (xy 51.891173 124.161673) (xy 51.999654 124.250557) (xy 52.099758 124.32032)
+				(xy 52.194675 124.37523) (xy 52.382468 124.453487) (xy 52.635756 124.516431) (xy 52.806115 124.554901)
+				(xy 52.992321 124.611608) (xy 53.202413 124.703135) (xy 53.44443 124.84607) (xy 54.000707 124.015307)
+				(xy 53.80491 123.033815) (xy 53.604564 123.0914) (xy 53.40551 123.18306) (xy 53.298308 123.24248)
+				(xy 53.130234 123.331011) (xy 53.051014 123.360219) (xy 52.972345 123.374318) (xy 52.89223 123.369504)
+				(xy 52.808676 123.341973) (xy 52.719686 123.287923) (xy 52.623264 123.20355)
 			)
 		)
