File: A1_MB/A1_MB.kicad_pcb (KiCad board)
At the start: 2 copper layers, 180 x 60 mm, 34 parts, among them J1 Conn_02x04_Counter_Clockwise, J10 Conn_01x03, J11 Conn_01x04, J12 Conn_01x02_Pin, J13 Conn_01x03, J14 Conn_01x04, J2 Screw_Terminal_01x02, J3 Conn_01x02_Pin, J4 Conn_01x03, J5 Conn_01x04, J6 Conn_01x02_Pin, J7 Conn_01x03, J8 Conn_01x04, J9 Conn_01x02_Pin, M2 TMC2209 Breakout, M4 TMC2209 Breakout, U1 Pico

Commit message: e
e
Parts:
- removed J1: Conn_02x04_Counter_Clockwise, Connector_PinHeader_2.54mm:PinHeader_2x04_P2.54mm_Vertical
- removed J12: Conn_01x02_Pin, Connector_PinHeader_2.54mm:PinHeader_1x02_P2.54mm_Vertical
- removed J13: Conn_01x03, Connector_JST:JST_XH_B3B-XH-AM_1x03_P2.50mm_Vertical
- removed J14: Conn_01x04, Connector_JST:JST_XH_B4B-XH-A_1x04_P2.50mm_Vertical
- removed X_MOTOR, Z_MOTOR: TMC2209 Breakout, OpenA1K:TMC2209 Footprint
- added C5: 220uF, Capacitor_THT:CP_Radial_D8.0mm_P3.50mm, F.Cu at (154.0, 72.0)
- added J16: SensorlessHoming, Connector_PinHeader_2.54mm:PinHeader_1x02_P2.54mm_Vertical, F.Cu at (74.2, 72.0)
- added J17: Endstop, Connector_JST:JST_XH_B3B-XH-AM_1x03_P2.50mm_Vertical, F.Cu at (73.0, 38.0)
- added J18: SensorlessHoming, Connector_PinHeader_2.54mm:PinHeader_1x02_P2.54mm_Vertical, F.Cu at (121.1, 72.3)
- added J19: Endstop, Connector_JST:JST_XH_B3B-XH-AM_1x03_P2.50mm_Vertical, F.Cu at (95.0, 38.0)
- added J20: Conn_01x04, Connector_JST:JST_XH_B4B-XH-A_1x04_P2.50mm_Vertical, F.Cu at (135.9, 88.5)
- added J21: SensorlessHoming, Connector_PinHeader_2.54mm:PinHeader_1x02_P2.54mm_Vertical, F.Cu at (98.4, 72.0)
- added J22: Endstop, Connector_JST:JST_XH_B3B-XH-AM_1x03_P2.50mm_Vertical, F.Cu at (84.0, 38.0)
- added J23: Conn_01x04, Connector_JST:JST_XH_B4B-XH-A_1x04_P2.50mm_Vertical, F.Cu at (113.0, 88.5)
- added J24: SensorlessHoming, Connector_PinHeader_2.54mm:PinHeader_1x02_P2.54mm_Vertical, F.Cu at (89.0, 46.5)
- added J25: Endstop, Connector_JST:JST_XH_B3B-XH-AM_1x03_P2.50mm_Vertical, F.Cu at (106.0, 38.0)
- added J26: Conn_01x04, Connector_JST:JST_XH_B4B-XH-A_1x04_P2.50mm_Vertical, F.Cu at (72.5, 61.0)
- added M1: TMC2209 Breakout, OpenA1K:TMC2209 Footprint, F.Cu at (71.8, 75.3)
- added M3: TMC2209 Breakout, OpenA1K:TMC2209 Footprint, F.Cu at (95.7, 75.6)
- added MotorConnector1: Conn_01x04, Connector_JST:JST_XH_B4B-XH-A_1x04_P2.50mm_Vertical, F.Cu at (89.0, 88.0)
- added Q1: HB_NMOS, OpenA1K:TO254P1054X469X1930-3, F.Cu at (175.5, 80.6)
- added Q2: HE_NMOS, OpenA1K:TO254P1054X469X1930-3, F.Cu at (208.5, 80.6)
- added Q3: RGB_NMOS, OpenA1K:TO254P1054X469X1930-3, F.Cu at (197.5, 80.6)
- added Q4: FAN_NMOS, OpenA1K:TO254P1054X469X1930-3, F.Cu at (186.5, 80.6)
- added R10: 10k, Resistor_THT:R_Axial_DIN0207_L6.3mm_D2.5mm_P10.16mm_Horizontal, F.Cu at (167.0, 76.5)
- added R11: 10k, Resistor_THT:R_Axial_DIN0207_L6.3mm_D2.5mm_P10.16mm_Horizontal, F.Cu at (163.5, 76.6)
- added R12: 10kΩ, Resistor_THT:R_Axial_DIN0207_L6.3mm_D2.5mm_P10.16mm_Horizontal, F.Cu at (75.0, 78.0)
- added R13: 10kΩ, Resistor_THT:R_Axial_DIN0207_L6.3mm_D2.5mm_P10.16mm_Horizontal, F.Cu at (122.0, 78.4)
- added R14: 10kΩ, Resistor_THT:R_Axial_DIN0207_L6.3mm_D2.5mm_P10.16mm_Horizontal, F.Cu at (99.0, 78.5)
- added R15: 10kΩ, Resistor_THT:R_Axial_DIN0207_L6.3mm_D2.5mm_P10.16mm_Horizontal, F.Cu at (82.6, 47.0)
- added R6: 1k, Resistor_THT:R_Axial_DIN0207_L6.3mm_D2.5mm_P10.16mm_Horizontal, F.Cu at (199.5, 66.3)
- added R7: 100k, Resistor_THT:R_Axial_DIN0207_L6.3mm_D2.5mm_P10.16mm_Horizontal, F.Cu at (189.0, 66.3)
- added R8: 1k, Resistor_THT:R_Axial_DIN0207_L6.3mm_D2.5mm_P10.16mm_Horizontal, F.Cu at (185.5, 66.3)
- added R9: 1kΩ, Resistor_THT:R_Axial_DIN0207_L6.3mm_D2.5mm_P10.16mm_Horizontal, F.Cu at (135.9, 65.5)
- C1, C2, C3, C4: value 470uF -> 220uF; footprint OpenA1K:Cap ~ 12.5, 2.5mm-7.5mm pitch -> Capacitor_THT:CP_Radial_D8.0mm_P3.50mm
- J10: value Conn_01x03 -> Screw_Terminal_01x02; footprint Connector_JST:JST_XH_B3B-XH-AM_1x03_P2.50mm_Vertical -> OpenA1K:1x2 Terminal Block
- J11: value Conn_01x04 -> Bed Thermisters
- J2: value Screw_Terminal_01x02 -> Neopixel; footprint OpenA1K:1x2 Terminal Block -> Connector_JST:JST_XH_B3B-XH-AM_1x03_P2.50mm_Vertical
- J3: value Conn_01x02_Pin -> FAN0_VS; footprint Connector_PinHeader_2.54mm:PinHeader_1x02_P2.54mm_Vertical -> Connector_PinHeader_2.54mm:PinHeader_1x03_P2.54mm_Vertical
- J4: value Conn_01x03 -> RGB_2PIN; footprint Connector_JST:JST_XH_B3B-XH-AM_1x03_P2.50mm_Vertical -> Connector_JST:JST_XH_B2B-XH-AM_1x02_P2.50mm_Vertical
- J5: value Conn_01x04 -> Molex 2x02 Microfit; footprint Connector_JST:JST_XH_B4B-XH-A_1x04_P2.50mm_Vertical -> Connector_Molex:Molex_Micro-Fit_3.0_43045-0412_2x02_P3.00mm_Vertical
- J6: value Conn_01x02_Pin -> HeatedBed; footprint Connector_PinHeader_2.54mm:PinHeader_1x02_P2.54mm_Vertical -> OpenA1K:ScrewTerminal 7mm x 7mm
- J7: value Conn_01x03 -> FAN0
- J8: value Conn_01x04 -> SFS; footprint Connector_JST:JST_XH_B4B-XH-A_1x04_P2.50mm_Vertical -> Connector_JST:JST_XH_B4B-XH-AM_1x04_P2.50mm_Vertical
- J9: value Conn_01x02_Pin -> Hotend; footprint Connector_PinHeader_2.54mm:PinHeader_1x02_P2.54mm_Vertical -> OpenA1K:ScrewTerminal 7mm x 7mm
- R1: value 1kΩ -> 100k
- R2, R5: value 10kΩ -> 100k
- R3, R4: value 10kΩ -> 1k
- U1: value Pico -> ~; footprint OpenA1K:Socketed MCU - Pico (No Text) -> OpenA1K:STM32 Blackpill Socketed
- moved C4 115.5 mm to (89.0, 62.5), turned to 180 degrees
- moved R1 111.0 mm to (178.0, 66.3), turned to -90 degrees
- moved M4 99.9 mm to (85.2, 43.8), turned to -90 degrees
- moved J2 69.1 mm to (199.0, 61.0), turned to 180 degrees
- moved U1 68.4 mm to (148.4, 53.1)
- moved C1 67.1 mm to (90.0, 70.5)
- moved C3 53.0 mm to (113.5, 69.5), turned to -90 degrees
- moved M2 51.1 mm to (118.7, 75.6), turned to 0 degrees
- moved J7 50.6 mm to (183.5, 91.0), turned to 0 degrees
- moved J11 49.9 mm to (164.5, 92.0), turned to 90 degrees
- moved J8 45.0 mm to (188.0, 61.0), turned to 180 degrees
- moved C2 44.0 mm to (137.0, 70.8)
- moved J10 42.8 mm to (143.0, 88.5), turned to 0 degrees
- moved R5 35.3 mm to (202.5, 66.3), turned to -90 degrees
- moved J4 35.1 mm to (197.0, 91.0), turned to 0 degrees
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- renumbered H5 to H1, H10 to H2, H6 to H3, H9 to H4, H7 to H5
Connections:
- C1 pad 1: /M_VBUS -> +24V
- C2 pad 1: /M_VBUS -> +24V
- C3 pad 1: /M_VBUS -> +24V
- C4 pad 1: /M_VBUS -> +24V
- F1 pad 1: /M_VBUS -> +24V
- F1 pad 2: /VIN -> Net-(J10-Pin_2)
- J10 pad 1: +3V3 -> GND
- J10 pad 2: /MZ_DIAG -> Net-(J10-Pin_2)
- J11 pad 1: /ZMotor/COIL-B2 -> +3V3
- J11 pad 2: /ZMotor/COIL-B1 -> /BED_THM_2
- J11 pad 3: /ZMotor/COIL-A1 -> +3V3
- J11 pad 4: /ZMotor/COIL-A2 -> /BED_THM_1
- J2 pad 1: GND -> +5V
- J2 pad 2: /VIN -> /NEOPIXEL_PIN
- J3 pad 1: /MX_DIAG -> +5V
- J4 pad 1: +3V3 -> +5V
- J4 pad 2: /MX_DIAG -> Net-(J4-Pin_2)
- J5 pad 1: /XMotor/COIL-B2 -> 24V
- J5 pad 2: /XMotor/COIL-B1 -> GND
- J5 pad 3: /XMotor/COIL-A1 -> /HEATER_RETURN
- J5 pad 4: /XMotor/COIL-A2 -> 24V
- J6 pad 1: /MY_DIAG -> 24V
- J6 pad 2: Net-(J6-Pin_2) -> /HEATED_BED_RETURN
- J7 pad 1: +3V3 -> Net-(J3-Pin_2)
- J7 pad 2: /MY_DIAG -> GND
- J7 pad 3: GND -> 3V3
- J8 pad 1: /YMotor/COIL-B2 -> +5V
- J8 pad 2: /YMotor/COIL-B1 -> /SwitchSensor
- J8 pad 3: /YMotor/COIL-A1 -> GND
- J8 pad 4: /YMotor/COIL-A2 -> /OpticSensor
- J9 pad 1: /MZ_DIAG -> 24V
- J9 pad 2: Net-(J9-Pin_2) -> /HEATER_RETURN
- M2 pad 11: /YMotor/COIL-B2 -> /YMotor/B2
- M2 pad 12: /YMotor/COIL-B1 -> /YMotor/B1
- M2 pad 13: /YMotor/COIL-A1 -> /YMotor/A1
- M2 pad 14: /YMotor/COIL-A2 -> /YMotor/A2
- M2 pad 16: /M_VBUS -> +24V
- M2 pad 18: Net-(J6-Pin_2) -> Net-(J18-Pin_2)
- M2 pad 2: /3V3 -> +3V3
- M4 pad 11: /EMotor/COIL-B2 -> /EMotor/B2
- M4 pad 12: /EMotor/COIL-B1 -> /EMotor/B1
- M4 pad 13: /EMotor/COIL-A1 -> /EMotor/A1
- M4 pad 14: /EMotor/COIL-A2 -> /EMotor/A2
- M4 pad 16: /M_VBUS -> +24V
- M4 pad 2: /3V3 -> +3V3
- M4 pad 3: /3V3 -> +3V3
- R1 pad 1: /UART_RX -> / HEATED_BED_PIN
- R1 pad 2: /M_UART -> GND
- R2 pad 1: /MX_EN -> /HEATER_PIN
- R2 pad 2: +3V3 -> GND
- R3 pad 1: /MY_EN -> / HEATED_BED_PIN
- R3 pad 2: +3V3 -> Net-(Q1-G)
- R4 pad 1: /MZ_EN -> /HEATER_PIN
- R4 pad 2: +3V3 -> Net-(Q2-G)
- R5 pad 1: /ME_EN -> /RGB_PIN
- R5 pad 2: +3V3 -> GND
- U1 pad 1: /MX_EN -> unconnected-(U1-VBAT-Pad1)
- U1 pad 10: /MY_STEP -> /OpticSensor
- U1 pad 11: /MY_DIR -> /SwitchSensor
- U1 pad 12: /S_GPIO9 -> /MS_EN
- U1 pad 13: GND -> /MZ_DIAG
- U1 pad 14: /MZ_EN -> /MY_DIR
- U1 pad 15: /MZ_DIAG -> /MY_STEP
- U1 pad 16: /M_UART -> /RGB_PIN
- U1 pad 17: /UART_RX -> /MS_DIAG
- U1 pad 18: GND -> +3V3
- U1 pad 19: /MZ_STEP -> GND
- U1 pad 2: /MX_DIAG -> /SGPIO_4
- U1 pad 20: /MZ_DIR -> unconnected-(U1-5V-Pad20)
- U1 pad 21: /S_GPIO16 -> /MX_EN
- U1 pad 22: /S_GPIO17 -> /MX_STEP
- U1 pad 23: GND -> /MX_DIR
- U1 pad 24: /S_GPIO18 -> /MX_DIAG
- U1 pad 25: /S_GPIO19 -> /MY_EN
- U1 pad 26: /ME_DIR -> /NEOPIXEL_PIN
- U1 pad 27: /S_GPIO21 -> /FAN0_PIN
- U1 pad 28: GND -> /PA11
- U1 pad 29: /ME_STEP -> /PA12
- U1 pad 3: GND -> /SGPIO_3
- U1 pad 30: unconnected-(U1-RUN-Pad30) -> /MY_DIAG
- U1 pad 31: /ME_DIAG -> /MZ_EN
- U1 pad 32: /ME_EN -> /MZ_STEP
- U1 pad 33: GND -> /MZ_DIR
- U1 pad 34: /S_GPIO28_ADC -> /HEATER_PIN
- U1 pad 35: unconnected-(U1-ADC_VREF-Pad35) -> /HEATED_BED_PIN
- U1 pad 36: +3V3 -> /MS_STEP
- U1 pad 37: unconnected-(U1-3V3_EN-Pad37) -> /MS_DIR
- U1 pad 38: GND -> unconnected-(U1-5V-Pad38)
- U1 pad 39: unconnected-(U1-VSYS-Pad39) -> GND
- U1 pad 4: /MX_STEP -> /BED_THM_2
- U1 pad 40: unconnected-(U1-VBUS-Pad40) -> +3V3
- U1 pad 5: /MX_DIR -> unconnected-(U1-nRST-Pad5)
- U1 pad 6: /S_GPIO4 -> /BED_THM_1
- U1 pad 7: /MY_EN -> /UART_RX
- U1 pad 8: GND -> /M_UART
- U1 pad 9: /MY_DIAG -> /SGPIO_5
Routing:
- net GND: track 10.4 -> 423.9 mm, vias 0 -> 1
- net +3V3: track 96.0 -> 265.1 mm, vias 0 -> 3
- net /M_UART: track 0.00 -> 156.8 mm, vias 0 -> 1
- net /MZ_DIR: track 0.00 -> 145.3 mm, vias 0 -> 5
- net /MX_DIR: track 0.00 -> 142.3 mm, vias 0 -> 2
- net /MX_DIAG: track 0.00 -> 133.4 mm, vias 0 -> 2
- net /MX_EN: track 0.00 -> 130.7 mm, vias 0 -> 2
- net +24V: track 0.00 -> 127.4 mm
- net /MX_STEP: track 0.00 -> 120.8 mm, vias 0 -> 1
- net /M_VBUS: track 110.9 -> 0.00 mm
- net /MZ_DIAG: track 0.00 -> 103.5 mm, vias 0 -> 2
- net /MY_DIAG: track 0.00 -> 100.5 mm, vias 0 -> 3
- net /MZ_STEP: track 0.00 -> 87.3 mm, vias 0 -> 3
- net /MZ_EN: track 0.00 -> 73.1 mm, vias 0 -> 1
- net /MY_STEP: track 0.00 -> 70.1 mm
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