File: A1_MB/DriverSlot.kicad_sch (KiCad schematic)
At the start: 6 parts, among them J4 Conn_01x03, J5 Conn_01x04, M1 TMC2209 Breakout

Commit message: e
e
Parts:
- C1: value 470uF -> 220uF; footprint OpenA1K:Cap ~ 12.5, 2.5mm-7.5mm pitch -> Capacitor_THT:CP_Radial_D8.0mm_P3.50mm
- J16: renamed from J; value Conn_01x02_Pin -> SensorlessHoming
- J17: renamed from J4; value Conn_01x03 -> Endstop
- renumbered J5 to MotorConnector1, R2 to R12
