File: KicadProjects/A1_MB/A1_MB.kicad_pcb (KiCad board)
At the start: 2 copper layers, 180 x 60 mm, 72 parts, among them J10 Screw_Terminal_01x02, J11 Bed Thermisters, J13 USB_A, J14 PA11J, J15 PA12J, J16 SensorlessHoming, J17 Endstop, J18 SensorlessHoming, J19 Endstop, J2 Neopixel, J20 Conn_01x04, J21 SensorlessHoming, J22 Endstop, J23 Conn_01x04, J24 SensorlessHoming, J25 Endstop, J26 Conn_01x04, J3 FAN0_VS, J4 RGB_2PIN, J5 Molex 2x02 Microfit, J6 HeatedBed, J7 FAN0, J8 SFS, J9 Hotend, M1 TMC2209 Breakout, M2 TMC2209 Breakout, M3 TMC2209 Breakout, M4 TMC2209 Breakout, Q10 2n7000, Q5 2n7000, Q6 NMOS, Q7 2n7000, Q8 NMOS, Q9 2n7000

Commit message: e
e
Parts:
- removed D1, D3, D4, D6: D, OpenA1K:Diode
- removed the J3 at (156.8, 37.0)
- removed J6: HeatedBed, Connector_JST:JST_XH_B2B-XH-AM_1x02_P2.50mm_Vertical
- removed the J9 at (202.0, 40.5)
- removed Q10, Q5, Q7, Q9: 2n7000, OpenA1K:2n7000
- removed Q6, Q8: NMOS, OpenA1K:IRLZ44N
- removed R10, R11: 10k, Resistor_THT:R_Axial_DIN0207_L6.3mm_D2.5mm_P10.16mm_Horizontal
- removed R16, R19, R20, R22: 10kΩ, Resistor_THT:R_Axial_DIN0207_L6.3mm_D2.5mm_P10.16mm_Horizontal
- removed R17, R18, R21, R23, R25, R27: 1kΩ, Resistor_THT:R_Axial_DIN0207_L6.3mm_D2.5mm_P10.16mm_Horizontal
- removed R24, R26: 0.1MΩ, Resistor_THT:R_Axial_DIN0207_L6.3mm_D2.5mm_P10.16mm_Horizontal
- added D9: D, OpenA1K:Diode, F.Cu at (224.1, 77.1)
- added J5: HotendConn, Connector_JST:JST_XH_B2B-XH-AM_1x02_P2.50mm_Vertical, F.Cu at (222.8, 62.1)
- added M5: ~, OpenA1K:MosfetModule, F.Cu at (176.0, 35.4)
- added M6: ~, OpenA1K:MosfetModule, F.Cu at (214.2, 70.5)
- added M7: ~, OpenA1K:MosfetModule, F.Cu at (159.3, 35.5)
- added R2: 4.7kΩ, Resistor_THT:R_Axial_DIN0207_L6.3mm_D2.5mm_P10.16mm_Horizontal, F.Cu at (270.9, 77.8)
- added R3: 4.7kΩ, Resistor_THT:R_Axial_DIN0207_L6.3mm_D2.5mm_P10.16mm_Horizontal, F.Cu at (270.9, 81.8)
- J4: value RGB_2PIN -> HeatedBedConn
- J7: value FAN0 -> FanConn; footprint Connector_JST:JST_XH_B3B-XH-AM_1x03_P2.50mm_Vertical -> Connector_JST:JST_XH_B2B-XH-AM_1x02_P2.50mm_Vertical
- J8: value SFS -> SmFilSns
- moved J7 107.8 mm to (263.4, 94.7), turned to 0 degrees
- moved J4 93.2 mm to (263.4, 79.1), turned to 0 degrees
- moved D2 67.0 mm to (233.2, 70.2), turned to 0 degrees
- moved D5 46.0 mm to (233.2, 76.1), turned to 0 degrees
- moved J1 4.49 mm to (204.9, 75.1)
- moved C7 2.96 mm to (153.6, 70.7)
- renumbered C5 to C1, C1 to C4, C2 to C5, C3 to C6, C4 to C7, J5 to J1, J13 to J10, J16 to J12, J17 to J13, J18 to J14, J19 to J15, J20 to J16, J21 to J17, J22 to J18, J23 to J19, J24 to J20, J25 to J21, J26 to J22, J2 to J3, J10 to J9, R9 to R1, R12 to R4, R13 to R5, R14 to R6, R15 to R7
Connections:
- D2 pad 1: GND -> +24V
- D2 pad 2: 5V -> /Mosfet2/Output_Return
- D5 pad 1: GND -> +24V
- D5 pad 2: +24V -> /Mosfet1/Output_Return
- J1 pad 3: /Mosfet/Output_Return -> /Mosfet2/Output_Return
- J10 pad 2: /D- -> unconnected-(J10-D--Pad2)
- J10 pad 3: /D+ -> unconnected-(J10-D+-Pad3)
- J11 pad 1: +3V3 -> GNDA
- J11 pad 2: /BED_THM_2 -> /BED_THM_1
- J11 pad 3: +3V3 -> GNDA
- J11 pad 4: /BED_THM_1 -> /BED_THM_2
- J4 pad 1: 5V -> +24V
- J4 pad 2: /Transistor1/Output_GND -> /Mosfet1/Output_Return
- J7 pad 1: Net-(J3-Pin_2) -> +24V
- J7 pad 2: GND -> /Mosfet3/Output_Return
- M1 pad 2: GND -> GNDA
- M1 pad 3: GND -> GNDA
- M2 pad 3: GND -> GNDA
- M3 pad 2: GND -> GNDA
Routing:
- net (no net): track 0.00 -> 84.0 mm
- net /Mosfet2/Output_Return: track 0.00 -> 42.6 mm, vias 0 -> 1
- net /Mosfet/Output_Return: track 42.6 -> 0.00 mm, vias 1 -> 0
- net 5V: track 29.3 -> 0.00 mm
- net Net-(J3-Pin_2): track 13.4 -> 0.00 mm
- net /Transistor1/Output_GND: track 7.65 -> 0.00 mm
- net Net-(Q6-G): track 5.48 -> 0.00 mm
- net Net-(Q8-G): track 5.40 -> 0.00 mm
- net Net-(Q7-G): track 3.69 -> 0.00 mm
- net Net-(Q5-G): track 3.67 -> 0.00 mm
- net Net-(Q10-G): track 3.21 -> 0.00 mm
- net /FAN0_PIN: track 3.20 -> 0.00 mm
- net /HEATER_PIN: track 3.00 -> 0.00 mm
- net / HEATED_BED_PIN: track 3.00 -> 0.00 mm
- net Net-(Q9-G): track 3.00 -> 0.00 mm
