File: KicadProjects/A1_MB/A1_MB.kicad_sch (KiCad schematic)
At the start: 26 parts, among them J1 Conn_02x04_Counter_Clockwise, J10 Screw_Terminal_01x02, J11 Bed Thermisters, J12 SpareGPIO, J13 USB_A, J14 PA11J, J15 PA12J, J2 Neopixel, J3 FAN0_VS, J4 RGB_2PIN, J5 Molex 2x02 Microfit, J6 HeatedBed, J7 FAN0, J8 SFS, J9 Hotend

Commit message: e
e
Parts:
- removed J12: SpareGPIO, Connector_PinHeader_2.54mm:PinHeader_2x05_P2.54mm_Vertical, symbol Connector_Generic:Conn_02x05_Counter_Clockwise
- removed J14: PA11J, Connector_PinHeader_2.54mm:PinHeader_1x02_P2.54mm_Vertical, symbol Connector:Conn_01x02_Pin
- removed J15: PA12J, Connector_PinHeader_2.54mm:PinHeader_1x02_P2.54mm_Vertical, symbol Connector:Conn_01x02_Pin
- removed J3: FAN0_VS, Connector_PinHeader_2.54mm:PinHeader_1x03_P2.54mm_Vertical, symbol Connector:Conn_01x03_Pin
- removed J7: FAN0, Connector_JST:JST_XH_B3B-XH-AM_1x03_P2.50mm_Vertical, symbol Connector_Generic:Conn_01x03
- removed J9: Hotend, Connector_JST:JST_XH_B2B-XH-AM_1x02_P2.50mm_Vertical, symbol Connector:Screw_Terminal_01x02
- removed R10, R11: 10k, Resistor_THT:R_Axial_DIN0207_L6.3mm_D2.5mm_P10.16mm_Horizontal, symbol Device:R
- added C2, C3: 100nF, symbol Device:C
- added J5: HotendConn, Connector_JST:JST_XH_B2B-XH-AM_1x02_P2.50mm_Vertical, symbol Connector:Screw_Terminal_01x02
- added J7: FanConn, Connector_JST:JST_XH_B2B-XH-AM_1x02_P2.50mm_Vertical, symbol Connector:Screw_Terminal_01x02
- added R2, R3: 4.7kΩ, Resistor_THT:R_Axial_DIN0207_L6.3mm_D2.5mm_P10.16mm_Horizontal, symbol Device:R
- J4: renamed from J6; value HeatedBed -> HeatedBedConn
- J6: renamed from J4; now not fitted; now left out of the parts list
- J8: value SFS -> SmFilSns
- renumbered C5 to C1, J5 to J1, J13 to J10, J1 to J2, J2 to J3, J10 to J9, R9 to R1
Connections:
- net +3V3: now also R2.1, R3.1; no longer J11.1 (Pin_1), J11.3 (Pin_3)
- net BED_THM_1: now also J11.2 (Pin_2), C2.1, R2.2; no longer J11.4 (Pin_4)
- net BED_THM_2: now also J11.4 (Pin_4), C3.1, R3.2; no longer J11.2 (Pin_2)
- net D+: no longer names the net of J10.3 (D+)
- net D-: no longer names the net of J10.2 (D-)
- net Mosfet/Output_24V renamed Mosfet2/Output_24V
- net Mosfet2/Output_24V: now also J5.1 (Pin_1)
- net Mosfet/Output_Return renamed Mosfet2/Output_Return
- net Mosfet2/Output_Return: now also J5.2 (Pin_2)
- new net GNDA: C2.2, C3.2, J11.1 (Pin_1), J11.3 (Pin_3)
- new net Mosfet3/Output_24V: J7.1 (Pin_1)
- new net Mosfet3/Output_Return: J7.2 (Pin_2)
Other:
- removed sheet Mosfet
- removed sheet Transistor
- added sheet Mosfet2 (mosfet.kicad_sch)
- added sheet Mosfet3 (mosfet.kicad_sch)
- sheet Mosfet1 ports: added GND, Signal GND, VIN; removed none
- note removed: "Connectors"
- moved on the sheet: J1, J11, J4
