File: KicadProjects/A1_MB/DriverSlot.kicad_sch (KiCad schematic)
At the start: 6 parts, among them J16 SensorlessHoming, J17 Endstop, M1 TMC2209 Breakout

Commit message: e
e
Parts:
- renumbered C1 to C4, J16 to J12, J17 to J13, R12 to R4
