File: KicadProjects/A1_MB/Transistor.kicad_sch (KiCad schematic)
At the start: 4 parts, among them Q9 2n7000

Commit message: e
e
Parts:
- renumbered D1 to D7, Q9 to Q5, R24 to R16, R25 to R17
Changed lines of the file:
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@@
 		(dnp no)
 		(fields_autoplaced yes)
-		(property "Reference" "R24"
+		(property "Reference" "R16"
 			(at 135.89 105.4099 0)
 			(effects
@@
 		(instances
 			(project "A1_MB"
-				(path "/989d6d42-19bd-451f-8ed3-d8ee079df240/949f0074-f658-4572-9b27-0f650e94e32f"
-					(reference "R24")
-					(unit 1)
-				)
-				(path "/989d6d42-19bd-451f-8ed3-d8ee079df240/d0bcb683-06b6-4f24-ad94-39c20cda3fb0"
-					(reference "R26")
+				(path "/989d6d42-19bd-451f-8ed3-d8ee079df240/d0bcb683-06b6-4f24-ad94-39c20cda3fb0"
+					(reference "R16")
 					(unit 1)
 				)
@@
 		(on_board yes)
 		(dnp no)
-		(property "Reference" "#PWR082"
+		(property "Reference" "#PWR081"
 			(at 152.4 119.38 0)
 			(effects
@@
 		(instances
 			(project "A1_MB"
-				(path "/989d6d42-19bd-451f-8ed3-d8ee079df240/949f0074-f658-4572-9b27-0f650e94e32f"
-					(reference "#PWR082")
-					(unit 1)
-				)
-				(path "/989d6d42-19bd-451f-8ed3-d8ee079df240/d0bcb683-06b6-4f24-ad94-39c20cda3fb0"
-					(reference "#PWR084")
+				(path "/989d6d42-19bd-451f-8ed3-d8ee079df240/d0bcb683-06b6-4f24-ad94-39c20cda3fb0"
+					(reference "#PWR081")
 					(unit 1)
 				)
@@
 		(on_board yes)
 		(dnp no)
-		(property "Reference" "R25"
+		(property "Reference" "R17"
 			(at 139.446 96.774 90)
 			(effects
@@
 		(instances
 			(project "A1_MB"
-				(path "/989d6d42-19bd-451f-8ed3-d8ee079df240/949f0074-f658-4572-9b27-0f650e94e32f"
-					(reference "R25")
-					(unit 1)
-				)
-				(path "/989d6d42-19bd-451f-8ed3-d8ee079df240/d0bcb683-06b6-4f24-ad94-39c20cda3fb0"
-					(reference "R27")
+				(path "/989d6d42-19bd-451f-8ed3-d8ee079df240/d0bcb683-06b6-4f24-ad94-39c20cda3fb0"
+					(reference "R17")
 					(unit 1)
 				)
@@
 		(dnp no)
 		(fields_autoplaced yes)
-		(property "Reference" "D1"
+		(property "Reference" "D7"
 			(at 135.89 80.01 0)
 			(effects
@@
 		(instances
 			(project ""
-				(path "/989d6d42-19bd-451f-8ed3-d8ee079df240/949f0074-f658-4572-9b27-0f650e94e32f"
-					(reference "D1")
-					(unit 1)
-				)
-				(path "/989d6d42-19bd-451f-8ed3-d8ee079df240/d0bcb683-06b6-4f24-ad94-39c20cda3fb0"
-					(reference "D2")
+				(path "/989d6d42-19bd-451f-8ed3-d8ee079df240/d0bcb683-06b6-4f24-ad94-39c20cda3fb0"
+					(reference "D7")
 					(unit 1)
 				)
@@
 		(dnp no)
 		(fields_autoplaced yes)
-		(property "Reference" "#PWR07"
+		(property "Reference" "#PWR079"
 			(at 132.08 92.71 0)
 			(effects
@@
 		(instances
 			(project ""
-				(path "/989d6d42-19bd-451f-8ed3-d8ee079df240/949f0074-f658-4572-9b27-0f650e94e32f"
-					(reference "#PWR07")
-					(unit 1)
-				)
-				(path "/989d6d42-19bd-451f-8ed3-d8ee079df240/d0bcb683-06b6-4f24-ad94-39c20cda3fb0"
-					(reference "#PWR08")
+				(path "/989d6d42-19bd-451f-8ed3-d8ee079df240/d0bcb683-06b6-4f24-ad94-39c20cda3fb0"
+					(reference "#PWR079")
 					(unit 1)
 				)
@@
 		(on_board yes)
 		(dnp no)
-		(property "Reference" "#PWR081"
+		(property "Reference" "#PWR080"
 			(at 152.4 96.52 0)
 			(effects
@@
 		(instances
 			(project "A1_MB"
-				(path "/989d6d42-19bd-451f-8ed3-d8ee079df240/949f0074-f658-4572-9b27-0f650e94e32f"
-					(reference "#PWR081")
-					(unit 1)
-				)
-				(path "/989d6d42-19bd-451f-8ed3-d8ee079df240/d0bcb683-06b6-4f24-ad94-39c20cda3fb0"
-					(reference "#PWR083")
+				(path "/989d6d42-19bd-451f-8ed3-d8ee079df240/d0bcb683-06b6-4f24-ad94-39c20cda3fb0"
+					(reference "#PWR080")
 					(unit 1)
 				)
@@
 		(dnp no)
 		(fields_autoplaced yes)
-		(property "Reference" "Q9"
+		(property "Reference" "Q5"
 			(at 156.21 101.5999 0)
 			(effects
@@
 		(instances
 			(project "A1_MB"
-				(path "/989d6d42-19bd-451f-8ed3-d8ee079df240/949f0074-f658-4572-9b27-0f650e94e32f"
-					(reference "Q9")
-					(unit 1)
-				)
-				(path "/989d6d42-19bd-451f-8ed3-d8ee079df240/d0bcb683-06b6-4f24-ad94-39c20cda3fb0"
-					(reference "Q10")
-					(unit 1)
-				)
+				(path "/989d6d42-19bd-451f-8ed3-d8ee079df240/d0bcb683-06b6-4f24-ad94-39c20cda3fb0"
+					(reference "Q5")
+					(unit 1)
+				)
