File: KicadProjects/A1_MB/mosfet.kicad_sch (KiCad schematic)
At the start: 8 parts, among them Q5 2n7000, Q6 NMOS

Commit message: e
e
Parts:
- added D2: D, OpenA1K:Diode, symbol Device:D
- added M5: ~, OpenA1K:MosfetModule, symbol OpenA1KSymbols:MOSFET-MODULE
- D1: renamed from D3; now not fitted; now left out of the parts list
- D3: renamed from D4; now not fitted; now left out of the parts list
- Q1: renamed from Q5; now not fitted; now left out of the parts list
- Q2: renamed from Q6; now not fitted; now left out of the parts list
- R10: renamed from R19; now not fitted; now left out of the parts list
- R11: renamed from R18; now not fitted; now left out of the parts list
- R8: renamed from R16; now not fitted; now left out of the parts list
- R9: renamed from R17; now not fitted; now left out of the parts list
Connections:
- net +24V: now also D2.1 (K), M5. (GND)
- net GND: now also M5. (GND)
- net Output_Return: now also D2.2 (A), M5. (GND)
- net Signal 3V3: now also M5. (GND)
- new net Signal GND: M5. (GND)
Other:
- note added: "OLD"
