File: KicadProjects/A1_SMD_MB/A1_MB_V2/A1_MB_V2.kicad_pcb (KiCad board)
At the start: 2 copper layers, 92 parts, among them J6 THB2, J7 HE, J8 HE, J9 THB1, U1 STM32F407VGTx, U2 AMS1117-3.3, U3 TMC2209-LA, U4 TMC2209-LA, U5 TMC2209-LA, U6 TMC2209-LA

Commit message: e
e
Parts:
- removed U1: STM32F407VGTx, Package_QFP:LQFP-100_14x14mm_P0.5mm
- removed U2: AMS1117-3.3, Package_TO_SOT_SMD:SOT-223-3_TabPin2
- added C15: 15pF, Capacitor_SMD:C_0402_1005Metric, F.Cu at (92.0, 57.2)
- added C16: 15pF, Capacitor_SMD:C_0402_1005Metric, F.Cu at (92.1, 52.8)
- added C17: 10uF, Capacitor_SMD:C_0805_2012Metric, F.Cu at (108.6, 67.7)
- added C18: 10uF, Capacitor_SMD:C_0805_2012Metric, F.Cu at (104.0, 62.0)
- added C19: 10uF, Capacitor_SMD:C_0805_2012Metric, F.Cu at (104.0, 49.0)
- added C20: 10uF, Capacitor_SMD:C_0805_2012Metric, F.Cu at (118.2, 67.8)
- added C51: 100nF, Capacitor_SMD:C_0402_1005Metric, F.Cu at (98.0, 56.0)
- added C52: 100nF, Capacitor_SMD:C_0402_1005Metric, F.Cu at (108.4, 54.8)
- added C53: 1uF, Capacitor_SMD:C_0603_1608Metric, F.Cu at (109.0, 56.9)
- added C54: 1uF, Capacitor_SMD:C_0603_1608Metric, F.Cu at (109.0, 58.4)
- added C55: 100nF, Capacitor_SMD:C_0402_1005Metric, F.Cu at (108.5, 59.6)
- added C56: 100nF, Capacitor_SMD:C_0402_1005Metric, F.Cu at (105.8, 60.6)
- added C57: 100nF, Capacitor_SMD:C_0402_1005Metric, F.Cu at (102.2, 60.6)
- added C58: 100nF, Capacitor_SMD:C_0402_1005Metric, F.Cu at (108.4, 55.7)
- added C59: 100nF, Capacitor_SMD:C_0402_1005Metric, F.Cu at (105.8, 50.1)
- added C60: 100nF, Capacitor_SMD:C_0402_1005Metric, F.Cu at (102.2, 50.1)
- added C61: 100nF, Capacitor_SMD:C_0402_1005Metric, F.Cu at (98.0, 54.4)
- added C62: 100nF, Capacitor_SMD:C_0402_1005Metric, F.Cu at (117.3, 54.1)
- added D4: D, Diode_SMD:D_SMA, F.Cu at (157.0, 39.0)
- added D7: D, Diode_SMD:D_SMA, F.Cu at (143.5, 39.0)
- added J10: BedTherms, Connector_JST:JST_XH_B4B-XH-A_1x04_P2.50mm_Vertical, F.Cu at (96.8, 85.0)
- added J11: SWD, Connector_PinHeader_1.27mm:PinHeader_1x04_P1.27mm_Vertical, F.Cu at (97.0, 45.6)
- added J12: Conn_01x02_Pin, Connector_PinHeader_2.54mm:PinHeader_1x02_P2.54mm_Vertical, F.Cu at (116.6, 38.7)
- added J13: THM2JMP, Connector_PinHeader_2.54mm:PinHeader_1x02_P2.54mm_Vertical, F.Cu at (151.2, 79.8)
- added J14: THM1JMP, Connector_PinHeader_2.54mm:PinHeader_1x02_P2.54mm_Vertical, F.Cu at (148.5, 79.8)
- added J15: Sensorless, Connector_PinHeader_2.54mm:PinHeader_1x02_P2.54mm_Vertical, F.Cu at (45.0, 55.5)
- added J16: Sensorless, Connector_PinHeader_2.54mm:PinHeader_1x02_P2.54mm_Vertical, F.Cu at (70.5, 56.5)
- added J17: Sensorless, Connector_PinHeader_2.54mm:PinHeader_1x02_P2.54mm_Vertical, F.Cu at (67.5, 64.5)
- added J18: Sensorless, Connector_PinHeader_2.54mm:PinHeader_1x02_P2.54mm_Vertical, F.Cu at (42.5, 65.5)
- added J19: Endstop, Connector_JST:JST_XH_B3B-XH-A_1x03_P2.50mm_Vertical, F.Cu at (53.0, 46.1)
- added J20: Endstop, Connector_JST:JST_XH_B3B-XH-A_1x03_P2.50mm_Vertical, F.Cu at (78.0, 45.5)
- added J21: Endstop, Connector_JST:JST_XH_B3B-XH-A_1x03_P2.50mm_Vertical, F.Cu at (61.5, 71.0)
- added J22: Endstop, Connector_JST:JST_XH_B3B-XH-A_1x03_P2.50mm_Vertical, F.Cu at (35.5, 71.0)
- added J23: PWR, OpenA1K:1x2 Terminal Block, F.Cu at (119.9, 83.1)
- added J24: FAN1, Connector_JST:JST_XH_B4B-XH-A_1x04_P2.50mm_Vertical, F.Cu at (144.0, 34.0)
- added J25: SPR_IO, Connector_PinHeader_2.54mm:PinHeader_1x03_P2.54mm_Vertical, F.Cu at (106.0, 30.9)
- added J3: FPC2, Connector_PinHeader_2.54mm:PinHeader_1x08_P2.54mm_Vertical, F.Cu at (166.5, 83.6)
- added J4: FPC1, Connector_PinHeader_2.54mm:PinHeader_1x08_P2.54mm_Vertical, F.Cu at (166.5, 87.6)
- added P1: MCUTOPI, Connector_USB:USB_C_Receptacle_HCTL_HC-TYPE-C-16P-01A, F.Cu at (174.9, 51.5)
- added P2: THBINPUT, Connector_USB:USB_C_Receptacle_HCTL_HC-TYPE-C-16P-01A, F.Cu at (174.9, 62.1)
- added P3: THBTOPI, Connector_USB:USB_C_Receptacle_HCTL_HC-TYPE-C-16P-01A, F.Cu at (174.9, 72.8)
- added Q1: NMOS, Package_TO_SOT_SMD:SOT-23-3, F.Cu at (104.5, 79.5)
- added Q2: NMOS, Package_TO_SOT_SMD:SOT-23-3, F.Cu at (112.6, 79.5)
- added R4: 27.4o, Resistor_SMD:R_0402_1005Metric, F.Cu at (168.5, 52.0)
- added R5: 1k, Resistor_SMD:R_0603_1608Metric, F.Cu at (90.2, 58.2)
- added R56: 10k, Resistor_SMD:R_0402_1005Metric, F.Cu at (96.0, 60.0)
- added R57: 100R, Resistor_SMD:R_0402_1005Metric, F.Cu at (152.5, 40.0)
- added R58: 20kR, Resistor_SMD:R_0402_1005Metric, F.Cu at (150.0, 38.0)
- added R59: 100R, Resistor_SMD:R_0402_1005Metric, F.Cu at (152.5, 38.0)
- added R6: 27.4o, Resistor_SMD:R_0402_1005Metric, F.Cu at (168.5, 51.0)
- added R62: 100R, Resistor_SMD:R_0402_1005Metric, F.Cu at (139.0, 40.0)
- added R63: 100R, Resistor_SMD:R_0402_1005Metric, F.Cu at (139.0, 38.0)
- added R64: 20kR, Resistor_SMD:R_0402_1005Metric, F.Cu at (136.5, 38.0)
- added R7: 1ko, Resistor_SMD:R_0603_1608Metric, F.Cu at (117.3, 42.1)
- added U7: NCP1117-1.5_SOT223, Package_TO_SOT_SMD:SOT-223-3_TabPin2, F.Cu at (113.5, 67.5)
- added U8: RP2040, Package_DFN_QFN:QFN-56-1EP_7x7mm_P0.4mm_EP3.2x3.2mm, F.Cu at (103.2, 55.4)
- added U9: W25Q128JVS, Package_SO:SOIC-8_5.3x5.3mm_P1.27mm, F.Cu at (115.5, 48.5)
- added Y2: ABM8-272-T3, Crystal:Crystal_SMD_Abracon_ABM8AIG-4Pin_3.2x2.5mm, F.Cu at (92.0, 55.0)
- J6: value THB2 -> FAN0; footprint Connector_JST:JST_XH_B2B-XH-A_1x02_P2.50mm_Vertical -> Connector_JST:JST_XH_B4B-XH-A_1x04_P2.50mm_Vertical
- J7: footprint Connector_JST:JST_XH_B2B-XH-A_1x02_P2.50mm_Vertical -> OpenA1K:ScrewTerminal 7mm x 7mm
- J8: value HE -> HB; footprint Connector_JST:JST_XH_B2B-XH-A_1x02_P2.50mm_Vertical -> OpenA1K:ScrewTerminal 7mm x 7mm
- J9: value THB1 -> Conn_01x03_Pin; footprint Connector_JST:JST_XH_B2B-XH-A_1x02_P2.50mm_Vertical -> Connector_PinHeader_2.54mm:PinHeader_1x03_P2.54mm_Vertical
- moved U3 106.5 mm to (39.8, 47.9)
- moved U4 89.5 mm to (65.3, 48.6)
- moved U6 83.7 mm to (47.5, 72.8), turned to 180 degrees
- moved R9 80.5 mm to (36.6, 43.0), turned to 180 degrees
- moved U5 76.7 mm to (72.7, 72.5), turned to 180 degrees
- moved C27 75.8 mm to (35.1, 45.5)
- moved R8 73.5 mm to (42.8, 43.2)
- moved R34 72.4 mm to (34.0, 47.8)
- moved C24 71.2 mm to (35.1, 50.3)
- moved J6 70.3 mm to (157.5, 34.0), turned to 180 degrees
- moved EXM2 70.2 mm to (36.0, 37.0)
- moved C38 70.1 mm to (60.1, 84.3), turned to 180 degrees
- moved R12 70.0 mm to (34.0, 46.8)
- moved C21 69.4 mm to (35.8, 48.0), turned to 90 degrees
- moved C25 69.2 mm to (52.5, 37.0)
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Connections:
- net /mosfets/HB_SIG renamed /mcu/G2
- net /mosfets/THB1 renamed /fpc/THM1
- net /mosfets/THB2 renamed /fpc/THM2
- C22 pad 2: 3V3 -> +3V3
- C34 pad 2: 3V3 -> +3V3
- C41 pad 2: 3V3 -> +3V3
- C48 pad 2: 3V3 -> +3V3
- J6 pad 1: Net-(J6-Pin_1) -> +24V
- J9 pad 1: Net-(J9-Pin_1) -> +3V3
- J9 pad 2: GND -> Net-(J9-Pin_2)
- R28 pad 1: /mosfets/HE_SIG -> /mcu/G3
- R28 pad 2: /mosfets/HE_SIG -> /stuff/HE_S
- R29 pad 1: /mosfets/HE_SIG -> /mcu/G3
- R31 pad 2: /mosfets/HE_SIG -> /stuff/HB_S
- R35 pad 1: Net-(U3-DIAG) -> Net-(J15-Pin_1)
- R39 pad 1: Net-(U4-DIAG) -> Net-(J16-Pin_1)
- R43 pad 1: Net-(U5-DIAG) -> Net-(J17-Pin_1)
- R47 pad 1: Net-(U6-DIAG) -> Net-(J18-Pin_1)
- R50 pad 2: Net-(J6-Pin_1) -> Net-(J10-Pin_1)
- R51 pad 1: Net-(J6-Pin_1) -> Net-(J10-Pin_1)
- R53 pad 2: Net-(J9-Pin_1) -> Net-(J10-Pin_3)
- R54 pad 1: Net-(J9-Pin_1) -> Net-(J10-Pin_3)
- U3 pad 11: Net-(U3-DIAG) -> Net-(J15-Pin_2)
- U3 pad 15: 3V3 -> +3V3
- U4 pad 11: Net-(U4-DIAG) -> Net-(J16-Pin_2)
- U4 pad 15: 3V3 -> +3V3
- U5 pad 11: Net-(U5-DIAG) -> Net-(J17-Pin_2)
- U5 pad 15: 3V3 -> +3V3
- U6 pad 11: Net-(U6-DIAG) -> Net-(J18-Pin_2)
- U6 pad 15: 3V3 -> +3V3
Other:
- board outline added: 150 x 60 mm
- board text added: "S Motor"
- board text added: "X Motor"
- board text added: "Y Motor"
- board text added: "Z Motor"
