File: KicadProjects/A1_SMD_MB/A1_MB_V2/A1_MB_V2.kicad_sch (KiCad schematic)
At the start: 0 parts

Commit message: e
e
Other:
- added sheet fpc (fpc.kicad_sch)
- added sheet mosfets (mosfets.kicad_sch)
- sheet Motors ports: added UART; removed none
Changed lines of the file:
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@@
+	)
+	(sheet
+		(at 48.895 86.995)
+		(size 26.67 15.24)
+		(exclude_from_sim no)
+		(in_bom yes)
+		(on_board yes)
+		(dnp no)
+		(fields_autoplaced yes)
+		(stroke
+			(width 0.1524)
+			(type solid)
+		)
+		(fill
+			(color 0 0 0 0.0000)
+		)
+		(property "Sheetname" "mosfets"
+			(at 48.895 86.2834 0)
+			(effects
+				(font
+					(size 1.27 1.27)
+				)
+				(justify left bottom)
+			)
+		)
+		(property "Sheetfile" "mosfets.kicad_sch"
+			(at 48.895 102.8196 0)
+			(effects
+				(font
+					(size 1.27 1.27)
+				)
+				(justify left top)
+			)
+		)
+		(pin "HE_SIG" input
+			(at 75.565 100.33 0)
+			(effects
+				(font
+					(size 1.27 1.27)
+				)
+				(justify right)
+			)
+		)
+		(pin "HB_SIG" input
+			(at 75.565 97.79 0)
+			(effects
+				(font
+					(size 1.27 1.27)
+				)
+				(justify right)
+			)
+		)
+		(instances
+			(project "A1_MB_V2"
+				(path "/a288b6e0-7c74-4cd9-8c53-d587802da1e5"
+					(page "9")
+				)
+			)
+		)
+	)
+	(sheet
+		(at 48.895 106.68)
+		(size 26.67 10.16)
+		(exclude_from_sim no)
+		(in_bom yes)
+		(on_board yes)
+		(dnp no)
+		(fields_autoplaced yes)
+		(stroke
+			(width 0.1524)
+			(type solid)
+		)
+		(fill
+			(color 0 0 0 0.0000)
+		)
+		(property "Sheetname" "fpc"
+			(at 48.895 105.9684 0)
+			(effects
+				(font
+					(size 1.27 1.27)
+				)
+				(justify left bottom)
+			)
+		)
+		(property "Sheetfile" "fpc.kicad_sch"
+			(at 48.895 117.4246 0)
+			(effects
+				(font
+					(size 1.27 1.27)
+				)
+				(justify left top)
+			)
+		)
+		(pin "THM2" input
+			(at 75.565 114.3 0)
+			(effects
+				(font
+					(size 1.27 1.27)
+				)
+				(justify right)
+			)
+		)
+		(pin "THM1" input
+			(at 75.565 111.76 0)
+			(effects
+				(font
+					(size 1.27 1.27)
+				)
+				(justify right)
+			)
+		)
+		(pin "HB_CT" input
+			(at 75.565 109.22 0)
+			(effects
+				(font
+					(size 1.27 1.27)
+				)
+				(justify right)
+			)
+		)
+		(instances
+			(project "A1_MB_V2"
+				(path "/a288b6e0-7c74-4cd9-8c53-d587802da1e5"
+					(page "8")
+				)
+			)
+		)
 	)
 	(sheet
@@
 	)
 	(sheet
-		(at 48.26 130.81)
-		(size 26.67 46.99)
+		(at 48.26 122.555)
+		(size 26.67 55.245)
 		(exclude_from_sim no)
 		(in_bom yes)
@@
 		)
 		(property "Sheetname" "Motors"
-			(at 48.26 130.0984 0)
+			(at 48.26 121.8434 0)
 			(effects
 				(font
@@
 			(effects
 				(font
+					(size 1.27 1.27)
+				)
+				(justify right)
+			)
+		)
+		(pin "UART" input
+			(at 74.93 129.54 0)
+			(effects
+				(font

Commit message: e
e
Parts:
- added R61: 1k, symbol Device:R
Connections:
- net Motors/UART: now also R61.1
- new net mcu/G5: R61.2
Other:
- sheet mosfets renamed stuff
- added sheet mcu (mcu.kicad_sch)
- added sheet power (power.kicad_sch)
- added sheet spare (spare.kicad_sch)
- added sheet usbc (usbc.kicad_sch)
- sheet stuff ports: added FAN0_PWM, FAN0_TACH, FAN1_PWM, FAN1_TACH, THB1, THB2; removed none
- note added: "STM32 CHIP, NOT IN USE"
