File: KicadProjects/A1_SMD_MB/A1_MB_V2/motors.kicad_sch (KiCad schematic)
At the start: 0 parts

Commit message: e
e
Other:
- added sheet motor (motor.kicad_sch)
- added sheet motor1 (motor.kicad_sch)
- added sheet motor2 (motor.kicad_sch)
- added sheet motor3 (motor.kicad_sch)
- note added: "SMOTOR"
- note added: "XMOTOR"
- note added: "YMOTOR"
- note added: "ZMOTOR"

Commit message: e
e
Changed lines of the file:
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@@
 	(text "XMOTOR"
 		(exclude_from_sim no)
-		(at 50.165 43.688 0)
+		(at 50.8 42.418 0)
 		(effects
 			(font
@@
 	(wire
 		(pts
-			(xy 55.88 55.88) (xy 58.42 55.88)
+			(xy 56.515 54.61) (xy 59.055 54.61)
 		)
 		(stroke
@@
 	(wire
 		(pts
-			(xy 55.88 53.34) (xy 62.23 53.34)
+			(xy 56.515 52.07) (xy 62.865 52.07)
 		)
 		(stroke
@@
 	(hierarchical_label "UART"
 		(shape input)
-		(at 55.88 50.8 0)
+		(at 56.515 49.53 0)
 		(effects
 			(font
@@
 	(hierarchical_label "MX_DIR"
 		(shape input)
-		(at 42.545 55.88 180)
+		(at 43.18 54.61 180)
 		(effects
 			(font
@@
 	(hierarchical_label "MX_EN"
 		(shape input)
-		(at 42.545 50.8 180)
+		(at 43.18 49.53 180)
 		(effects
 			(font
@@
 	(hierarchical_label "MX_STEP"
 		(shape input)
-		(at 42.545 53.34 180)
+		(at 43.18 52.07 180)
 		(effects
 			(font
@@
 	(hierarchical_label "MX_DIAG"
 		(shape input)
-		(at 42.545 58.42 180)
+		(at 43.18 57.15 180)
 		(effects
 			(font
@@
 	(symbol
 		(lib_id "power:GND")
-		(at 58.42 55.88 0)
+		(at 59.055 54.61 0)
 		(unit 1)
 		(exclude_from_sim no)
@@
 		(fields_autoplaced yes)
 		(property "Reference" "#PWR019"
-			(at 58.42 62.23 0)
+			(at 59.055 60.96 0)
 			(effects
 				(font
@@
 		)
 		(property "Value" "GND"
-			(at 58.42 60.96 0)
+			(at 59.055 59.69 0)
 			(effects
 				(font
@@
 		)
 		(property "Footprint" ""
-			(at 58.42 55.88 0)
+			(at 59.055 54.61 0)
 			(effects
 				(font
@@
 		)
 		(property "Datasheet" ""
-			(at 58.42 55.88 0)
+			(at 59.055 54.61 0)
 			(effects
 				(font
@@
 		)
 		(property "Description" "Power symbol creates a global label with name \"GND\" , ground"
-			(at 58.42 55.88 0)
+			(at 59.055 54.61 0)
 			(effects
 				(font
@@
 	(symbol
 		(lib_id "power:GND")
-		(at 62.23 53.34 0)
+		(at 62.865 52.07 0)
 		(unit 1)
 		(exclude_from_sim no)
@@
 		(fields_autoplaced yes)
 		(property "Reference" "#PWR020"
-			(at 62.23 59.69 0)
+			(at 62.865 58.42 0)
 			(effects
 				(font
@@
 		)
 		(property "Value" "GND"
-			(at 62.23 58.42 0)
+			(at 62.865 57.15 0)
 			(effects
 				(font
@@
 		)
 		(property "Footprint" ""
-			(at 62.23 53.34 0)
+			(at 62.865 52.07 0)
 			(effects
 				(font
@@
 		)
 		(property "Datasheet" ""
-			(at 62.23 53.34 0)
+			(at 62.865 52.07 0)
 			(effects
 				(font
@@
 		)
 		(property "Description" "Power symbol creates a global label with name \"GND\" , ground"
-			(at 62.23 53.34 0)
+			(at 62.865 52.07 0)
 			(effects
 				(font
@@
 	)
 	(sheet
-		(at 42.545 48.26)
+		(at 43.18 46.99)
 		(size 13.335 12.7)
 		(exclude_from_sim no)
@@
 		)
 		(property "Sheetname" "motor"
-			(at 42.545 47.5484 0)
+			(at 43.18 46.2784 0)
 			(effects
 				(font
@@
 		)
 		(property "Sheetfile" "motor.kicad_sch"
-			(at 41.656 63.754 0)
+			(at 42.291 62.484 0)
 			(effects
 				(font
@@
 		)
 		(pin "DIAG" input
-			(at 42.545 58.42 180)
+			(at 43.18 57.15 180)
 			(effects
 				(font
@@
 		)
 		(pin "UART" input
-			(at 55.88 50.8 0)
+			(at 56.515 49.53 0)
 			(effects
 				(font
@@
 		)
 		(pin "STEP" input
-			(at 42.545 53.34 180)
+			(at 43.18 52.07 180)
 			(effects
 				(font
@@
 		)
 		(pin "DIR" input
-			(at 42.545 55.88 180)
+			(at 43.18 54.61 180)
 			(effects
 				(font
@@
 		)
 		(pin "EN" input
-			(at 42.545 50.8 180)
+			(at 43.18 49.53 180)
 			(effects
 				(font
@@
 		)
 		(pin "MS1" input
-			(at 55.88 53.34 0)
+			(at 56.515 52.07 0)
 			(effects
 				(font
@@
 		)
 		(pin "MS2" input
-			(at 55.88 55.88 0)
-			(effects
-				(font
+			(at 56.515 54.61 0)
+			(effects
+				(font
