File: KicadProjects/A1_SMD_MB/A1_MB_V2/stm32.kicad_sch (KiCad schematic)
At the start: 25 parts, among them J1 USB_A, J2 Conn_01x04_Pin, SW1 SW_SPDT, U1 STM32F407VGTx, U2 AMS1117-3.3, Y1 16mH

Commit message: e
e
Parts:
- Y1: value 16mH -> 16MhZ
Changed lines of the file:
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@@
 		(fields_autoplaced yes)
 		(property "Reference" "Y1"
-			(at 66.04 106.6098 0)
+			(at 67.31 106.6098 0)
 			(effects
 				(font
@@
 			)
 		)
-		(property "Value" "16mH"
-			(at 66.04 109.1498 0)
+		(property "Value" "16MhZ"
+			(at 67.31 109.1498 0)
 			(effects
 				(font
