File: KicadProjects/A1_SMD_THB/gpiobreakout.kicad_sch (KiCad schematic)
At the start: 0 parts

Commit message: e
e
Other:
- note added: "Just the spare gpio pins that aren't being used, might be excluded"
Changed lines of the file:
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@@
 	(generator_version "9.0")
 	(paper "A5")
+	(text "Just the spare gpio pins that aren't being used, might be excluded"
+		(exclude_from_sim no)
+		(at 111.76 63.246 0)
+		(effects
+			(font
+				(size 1.27 1.27)
+			)
+		)
+	)
 	(hierarchical_label "GPIO_28"
 		(shape input)
