File: KicadProjects/A1_SMD_THB/mcu.kicad_sch (KiCad schematic)
At the start: 30 parts, among them J1 Conn_01x02_Pin, J2 Conn_01x04_Pin, J4 Conn_01x03_Pin, U1 RP2040, U2 NCP1117-1.5_SOT223, U4 W25Q128JVS, Y1 ABM8-272-T3

Commit message: e
e
Parts:
- added R36: 10k, Resistor_SMD:R_0402_1005Metric, symbol Device:R
- J2: value Conn_01x04_Pin -> SWD; footprint Connector_PinHeader_2.54mm:PinHeader_1x04_P2.54mm_Vertical -> Connector_PinHeader_1.27mm:PinHeader_1x04_P1.27mm_Vertical; now not fitted
- J4: now not fitted; now left out of the parts list
Connections:
- net +3V3: now also J4.2 (Pin_2), R36.1
- net at U1.26 (RUN): now also R36.2; no longer J4.2 (Pin_2)
Changed lines of the file:
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@@
 	)
 	(junction
+		(at 78.74 62.23)
+		(diameter 0)
+		(color 0 0 0 0)
+	)
+	(junction
 		(at 135.89 30.48)
 		(diameter 0)
@@
 	)
 	(junction
+		(at 78.74 58.42)
+		(diameter 0)
+		(color 0 0 0 0)
+	)
+	(junction
 		(at 189.23 38.1)
 		(diameter 0)
@@
 	(wire
 		(pts
-			(xy 106.68 62.23) (xy 81.28 62.23)
+			(xy 106.68 62.23) (xy 97.79 62.23)
 		)
 		(stroke
@@
 	(wire
 		(pts
+			(xy 90.17 62.23) (xy 78.74 62.23)
+		)
+		(stroke
+			(width 0)
+			(type default)
+		)
+	)
+	(wire
+		(pts
 			(xy 135.89 54.61) (xy 137.16 54.61)
 		)
@@
 	(wire
 		(pts
-			(xy 81.28 62.23) (xy 81.28 60.96)
+			(xy 76.2 62.23) (xy 76.2 60.96)
 		)
 		(stroke
@@
 	(wire
 		(pts
+			(xy 78.74 58.42) (xy 78.74 62.23)
+		)
+		(stroke
+			(width 0)
+			(type default)
+		)
+	)
+	(wire
+		(pts
 			(xy 127 41.91) (xy 127 54.61)
 		)
@@
 	(wire
 		(pts
+			(xy 78.74 62.23) (xy 76.2 62.23)
+		)
+		(stroke
+			(width 0)
+			(type default)
+		)
+	)
+	(wire
+		(pts
 			(xy 127 30.48) (xy 127 27.94)
 		)
@@
 	(wire
 		(pts
+			(xy 76.2 63.5) (xy 81.28 63.5)
+		)
+		(stroke
+			(width 0)
+			(type default)
+		)
+	)
+	(wire
+		(pts
 			(xy 118.11 44.45) (xy 118.11 41.91)
 		)
@@
 	(wire
 		(pts
-			(xy 87.63 58.42) (xy 81.28 58.42)
+			(xy 87.63 58.42) (xy 78.74 58.42)
 		)
 		(stroke
@@
 	(wire
 		(pts
+			(xy 78.74 58.42) (xy 76.2 58.42)
+		)
+		(stroke
+			(width 0)
+			(type default)
+		)
+	)
+	(wire
+		(pts
 			(xy 135.89 29.21) (xy 135.89 30.48)
 		)
@@
 	)
 	(symbol
-		(lib_id "Connector:Conn_01x03_Pin")
-		(at 76.2 60.96 0)
+		(lib_id "Device:R")
+		(at 93.98 62.23 90)
 		(unit 1)
 		(exclude_from_sim no)
@@
 		(dnp no)
 		(fields_autoplaced yes)
+		(property "Reference" "R36"
+			(at 93.98 55.88 90)
+			(effects
+				(font
+					(size 1.27 1.27)
+				)
+			)
+		)
+		(property "Value" "10k"
+			(at 93.98 58.42 90)
+			(effects
+				(font
+					(size 1.27 1.27)
+				)
+			)
+		)
+		(property "Footprint" "Resistor_SMD:R_0402_1005Metric"
+			(at 93.98 64.008 90)
+			(effects
+				(font
+					(size 1.27 1.27)
+				)
+				(hide yes)
+			)
+		)
+		(property "Datasheet" "~"
+			(at 93.98 62.23 0)
+			(effects
+				(font
+					(size 1.27 1.27)
+				)
+				(hide yes)
+			)
+		)
+		(property "Description" "Resistor"
+			(at 93.98 62.23 0)
+			(effects
+				(font
+					(size 1.27 1.27)
+				)
+				(hide yes)
+			)
+		)
+		(pin "1"
+		)
+		(pin "2"
+		)
+		(instances
+			(project "A1_SMD_THB"
+				(path "/34183abe-6288-4424-a0b3-d63b1476ac75/39133467-43bc-4492-b4f0-6de52d085be2"
+					(reference "R36")
+					(unit 1)
+				)
+			)
+		)
+	)
+	(symbol
+		(lib_id "Connector:Conn_01x03_Pin")
+		(at 71.12 60.96 0)
+		(unit 1)
+		(exclude_from_sim yes)
+		(in_bom no)
+		(on_board no)
+		(dnp yes)
+		(fields_autoplaced yes)
 		(property "Reference" "J4"
-			(at 76.835 53.34 0)
+			(at 71.755 53.34 0)
 			(effects
 				(font
@@
 		)
 		(property "Value" "Conn_01x03_Pin"
-			(at 76.835 55.88 0)
+			(at 71.755 55.88 0)
 			(effects
 				(font
@@
 		)
 		(property "Footprint" "Connector_PinHeader_2.54mm:PinHeader_1x03_P2.54mm_Vertical"
-			(at 76.2 60.96 0)
+			(at 71.12 60.96 0)
 			(effects
 				(font
@@
 		)
 		(property "Datasheet" "~"
-			(at 76.2 60.96 0)
+			(at 71.12 60.96 0)
 			(effects
 				(font
@@
 		)
 		(property "Description" "Generic connector, single row, 01x03, script generated"
-			(at 76.2 60.96 0)
+			(at 71.12 60.96 0)
 			(effects
 				(font
@@
 		(in_bom yes)
 		(on_board yes)
-		(dnp no)
+		(dnp yes)
 		(fields_autoplaced yes)
 		(property "Reference" "J2"
@@
 			)
 		)
-		(property "Value" "Conn_01x04_Pin"
+		(property "Value" "SWD"
 			(at 88.265 123.19 0)
 			(effects
@@
 			)
 		)
-		(property "Footprint" "Connector_PinHeader_2.54mm:PinHeader_1x04_P2.54mm_Vertical"
+		(property "Footprint" "Connector_PinHeader_1.27mm:PinHeader_1x04_P1.27mm_Vertical"
 			(at 87.63 128.27 0)
 			(effects

Commit message: e
e
Parts:
- renumbered C16 to C101, C15 to C102, C12 to C103, C18 to C104, C17 to C105, C13 to C106, C3 to C107, C2 to C108, C1 to C109, C4 to C110, C5 to C111, C6 to C112, C7 to C113, C8 to C114, C9 to C115, C10 to C116, C11 to C117, C14 to C118, J4 to J101, J2 to J102, J1 to J103, R5 to R102, R36 to R103, R1 to R104, R2 to R105, R3 to R106, R4 to R107, U2 to U101, U1 to U102, U4 to U103, Y1 to Y101
Other:
- note added: "Decoupling capacitors, stay close to 3v3 pins"
- note added: "Decoupling caps"
- note added: "Doesn't need to be strong."
- note added: "Don't add usb bus resistors"
- note added: "Keep Caps Close"
- note added: "Need ground pour for heat dissapation"
- note added: "Not neccesary, p = 1.25mm for size constraint"
- note added: "Specific Chip Doesn't require it"
- moved on the sheet: C101, C102, C103, C104, C105, C106, C107, C108, C109, C110, C111, C112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
