File: KicadProjects/A1_SMD_THB/A1_SMD_THB.kicad_pcb (KiCad board)
At the start: 2 copper layers, 52 parts, among them J1 Conn_01x02_Pin, J2 Conn_01x04_Pin, J3 PCF, J4 Conn_01x03_Pin, J5 EXF, J6 THO, J7 HE, J8 BL_PROBE, J9 BL_SERVO, P1 USB_C_Plug, U1 RP2040, U2 NCP1117-1.5_SOT223, U3 TMC2209-LA, U4 W25Q128JVS, Y1 ABM8-272-T3

Commit message: e
e
Parts:
- added C28: 100nF, Capacitor_SMD:C_0402_1005Metric, F.Cu at (113.2, 89.6)
- added C29: 100nF, Capacitor_SMD:C_0402_1005Metric, F.Cu at (113.2, 91.6)
- added C30: 100nF, Capacitor_SMD:C_0402_1005Metric, F.Cu at (113.2, 93.5)
- added D5: BAV99, Package_TO_SOT_SMD:SOT-23, F.Cu at (117.1, 91.0)
- added J16: SFS1, Connector_PinHeader_2.54mm:PinHeader_1x01_P2.54mm_Vertical, F.Cu at (59.0, 92.0)
- moved J1 129.3 mm to (62.5, 65.0), turned to 90 degrees
- moved J2 74.3 mm to (102.8, 90.9)
- moved J4 74.3 mm to (107.4, 90.9)
- moved C12 64.8 mm to (82.9, 62.2), turned to 0 degrees
- moved C13 60.7 mm to (85.6, 64.3), turned to 0 degrees
- moved U2 53.8 mm to (84.5, 70.0), turned to -90 degrees
- moved J8 48.2 mm to (68.5, 98.0), turned to -90 degrees
- moved C20 36.5 mm to (113.0, 66.0)
- moved J6 33.5 mm to (53.5, 86.0)
- moved J5 28.7 mm to (67.5, 90.5), turned to 0 degrees
- moved R8 28.3 mm to (88.0, 88.2)
- moved C25 28.2 mm to (94.0, 90.5)
- moved C22 26.9 mm to (85.5, 86.5)
- moved C26 26.2 mm to (92.1, 84.2)
- moved C27 26.2 mm to (92.1, 82.7)
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Connections:
- J6 pad 1: unconnected-(J6-Pin_1-Pad1) -> Net-(J6-Pin_1)
- J6 pad 2: unconnected-(J6-Pin_2-Pad2) -> GND
- J7 pad 1: unconnected-(J7-Pin_1-Pad1) -> +24V
- J7 pad 2: unconnected-(J7-Pin_2-Pad2) -> Net-(D1-K)
- J8 pad 1: unconnected-(J8-Pin_1-Pad1) -> GND3
- J8 pad 2: unconnected-(J8-Pin_2-Pad2) -> /mainio/BL_PROBE
- J9 pad 1: unconnected-(J9-Pin_1-Pad1) -> GND3
- J9 pad 2: unconnected-(J9-Pin_2-Pad2) -> +3V3
- J9 pad 3: unconnected-(J9-Pin_3-Pad3) -> /mainio/BL_SERVO

Commit message: e
e
Parts:
- removed C20: 100uF, Capacitor_SMD:CP_Elec_8x10
- removed J16: SFS1, Connector_PinHeader_2.54mm:PinHeader_1x01_P2.54mm_Vertical
- removed J4: Conn_01x03_Pin, Connector_PinHeader_2.54mm:PinHeader_1x03_P2.54mm_Vertical
- added J11: F_SR1, Connector_PinHeader_2.54mm:PinHeader_1x02_P2.54mm_Vertical, F.Cu at (61.0, 86.5)
- added J12: F_SR2, Connector_PinHeader_2.54mm:PinHeader_1x02_P2.54mm_Vertical, F.Cu at (54.5, 86.5)
- added J13: PCF_FAN, Connector_JST:JST_XH_B4B-XH-A_1x04_P2.50mm_Vertical, F.Cu at (85.3, 99.8)
- added Q1: NMOS, A1_SMD_THB:sot23f, F.Cu at (61.0, 72.4)
- added R13: 20k, Resistor_SMD:R_0402_1005Metric, F.Cu at (59.2, 89.4)
- added R14: 100, Resistor_SMD:R_0402_1005Metric, F.Cu at (60.2, 89.4)
- added R15: 100, Resistor_SMD:R_0402_1005Metric, F.Cu at (58.2, 89.4)
- added R16: 20k, Resistor_SMD:R_0402_1005Metric, F.Cu at (57.2, 89.4)
- added R17: 10R, Resistor_SMD:R_0402_1005Metric, F.Cu at (59.9, 74.8)
- added R18: 20kR, Resistor_SMD:R_0402_1005Metric, F.Cu at (61.6, 74.6)
- added R19: 20kR, Resistor_SMD:R_0402_1005Metric, F.Cu at (54.9, 69.8)
- added R20: 2.37kR, Resistor_SMD:R_0402_1005Metric, F.Cu at (61.8, 83.3)
- added R21: 10k, Resistor_SMD:R_0402_1005Metric, F.Cu at (88.2, 95.8)
- added R22: 100, Resistor_SMD:R_0402_1005Metric, F.Cu at (87.2, 95.8)
- added R25: 10k, Resistor_SMD:R_0402_1005Metric, F.Cu at (82.6, 95.8)
- added R26: 100, Resistor_SMD:R_0402_1005Metric, F.Cu at (81.6, 95.8)
- added R27: 4.7kR, Resistor_SMD:R_0402_1005Metric, F.Cu at (59.9, 83.3)
- added R28: 2.37kR, Resistor_SMD:R_0402_1005Metric, F.Cu at (62.1, 78.6)
- added R32: 100o, Resistor_SMD:R_0402_1005Metric, F.Cu at (74.0, 94.8)
- added R33: 100o, Resistor_SMD:R_0402_1005Metric, F.Cu at (75.5, 94.8)
- added R34: 100o, Resistor_SMD:R_0402_1005Metric, F.Cu at (76.0, 86.0)
- added R35: 100o, Resistor_SMD:R_0402_1005Metric, F.Cu at (70.7, 90.5)
- added R36: 10k, Resistor_SMD:R_0402_1005Metric, F.Cu at (73.9, 80.3)
- J2: value Conn_01x04_Pin -> SWD; footprint Connector_PinHeader_2.54mm:PinHeader_1x04_P2.54mm_Vertical -> Connector_PinHeader_1.27mm:PinHeader_1x04_P1.27mm_Vertical
- J3: value PCF -> EXF; footprint Connector_JST:JST_XH_B4B-XH-A_1x04_P2.50mm_Vertical -> Connector_JST:JST_XH_B5B-XH-A_1x05_P2.50mm_Vertical
- J5: value EXF -> ADXL345; footprint Connector_JST:JST_XH_B5B-XH-A_1x05_P2.50mm_Vertical -> Connector_PinHeader_2.54mm:PinHeader_1x04_P2.54mm_Vertical
- J8: footprint Connector_JST:JST_XH_B2B-XH-A_1x02_P2.50mm_Vertical -> Connector_PinHeader_2.54mm:PinHeader_1x02_P2.54mm_Vertical
- J9: footprint Connector_JST:JST_XH_B3B-XH-A_1x03_P2.50mm_Vertical -> Connector_PinHeader_2.54mm:PinHeader_1x03_P2.54mm_Vertical
- P1: footprint Connector_USB:USB_C_Receptacle_G-Switch_GT-USB-7025 -> Connector_USB:USB_C_Receptacle_HCTL_HC-TYPE-C-16P-01A
- R10, R11, R12: footprint Capacitor_SMD:C_0201_0603Metric -> Resistor_SMD:R_0402_1005Metric
- R6: footprint Resistor_SMD:R_0603_1608Metric -> Resistor_SMD:R_0402_1005Metric
- U3: footprint A1_SMD_THB:QFN50P500X500X90-29N -> A1_SMD_THB:TMC2209-LA
- moved C28 61.9 mm to (54.9, 68.6)
- moved D5 57.0 mm to (60.9, 81.0)
- moved C29 55.0 mm to (58.2, 91.3), turned to -90 degrees
- moved C30 51.4 mm to (64.0, 78.6)
- moved J5 31.3 mm to (97.8, 82.7)
- moved J2 21.1 mm to (84.0, 81.2), turned to -90 degrees
- moved J9 18.4 mm to (56.9, 94.1), turned to -90 degrees
- moved C26 18.3 mm to (77.4, 95.1), turned to 90 degrees
- moved C17 17.4 mm to (82.8, 72.8)
- moved C7 16.5 mm to (66.7, 75.2), turned to 180 degrees
- moved J3 16.5 mm to (69.2, 99.8)
- moved J8 16.1 mm to (54.5, 90.1)
- moved C21 15.5 mm to (74.0, 86.2)
- moved C24 15.1 mm to (73.4, 84.6)
- moved C22 15.0 mm to (73.0, 94.8), turned to 90 degrees
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Connections:
- net /accelerometer/SPI_CS renamed /mcu/G9
- net /accelerometer/SPI_SDO renamed /mcu/G8
- J3 pad 2: unconnected-(J3-Pin_2-Pad2) -> +24V
- J3 pad 3: unconnected-(J3-Pin_3-Pad3) -> GND
- J3 pad 4: unconnected-(J3-Pin_4-Pad4) -> Net-(J3-Pin_4)
- J5 pad 1: unconnected-(J5-Pin_1-Pad1) -> +3V3
- J5 pad 2: unconnected-(J5-Pin_2-Pad2) -> GND
- J5 pad 3: unconnected-(J5-Pin_3-Pad3) -> /accelerometer/SDA
- J5 pad 4: unconnected-(J5-Pin_4-Pad4) -> /accelerometer/SCL
- R12 pad 2: /mcu/G21 -> Net-(U3-~{EN})
- U1 pad 8: /accelerometer/SPI_SCK -> /accelerometer/SDA
- U1 pad 9: /accelerometer/SPI_SDI -> /accelerometer/SCL
- U3 pad 11: unconnected-(U3-DIAG-Pad11) -> Net-(U3-DIAG)
- U3 pad 16: /mcu/G22 -> Net-(U3-STEP)
- U3 pad 19: /mcu/G23 -> Net-(U3-DIR)
- U3 pad 2: /mcu/G21 -> Net-(U3-~{EN})
- U3 pad 21: Net-(EXM2-Pin_2) -> Net-(EXM2-Pin_4)
- U3 pad 24: Net-(EXM2-Pin_4) -> Net-(EXM2-Pin_3)
- U3 pad 26: Net-(EXM2-Pin_3) -> Net-(EXM2-Pin_2)
Routing:
- net GND: track 0.00 -> 29.8 mm, vias 0 -> 2
- net +24V: track 0.00 -> 18.5 mm
- net Net-(EXM2-Pin_1): track 0.00 -> 17.1 mm, vias 0 -> 1
- net Net-(EXM2-Pin_4): track 0.00 -> 16.9 mm, vias 0 -> 1
- net Net-(EXM2-Pin_2): track 0.00 -> 16.0 mm, vias 0 -> 1
- net Net-(EXM2-Pin_3): track 0.00 -> 15.7 mm, vias 0 -> 1
- net Net-(J6-Pin_1): track 0.00 -> 9.51 mm
- net Net-(J13-Pin_4): track 0.00 -> 6.05 mm
- net Net-(J13-Pin_3): track 0.00 -> 4.78 mm
- net +3.3VADC: track 0.00 -> 1.47 mm
Other:
- board outline added: 50 x 44 mm
- board text added: "GND"

Commit message: e
e
Parts:
- removed C11, C14, C22, C28, C29, C30: 100nF, Capacitor_SMD:C_0402_1005Metric
- removed C12, C13, C17, C18: 10uF, Capacitor_SMD:C_0805_2012Metric
- removed C15, C16: 15pF, Capacitor_SMD:C_0402_1005Metric
- removed C21: 22nF 50V, Capacitor_SMD:C_0603_1608Metric
- removed C23: 4.7uF, Capacitor_SMD:C_0603_1608Metric
- removed C24, C26, C27: 100nF 50V, Capacitor_SMD:C_0603_1608Metric
- removed C25: 100uF, Capacitor_SMD:CP_Elec_8x10
- removed D5: BAV99, Package_TO_SOT_SMD:SOT-23
- removed J2: SWD, Connector_PinHeader_1.27mm:PinHeader_1x04_P1.27mm_Vertical
- removed P1: USB_C_Plug, Connector_USB:USB_C_Receptacle_HCTL_HC-TYPE-C-16P-01A
- removed Q1: NMOS, A1_SMD_THB:sot23f
- removed R1, R2: 27.4o, Resistor_SMD:R_0402_1005Metric
- removed R10, R11, R12: 20kΩ, Resistor_SMD:R_0402_1005Metric
- removed R13, R16: 20k, Resistor_SMD:R_0402_1005Metric
- removed R14, R15, R22, R26: 100, Resistor_SMD:R_0402_1005Metric
- removed R17: 10R, Resistor_SMD:R_0402_1005Metric
- removed R18, R19: 20kR, Resistor_SMD:R_0402_1005Metric
- removed R20, R28: 2.37kR, Resistor_SMD:R_0402_1005Metric
- removed R21, R25, R36: 10k, Resistor_SMD:R_0402_1005Metric
- removed R27: 4.7kR, Resistor_SMD:R_0402_1005Metric
- removed R3: 1ko, Resistor_SMD:R_0603_1608Metric
- removed R32, R33, R34, R35: 100o, Resistor_SMD:R_0402_1005Metric
- removed R5: 1k, Resistor_SMD:R_0603_1608Metric
- removed R6: 1k, Resistor_SMD:R_0402_1005Metric
- removed R8, R9: 100mΩ, Resistor_SMD:R_1206_3216Metric
- removed U1: RP2040, Package_DFN_QFN:QFN-56-1EP_7x7mm_P0.4mm_EP3.2x3.2mm
- removed U2: NCP1117-1.5_SOT223, Package_TO_SOT_SMD:SOT-223-3_TabPin2
- removed U3: TMC2209-LA, A1_SMD_THB:TMC2209-LA
- removed U4: W25Q128JVS, Package_SO:SOIC-8_5.3x5.3mm_P1.27mm
- removed Y1: ABM8-272-T3, Crystal:Crystal_SMD_Abracon_ABM8AIG-4Pin_3.2x2.5mm
- added C119: 100nF, Capacitor_SMD:C_0402_1005Metric, F.Cu at (120.4, 105.0)
- added C120: 100nF, Capacitor_SMD:C_0402_1005Metric, F.Cu at (120.4, 107.0)
- added C121: 100nF, Capacitor_SMD:C_0402_1005Metric, F.Cu at (120.4, 108.9)
- added C122: 22nF 50V, Capacitor_SMD:C_0603_1608Metric, F.Cu at (108.2, 78.5)
- added C123: 100nF 50V, Capacitor_SMD:C_0603_1608Metric, F.Cu at (108.2, 81.0)
- added C124: 100nF 50V, Capacitor_SMD:C_0603_1608Metric, F.Cu at (108.2, 83.5)
- added C125: 100uF, Capacitor_SMD:CP_Elec_8x10, F.Cu at (123.2, 90.5)
- added C126: 100nF 50V, Capacitor_SMD:C_0603_1608Metric, F.Cu at (108.2, 86.0)
- added C127: 4.7uF, Capacitor_SMD:C_0603_1608Metric, F.Cu at (108.2, 88.5)
- added C128: 100nF, Capacitor_SMD:C_0402_1005Metric, F.Cu at (124.2, 96.4)
- added D101: BAV99, Package_TO_SOT_SMD:SOT-23, F.Cu at (121.4, 112.3)
- added P101: USB_C_Plug, Connector_USB:USB_C_Receptacle_HCTL_HC-TYPE-C-16P-01A, F.Cu at (131.7, 109.4)
- added R101: 1k, Resistor_SMD:R_0402_1005Metric, F.Cu at (77.5, 72.0)
- added R108: 100, Resistor_SMD:R_0402_1005Metric, F.Cu at (76.5, 91.5)
- added R109: 100, Resistor_SMD:R_0402_1005Metric, F.Cu at (113.7, 78.2)
- added R110: 4.7kR, Resistor_SMD:R_0402_1005Metric, F.Cu at (117.5, 107.0)
- added R111: 2.37kR, Resistor_SMD:R_0402_1005Metric, F.Cu at (82.0, 91.5)
- added R112: 20k, Resistor_SMD:R_0402_1005Metric, F.Cu at (113.7, 80.2)
- added R113: 20k, Resistor_SMD:R_0402_1005Metric, F.Cu at (113.7, 82.2)
- added R117: 2.37kR, Resistor_SMD:R_0402_1005Metric, F.Cu at (117.5, 109.0)
- added R118: 10k, Resistor_SMD:R_0402_1005Metric, F.Cu at (114.6, 113.0)
- added R119: 100, Resistor_SMD:R_0402_1005Metric, F.Cu at (117.5, 105.0)
- added R120: 10R, Resistor_SMD:R_0402_1005Metric, F.Cu at (111.7, 113.0)
- added R121: 20kR, Resistor_SMD:R_0402_1005Metric, F.Cu at (114.6, 105.0)
- added R123: 10k, Resistor_SMD:R_0402_1005Metric, F.Cu at (114.6, 109.0)
- added R124: 100, Resistor_SMD:R_0402_1005Metric, F.Cu at (114.6, 111.0)
- added R127: 20kΩ, Resistor_SMD:R_0402_1005Metric, F.Cu at (104.8, 78.2)
- added R128: 20kΩ, Resistor_SMD:R_0402_1005Metric, F.Cu at (104.8, 80.2)
- added R129: 20kΩ, Resistor_SMD:R_0402_1005Metric, F.Cu at (104.8, 82.2)
- added R130: 100o, Resistor_SMD:R_0402_1005Metric, F.Cu at (104.8, 84.2)
- added R131: 100o, Resistor_SMD:R_0402_1005Metric, F.Cu at (104.8, 86.2)
- added R132: 100o, Resistor_SMD:R_0402_1005Metric, F.Cu at (104.8, 88.2)
- added R133: 100mΩ, Resistor_SMD:R_1206_3216Metric, F.Cu at (119.9, 97.1)
- added R134: 100mΩ, Resistor_SMD:R_1206_3216Metric, F.Cu at (119.9, 100.4)
- added R135: 100o, Resistor_SMD:R_0402_1005Metric, F.Cu at (104.8, 90.1)
- added U104: TMC2209-LA, OpenA1K:TMC2209 Footprint, F.Cu at (119.3, 52.7)
- added U105: STM32G474RBTx, Package_QFP:LQFP-64_10x10mm_P0.5mm, F.Cu at (75.2, 79.8)
- C1: value 1uF -> 10uF; footprint Capacitor_SMD:C_0603_1608Metric -> Capacitor_SMD:C_0201_0603Metric
- C10, C6: value 100nF -> 10uF; footprint Capacitor_SMD:C_0402_1005Metric -> Capacitor_SMD:C_0603_1608Metric
- C4: value 1uF -> 100nF; footprint Capacitor_SMD:C_0603_1608Metric -> Capacitor_SMD:C_0402_1005Metric
- C7: value 100nF -> 10nF
- C8, C9: value 100nF -> 1uF; footprint Capacitor_SMD:C_0402_1005Metric -> Capacitor_SMD:C_0201_0603Metric
- moved C10 21.1 mm to (87.7, 74.5), turned to 0 degrees
- moved C4 16.6 mm to (67.5, 83.0), turned to 90 degrees
- moved C7 16.0 mm to (77.0, 87.5), turned to -90 degrees
- moved C9 11.6 mm to (88.2, 71.0)
- moved C8 11.0 mm to (88.2, 69.3)
- moved C1 10.5 mm to (82.5, 76.2), turned to -90 degrees
- moved C6 9.72 mm to (86.7, 83.5)
- moved C5 9.48 mm to (78.5, 87.0), turned to 180 degrees
- moved C3 7.89 mm to (71.5, 72.5), turned to 0 degrees
- moved C2 7.77 mm to (67.5, 76.0), turned to 180 degrees
- renumbered EXM2 to EXM101, J6 to J104, J12 to J105, J11 to J106, J3 to J107, J7 to J108, J13 to J109, J8 to J111, J9 to J112, J5 to J113
Connections:
- C1 pad 1: +1V1 -> +3V3
- C1 pad 2: GND3 -> GND
- C10 pad 1: +3V3 -> GND
- C10 pad 2: GND3 -> +3V3
- C2 pad 1: +1V1 -> +3V3
- C2 pad 2: GND3 -> GND
- C3 pad 1: +1V1 -> +3V3
- C3 pad 2: GND3 -> GND
- C4 pad 2: GND3 -> GND
- C5 pad 2: GND3 -> GND
- C6 pad 2: GND3 -> GND
- C7 pad 1: +3V3 -> +3V3A
- C7 pad 2: GND3 -> GND
- C8 pad 1: +3V3 -> +3V3A
- C8 pad 2: GND3 -> GND
- C9 pad 2: GND3 -> GND
Routing:
- net GND: track 29.8 -> 0.00 mm, vias 2 -> 0
- net +24V: track 18.5 -> 0.00 mm
- net Net-(EXM101-Pin_1): track 17.1 -> 0.00 mm, vias 1 -> 0
- net Net-(EXM101-Pin_4): track 16.9 -> 0.00 mm, vias 1 -> 0
- net Net-(EXM101-Pin_2): track 16.0 -> 0.00 mm, vias 1 -> 0
- net Net-(EXM101-Pin_3): track 15.7 -> 0.00 mm, vias 1 -> 0
- net Net-(J104-Pin_1): track 9.51 -> 0.00 mm
- net Net-(J109-Pin_4): track 6.05 -> 0.00 mm
- net Net-(J109-Pin_3): track 4.78 -> 0.00 mm
- net +3.3VADC: track 1.47 -> 0.00 mm

Commit message: e
e
Parts:
- removed C1: 10uF, Capacitor_SMD:C_0201_0603Metric
- removed C10, C6: 10uF, Capacitor_SMD:C_0603_1608Metric
- removed C2, C3, C4, C5: 100nF, Capacitor_SMD:C_0402_1005Metric
- removed C7: 10nF, Capacitor_SMD:C_0402_1005Metric
- removed C8, C9: 1uF, Capacitor_SMD:C_0201_0603Metric
- removed J1: Conn_01x02_Pin, Connector_PinHeader_2.54mm:PinHeader_1x02_P2.54mm_Vertical
- removed the J107 at (69.2, 99.8)
- removed the J108 at (53.5, 73.5)
- removed the R109 at (113.7, 78.2)
- removed R113: 20k, Resistor_SMD:R_0402_1005Metric
- removed R118: 10k, Resistor_SMD:R_0402_1005Metric
- removed R119: 100, Resistor_SMD:R_0402_1005Metric
- removed R120: 10R, Resistor_SMD:R_0402_1005Metric
- removed U105: STM32G474RBTx, Package_QFP:LQFP-64_10x10mm_P0.5mm
- added C145: 30pF, Capacitor_SMD:C_0402_1005Metric, F.Cu at (54.6, 72.0)
- added C146: 30pF, Capacitor_SMD:C_0402_1005Metric, F.Cu at (59.9, 71.7)
- added C147: 100nF, Capacitor_SMD:C_0402_1005Metric, F.Cu at (55.7, 68.6)
- added C148: 100nF, Capacitor_SMD:C_0402_1005Metric, F.Cu at (61.5, 71.9)
- added C149: 100nF, Capacitor_SMD:C_0402_1005Metric, F.Cu at (60.5, 60.3)
- added C150: 10uF, Capacitor_SMD:C_0603_1608Metric, F.Cu at (54.3, 69.4)
- added C151: 10nF, Capacitor_SMD:C_0402_1005Metric, F.Cu at (63.5, 62.2)
- added C152: 1uF, Capacitor_SMD:C_0201_0603Metric, F.Cu at (63.3, 63.2)
- added C153: 1uF, Capacitor_SMD:C_0201_0603Metric, F.Cu at (64.8, 62.5)
- added FB102: 120r 100MHz, Capacitor_SMD:C_0603_1608Metric, F.Cu at (64.0, 64.3)
- added J110: EXF, Connector_JST:JST_XH_B5B-XH-A_1x05_P2.50mm_Vertical, F.Cu at (61.9, 79.3)
- added J115: BOOT, Connector_PinHeader_2.54mm:PinHeader_1x03_P2.54mm_Vertical, F.Cu at (47.8, 63.1)
- added Q101: NMOS, A1KLibrary:PPAK-8L 5x6 Mosfet, F.Cu at (54.3, 48.1)
- added R111: 10R, Resistor_SMD:R_0402_1005Metric, F.Cu at (51.5, 53.1)
- added R114: 100, Resistor_SMD:R_0402_1005Metric, F.Cu at (44.0, 71.0)
- added R115: 100, Resistor_SMD:R_0402_1005Metric, F.Cu at (44.0, 63.0)
- added R116: 20k, Resistor_SMD:R_0402_1005Metric, F.Cu at (44.0, 73.0)
- added R122: 10k, Resistor_SMD:R_0402_1005Metric, F.Cu at (75.1, 72.6)
- added R125: 10k, Resistor_SMD:R_0402_1005Metric, F.Cu at (70.2, 75.2)
- added R126: 4.7k, Resistor_SMD:R_0402_1005Metric, F.Cu at (67.3, 75.7)
- added R138: 10kR, Resistor_SMD:R_0402_1005Metric, F.Cu at (50.6, 65.7)
- added SW101: SW_SPST, A1KLibrary:A Stupid Button, F.Cu at (63.4, 66.2)
- added U106: STM32G431KBU3, Package_DFN_QFN:QFN-32-1EP_5x5mm_P0.5mm_EP3.45x3.45mm, F.Cu at (58.7, 64.5)
- added Y103: Crystal_GND24, Crystal:Crystal_SMD_3225-4Pin_3.2x2.5mm, F.Cu at (57.2, 71.9)
- J104: value THO -> SGDBM-08-020P-H40; footprint Connector_JST:JST_XH_B2B-XH-A_1x02_P2.50mm_Vertical -> A1KLibrary:Mezzanine Connector
- J105: renamed from J111; footprint Connector_PinHeader_2.54mm:PinHeader_1x02_P2.54mm_Vertical -> Connector_JST:JST_PH_B2B-PH-K_1x02_P2.00mm_Vertical
- J106: renamed from J112; footprint Connector_PinHeader_2.54mm:PinHeader_1x03_P2.54mm_Vertical -> Connector_JST:JST_PH_B3B-PH-K_1x03_P2.00mm_Vertical
- J107: renamed from J105; footprint Connector_PinHeader_2.54mm:PinHeader_1x02_P2.54mm_Vertical -> Connector_JST:JST_PH_B2B-PH-K_1x02_P2.00mm_Vertical
- J108: renamed from J106; footprint Connector_PinHeader_2.54mm:PinHeader_1x02_P2.54mm_Vertical -> Connector_JST:JST_PH_B2B-PH-K_1x02_P2.00mm_Vertical
- J111: renamed from J113; footprint Connector_PinHeader_2.54mm:PinHeader_1x04_P2.54mm_Vertical -> Connector_JST:JST_PH_B4B-PH-K_1x04_P2.00mm_Vertical
- R108: value 100 -> 2.37kR
- R112: value 20k -> 20kR
- R117: value 2.37kR -> 20k
- R121: value 20kR -> 10k
- R123: value 10k -> 4.7k
- R124: value 100 -> 10k
- U104: footprint OpenA1K:TMC2209 Footprint -> A1KLibrary:TMC2209-LA-FOOTPRINT
- moved D101 98.2 mm to (43.4, 52.6), turned to -90 degrees
- moved P101 96.9 mm to (60.2, 44.0), turned to 180 degrees
- moved R110 94.7 mm to (40.7, 51.6), turned to 180 degrees
- moved C119 90.8 mm to (44.5, 55.0)
- moved C121 87.8 mm to (45.0, 64.0)
- moved R117 85.6 mm to (44.0, 65.0), turned to 180 degrees
- moved C120 83.1 mm to (45.0, 72.0)
- moved R112 68.8 mm to (50.5, 53.1), turned to 90 degrees
- moved C127 65.0 mm to (75.0, 46.8)
- moved J111 63.1 mm to (39.8, 57.8)
- moved C130 59.4 mm to (72.3, 67.3), turned to 90 degrees
- moved R134 59.3 mm to (78.7, 57.8), turned to 90 degrees
- moved R109 56.7 mm to (40.7, 52.6)
- moved R124 56.2 mm to (71.2, 75.2), turned to -90 degrees
- moved R133 51.8 mm to (78.7, 65.7), turned to -90 degrees
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- renumbered C122 to C124, C123 to C125, C124 to C126, C125 to C127, C126 to C128, C127 to C129, C128 to C130, R111 to R109
Connections:
- net /mcu_stm32/MT_UART_TX renamed /mcu_stm32_smol/MT_UART_TX
- C119 pad 1: Net-(C119-Pad1) -> /mainio/THO
- C119 pad 2: GND3 -> GND
- C121 pad 1: /mainio/THO -> Net-(C121-Pad1)
- C121 pad 2: GND -> GND3
- J104 pad 1: Net-(J104-Pin_1) -> +24V
- J104 pad 2: GND -> +24V
- J108 pad 1: unconnected-(J106-Pin_1-Pad1) -> GND
- J108 pad 2: Net-(J106-Pin_2) -> Net-(J108-Pin_2)
- J109 pad 3: Net-(J109-Pin_3) -> /mainio/PCF_PWM
- P101 pad A6: /power/USB_D+ -> /mcu_stm32_smol/USB_D+
- P101 pad A7: /power/USB_D- -> /mcu_stm32_smol/USB_D-
- R101 pad 1: /mcu_stm32/MT_UART_RX -> /mcu_stm32_smol/MT_UART_RX
- R108 pad 1: /mainio/FIL_SNS1 -> Net-(D101-K-Pad3)
- R108 pad 2: Net-(C119-Pad1) -> /mainio/THO
- R109 pad 1: Net-(J104-Pin_1) -> Net-(J104-Pin_16)
- R110 pad 2: Net-(J104-Pin_1) -> Net-(J104-Pin_16)
- R112 pad 1: Net-(C119-Pad1) -> /mainio/HE_SIG
- R112 pad 2: Net-(J106-Pin_2) -> GND
- R117 pad 1: Net-(D101-K-Pad3) -> Net-(C121-Pad1)
- R117 pad 2: /mainio/THO -> Net-(J108-Pin_2)
- R121 pad 1: /mainio/HE_SIG -> /mainio/PCF_TACH
- R121 pad 2: GND -> Net-(J109-Pin_4)
- R123 pad 1: /mainio/PCF_TACH -> /mainio/PCF_PWM
- R123 pad 2: Net-(J109-Pin_4) -> GND
- R124 pad 1: /mainio/PCF_PWM -> /mainio/EXF_TACH
- R124 pad 2: Net-(J109-Pin_3) -> Net-(J110-Pin_5)
- R130 pad 1: /mcu_stm32/MT_STEP -> /mcu_stm32_smol/MT_STEP
- R131 pad 1: /mcu_stm32/MT_DIR -> /mcu_stm32_smol/MT_DIR
- R132 pad 1: /mcu_stm32/MT_ENABLE -> /mcu_stm32_smol/MT_EN
- R135 pad 2: /mcu_stm32/MT_DIAG -> /mcu_stm32_smol/MT_DIAG
Other:
- board text added: "ABL_PR"
- board text added: "ABL_SV"
- board text added: "ADXL345"
- board text added: "BOOTSEL"
- board text added: "Buck"
- board text added: "EX-FAN"
- board text added: "FSR1"
- board text added: "MT-EX"
- board text added: "Open A1 Klipper Toolhead"
- board text added: "PC-FAN"
- board text added: "RUN"
