File: KicadProjects/A1_SMD_THB/accelerometer.kicad_sch (KiCad schematic)
At the start: 0 parts

Commit message: e
e
Changed lines of the file:
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@@
 	(generator "eeschema")
 	(generator_version "9.0")
-	(paper "A4")
+	(paper "A5")
 	(hierarchical_label "SPI_SDO"
 		(shape input)
-		(at 121.92 101.6 0)
+		(at 99.06 78.74 0)
 		(effects
 			(font
@@
 	(hierarchical_label "SPI_CS"
 		(shape input)
-		(at 121.92 96.52 0)
+		(at 99.06 73.66 0)
 		(effects
 			(font
@@
 	(hierarchical_label "SPI_SCK"
 		(shape input)
-		(at 121.92 93.98 0)
+		(at 99.06 71.12 0)
 		(effects
 			(font
@@
 	(hierarchical_label "SPI_SDI"
 		(shape input)
-		(at 121.92 99.06 0)
+		(at 99.06 76.2 0)
 		(effects
 			(font

Commit message: e
e
Parts:
- added J5: ADXL345, Connector_PinHeader_2.54mm:PinHeader_1x04_P2.54mm_Vertical, symbol Connector_Generic:Conn_01x04
Connections:
- new net +3V3: J5.1 (Pin_1)
- new net GND: J5.2 (Pin_2)
- new net SCL: J5.4 (Pin_4)
- new net SDA: J5.3 (Pin_3)
Changed lines of the file:
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@@
 	(generator_version "9.0")
 	(paper "A5")
-	(hierarchical_label "SPI_SDO"
+	(wire
+		(pts
+			(xy 82.55 73.66) (xy 92.71 73.66)
+		)
+		(stroke
+			(width 0)
+			(type default)
+		)
+	)
+	(wire
+		(pts
+			(xy 92.71 71.12) (xy 82.55 71.12)
+		)
+		(stroke
+			(width 0)
+			(type default)
+		)
+	)
+	(hierarchical_label "SDA"
 		(shape input)
-		(at 99.06 78.74 0)
+		(at 82.55 76.2 0)
 		(effects
 			(font
@@
 		)
 	)
-	(hierarchical_label "SPI_CS"
+	(hierarchical_label "SCL"
 		(shape input)
-		(at 99.06 73.66 0)
+		(at 82.55 78.74 0)
 		(effects
 			(font
@@
 		)
 	)
-	(hierarchical_label "SPI_SCK"
-		(shape input)
-		(at 99.06 71.12 0)
-		(effects
-			(font
-				(size 1.27 1.27)
-			)
-			(justify left)
-		)
-	)
-	(hierarchical_label "SPI_SDI"
-		(shape input)
-		(at 99.06 76.2 0)
-		(effects
-			(font
-				(size 1.27 1.27)
-			)
-			(justify left)
-		)
-	)
+	(symbol
+		(lib_id "power:GND")
+		(at 92.71 73.66 0)
+		(unit 1)
+		(exclude_from_sim no)
+		(in_bom yes)
+		(on_board yes)
+		(dnp no)
+		(fields_autoplaced yes)
+		(property "Reference" "#PWR071"
+			(at 92.71 80.01 0)
+			(effects
+				(font
+					(size 1.27 1.27)
+				)
+				(hide yes)
+			)
+		)
+		(property "Value" "GND"
+			(at 92.71 78.74 0)
+			(effects
+				(font
+					(size 1.27 1.27)
+				)
+			)
+		)
+		(property "Footprint" ""
+			(at 92.71 73.66 0)
+			(effects
+				(font
+					(size 1.27 1.27)
+				)
+				(hide yes)
+			)
+		)
+		(property "Datasheet" ""
+			(at 92.71 73.66 0)
+			(effects
+				(font
+					(size 1.27 1.27)
+				)
+				(hide yes)
+			)
+		)
+		(property "Description" "Power symbol creates a global label with name \"GND\" , ground"
+			(at 92.71 73.66 0)
+			(effects
+				(font
+					(size 1.27 1.27)
+				)
+				(hide yes)
+			)
+		)
+		(pin "1"
+		)
+		(instances
+			(project ""
+				(path "/34183abe-6288-4424-a0b3-d63b1476ac75/d136f52e-2f1b-437a-aa44-c69ff8c5465b"
+					(reference "#PWR071")
+					(unit 1)
+				)
+			)
+		)
+	)
+	(symbol
+		(lib_id "power:+3V3")
+		(at 92.71 71.12 0)
+		(unit 1)
+		(exclude_from_sim no)
+		(in_bom yes)
+		(on_board yes)
+		(dnp no)
+		(fields_autoplaced yes)
+		(property "Reference" "#PWR030"
+			(at 92.71 74.93 0)
+			(effects
+				(font
+					(size 1.27 1.27)
+				)
+				(hide yes)
+			)
+		)
+		(property "Value" "+3V3"
+			(at 92.71 66.04 0)
+			(effects
+				(font
+					(size 1.27 1.27)
+				)
+			)
+		)
+		(property "Footprint" ""
+			(at 92.71 71.12 0)
+			(effects
+				(font
+					(size 1.27 1.27)
+				)
+				(hide yes)
+			)
+		)
+		(property "Datasheet" ""
+			(at 92.71 71.12 0)
+			(effects
+				(font
+					(size 1.27 1.27)
+				)
+				(hide yes)
+			)
+		)
+		(property "Description" "Power symbol creates a global label with name \"+3V3\""
+			(at 92.71 71.12 0)
+			(effects
+				(font
+					(size 1.27 1.27)
+				)
+				(hide yes)
+			)
+		)
+		(pin "1"
+		)
+		(instances
+			(project ""
+				(path "/34183abe-6288-4424-a0b3-d63b1476ac75/d136f52e-2f1b-437a-aa44-c69ff8c5465b"
+					(reference "#PWR030")
+					(unit 1)
+				)
+			)
+		)
+	)
+	(symbol
+		(lib_id "Connector_Generic:Conn_01x04")
+		(at 77.47 73.66 0)
+		(mirror y)
+		(unit 1)
+		(exclude_from_sim no)
+		(in_bom yes)
+		(on_board yes)
+		(dnp no)
+		(fields_autoplaced yes)
+		(property "Reference" "J5"
+			(at 77.47 64.77 0)
+			(effects
+				(font
+					(size 1.27 1.27)
+				)
+			)
+		)
+		(property "Value" "ADXL345"
+			(at 77.47 67.31 0)
+			(effects
+				(font
+					(size 1.27 1.27)
+				)
+			)
+		)
+		(property "Footprint" "Connector_PinHeader_2.54mm:PinHeader_1x04_P2.54mm_Vertical"
+			(at 77.47 73.66 0)
+			(effects
+				(font
+					(size 1.27 1.27)
+				)
+				(hide yes)
+			)
+		)
+		(property "Datasheet" "~"
+			(at 77.47 73.66 0)
+			(effects
+				(font
+					(size 1.27 1.27)
+				)
+				(hide yes)
+			)
+		)
+		(property "Description" "Generic connector, single row, 01x04, script generated (kicad-library-utils/schlib/autogen/connector/)"
+			(at 77.47 73.66 0)
+			(effects
+				(font
+					(size 1.27 1.27)
+				)
+				(hide yes)
+			)
+		)
+		(pin "2"
+		)
+		(pin "4"
+		)
+		(pin "3"
+		)
+		(pin "1"
+		)
+		(instances
+			(project ""
+				(path "/34183abe-6288-4424-a0b3-d63b1476ac75/d136f52e-2f1b-437a-aa44-c69ff8c5465b"
+					(reference "J5")
+					(unit 1)
+				)
+			)
+		)
+	)

Commit message: e
e
Parts:
- renumbered J5 to J113
Other:
- note added: "Was gonna add axdl345 chip but people say nozzle accelerometers are better than board ones. So I added a slot so you can choose."
Changed lines of the file:
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@@
 	(generator_version "9.0")
 	(paper "A5")
+	(text "Was gonna add axdl345 chip but \npeople say nozzle accelerometers \nare better than board ones.\nSo I added a slot so you can choose."
+		(exclude_from_sim no)
+		(at 51.816 74.676 0)
+		(effects
+			(font
+				(size 1.27 1.27)
+			)
+		)
+	)
 	(wire
 		(pts
@@
 		(dnp no)
 		(fields_autoplaced yes)
-		(property "Reference" "#PWR071"
+		(property "Reference" "#PWR0167"
 			(at 92.71 80.01 0)
 			(effects
@@
 			(project ""
 				(path "/34183abe-6288-4424-a0b3-d63b1476ac75/d136f52e-2f1b-437a-aa44-c69ff8c5465b"
-					(reference "#PWR071")
+					(reference "#PWR0167")
 					(unit 1)
 				)
@@
 		(dnp no)
 		(fields_autoplaced yes)
-		(property "Reference" "#PWR030"
+		(property "Reference" "#PWR0166"
 			(at 92.71 74.93 0)
 			(effects
@@
 			(project ""
 				(path "/34183abe-6288-4424-a0b3-d63b1476ac75/d136f52e-2f1b-437a-aa44-c69ff8c5465b"
-					(reference "#PWR030")
+					(reference "#PWR0166")
 					(unit 1)
 				)
@@
 		(dnp no)
 		(fields_autoplaced yes)
-		(property "Reference" "J5"
+		(property "Reference" "J113"
 			(at 77.47 64.77 0)
 			(effects
@@
 			(project ""
 				(path "/34183abe-6288-4424-a0b3-d63b1476ac75/d136f52e-2f1b-437a-aa44-c69ff8c5465b"
-					(reference "J5")
+					(reference "J113")
 					(unit 1)
 				)

Commit message: e
e
Parts:
- J111: renamed from J113; footprint Connector_PinHeader_2.54mm:PinHeader_1x04_P2.54mm_Vertical -> Connector_JST:JST_PH_B4B-PH-K_1x04_P2.00mm_Vertical
Changed lines of the file:
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@@
 		(dnp no)
 		(fields_autoplaced yes)
-		(property "Reference" "#PWR0167"
+		(property "Reference" "#PWR0170"
 			(at 92.71 80.01 0)
 			(effects
@@
 			(project ""
 				(path "/34183abe-6288-4424-a0b3-d63b1476ac75/d136f52e-2f1b-437a-aa44-c69ff8c5465b"
-					(reference "#PWR0167")
+					(reference "#PWR0170")
 					(unit 1)
 				)
@@
 		(dnp no)
 		(fields_autoplaced yes)
-		(property "Reference" "#PWR0166"
+		(property "Reference" "#PWR0169"
 			(at 92.71 74.93 0)
 			(effects
@@
 			(project ""
 				(path "/34183abe-6288-4424-a0b3-d63b1476ac75/d136f52e-2f1b-437a-aa44-c69ff8c5465b"
-					(reference "#PWR0166")
+					(reference "#PWR0169")
 					(unit 1)
 				)
@@
 		(dnp no)
 		(fields_autoplaced yes)
-		(property "Reference" "J113"
+		(property "Reference" "J111"
 			(at 77.47 64.77 0)
 			(effects
@@
 			)
 		)
-		(property "Footprint" "Connector_PinHeader_2.54mm:PinHeader_1x04_P2.54mm_Vertical"
+		(property "Footprint" "Connector_JST:JST_PH_B4B-PH-K_1x04_P2.00mm_Vertical"
 			(at 77.47 73.66 0)
 			(effects
@@
 			(project ""
 				(path "/34183abe-6288-4424-a0b3-d63b1476ac75/d136f52e-2f1b-437a-aa44-c69ff8c5465b"
-					(reference "J113")
+					(reference "J111")
 					(unit 1)
 				)
