File: KicadProjects/A1_SMD_THB/mainio.kicad_sch (KiCad schematic)
At the start: 6 parts, among them J3 PCF, J5 EXF, J6 THO, J7 HE, J8 BL_PROBE, J9 BL_SERVO

Commit message: e
e
Parts:
- removed J3: PCF, Connector_JST:JST_XH_B4B-XH-A_1x04_P2.50mm_Vertical, symbol Connector_Generic:Conn_01x04
- removed J5: EXF, Connector_JST:JST_XH_B5B-XH-A_1x05_P2.50mm_Vertical, symbol Connector_Generic:Conn_01x05
- added C28, C29, C30: 100nF, Capacitor_SMD:C_0402_1005Metric, symbol Device:C
- added D1: LED, symbol Device:LED
- added D2, D3, D4: schotty, symbol Device:D_Schottky_Dual_CommonAnode_AKK_Split
- added D5: BAV99, Package_TO_SOT_SMD:SOT-23, symbol Diode:BAV99
- added J11: F_SR1, symbol Connector_Generic:Conn_01x02
- added J12: F_SR2, symbol Connector_Generic:Conn_01x02
- added J13: PCF_FAN, symbol Connector_Generic:Conn_01x04
- added J14: SP_FAN, symbol Connector_Generic:Conn_01x04
- added J3: EXF, symbol Connector_Generic:Conn_01x05
- added Q1: NMOS, symbol Simulation_SPICE:NMOS
- added R13, R16: 20k, symbol Device:R
- added R14, R15, R22, R24, R26: 100, symbol Device:R
- added R17: 10R, symbol Device:R
- added R18: 20kR, symbol Device:R
- added R19: R, symbol Device:R
- added R20, R28: 2.37kR, symbol Device:R
- added R21, R23, R25: 10k, symbol Device:R
- added R27: 4.7kR, symbol Device:R
- added R29, R30, R31: 0 OHMS, symbol Device:R
Connections:
- net BL_PROBE: now also J8.2 (Pin_2)
- net BL_SERVO: now also J9.3 (Pin_3)
- net EXF_PWM: now also R26.1
- net EXF_TACH: now also R25.1
- net FIL_SNS1: now also R14.1
- net FIL_SNS2: now also R15.1
- net HE_SIG: now also R17.1, R18.1
- net PCF_PWM: now also R22.1
- net PCF_TACH: now also R21.1
- net SPARE_FAN_PWM: now also R24.1
- net SPARE_FAN_TACH: now also R23.1
- net THO: now also C30.1, R28.2
- net at J6.1 (Pin_1): now also R20.1, R27.2
- net GND: now reaches J6.2 (Pin_2)
- net GND: now also C30.2, D2.1 (A), D3.1 (A), D4.1 (A), D5.1 (K), J12.1 (Pin_1), J13.2 (Pin_2), J14.2 (Pin_2), J3.3 (Pin_3), Q1.3 (S), R18.2
- net GND3: now reaches J9.1 (Pin_1)
- net GND3: now also J8.1 (Pin_1), C28.2, C29.2
- net +3V3: now reaches J9.2 (Pin_2)
- net +3V3: now also R29.1, R30.1, R31.1
- net +24V: now reaches J7.1 (Pin_1)
- net +24V: now also D2.2 (K), D3.2 (K), D4.2 (K), J13.1 (Pin_1), J14.1 (Pin_1), J3.2 (Pin_2), R19.2
- net at J7.2 (Pin_2): now also D1.1 (K), Q1.1 (D)
- new net: J14.3 (Pin_3), R24.2
- new net: J14.4 (Pin_4), R23.2
- new net: C28.1, R13.1, R14.2
- new net: D1.2 (A), R19.1
- new net: J11.2 (Pin_2), R13.2, R29.2, R31.2
- new net: Q1.2 (G), R17.2
- new net: D5.3 (K), R20.2, R28.1
- new net: J13.3 (Pin_3), R22.2
- new net: J3.4 (Pin_4), R26.2
- new net: J13.4 (Pin_4), R21.2
- new net: J3.5 (Pin_5), R25.2
- new net: C29.1, R15.2, R16.1
- new net: J12.2 (Pin_2), R16.2, R30.2
- new net +3.3VADC: D5.2 (A), R27.1
Other:
- moved on the sheet: J6, J7, J8, J9

Commit message: e
e
Parts:
- D1, D3, R29, R30: now not fitted; now left out of the parts list
- J11, J12: footprint (none) -> Connector_PinHeader_2.54mm:PinHeader_1x02_P2.54mm_Vertical; now left out of the parts list
- J13: footprint (none) -> Connector_JST:JST_XH_B4B-XH-A_1x04_P2.50mm_Vertical; now left out of the parts list
- J14: footprint (none) -> Connector_PinHeader_2.54mm:PinHeader_1x04_P2.54mm_Vertical; now not fitted; now left out of the parts list
- J3: footprint (none) -> Connector_JST:JST_XH_B5B-XH-A_1x05_P2.50mm_Vertical; now left out of the parts list
- J6, J7: now left out of the parts list
- J8: footprint Connector_JST:JST_XH_B2B-XH-A_1x02_P2.50mm_Vertical -> Connector_PinHeader_2.54mm:PinHeader_1x02_P2.54mm_Vertical; now left out of the parts list
- J9: footprint Connector_JST:JST_XH_B3B-XH-A_1x03_P2.50mm_Vertical -> Connector_PinHeader_2.54mm:PinHeader_1x03_P2.54mm_Vertical; now left out of the parts list
- Q1: footprint (none) -> A1_SMD_THB:sot23f
- R13, R14, R15, R16, R17, R18, R20, R21, R22, R25, R26, R27, R28: footprint (none) -> Resistor_SMD:R_0402_1005Metric
- R19: value R -> 20kR; footprint (none) -> Resistor_SMD:R_0402_1005Metric; now not fitted; now left out of the parts list
- R23, R24: footprint (none) -> Resistor_SMD:R_0402_1005Metric; now not fitted; now left out of the parts list
Connections:
- net HE_SIG: now also Q1.2 (G), R17.2
Other:
- note added: "WILL DO YOURSELF"
Changed lines of the file:
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@@
 	(generator_version "9.0")
 	(paper "A5")
+	(text "WILL DO YOURSELF"
+		(exclude_from_sim no)
+		(at 83.82 24.13 0)
+		(effects
+			(font
+				(size 1.27 1.27)
+			)
+		)
+	)
+	(text "WILL DO YOURSELF"
+		(exclude_from_sim no)
+		(at 129.54 15.24 0)
+		(effects
+			(font
+				(size 1.27 1.27)
+			)
+		)
+	)
+	(text "WILL DO YOURSELF"
+		(exclude_from_sim no)
+		(at 77.724 103.886 0)
+		(effects
+			(font
+				(size 1.27 1.27)
+			)
+		)
+	)
+	(text "WILL DO YOURSELF"
+		(exclude_from_sim no)
+		(at 166.624 15.24 0)
+		(effects
+			(font
+				(size 1.27 1.27)
+			)
+		)
+	)
+	(text "WILL DO YOURSELF"
+		(exclude_from_sim no)
+		(at 93.726 73.914 0)
+		(effects
+			(font
+				(size 1.27 1.27)
+			)
+		)
+	)
+	(text "WILL DO YOURSELF"
+		(exclude_from_sim no)
+		(at 186.436 78.74 0)
+		(effects
+			(font
+				(size 1.27 1.27)
+			)
+		)
+	)
+	(text "WILL DO YOURSELF"
+		(exclude_from_sim no)
+		(at 76.962 113.538 0)
+		(effects
+			(font
+				(size 1.27 1.27)
+			)
+		)
+	)
+	(text "WILL DO YOURSELF"
+		(exclude_from_sim no)
+		(at 21.59 45.974 0)
+		(effects
+			(font
+				(size 1.27 1.27)
+			)
+		)
+	)
 	(junction
 		(at 111.76 76.2)
@@
 	(wire
 		(pts
+			(xy 104.14 85.09) (xy 104.14 88.9)
+		)
+		(stroke
+			(width 0)
+			(type default)
+		)
+	)
+	(wire
+		(pts
 			(xy 123.19 78.74) (xy 123.19 76.2)
 		)
@@
 	(wire
 		(pts
+			(xy 102.87 85.09) (xy 102.87 88.9)
+		)
+		(stroke
+			(width 0)
+			(type default)
+		)
+	)
+	(wire
+		(pts
 			(xy 87.63 41.91) (xy 92.71 41.91)
 		)
@@
 	(wire
 		(pts
-			(xy 102.87 88.9) (xy 104.14 88.9)
+			(xy 102.87 85.09) (xy 104.14 85.09)
 		)
 		(stroke
@@
 		)
 	)
+	(label "HE_SIG"
+		(at 102.87 85.09 0)
+		(effects
+			(font
+				(size 1.27 1.27)
+			)
+			(justify left bottom)
+		)
+	)
 	(hierarchical_label "SPARE_FAN_PWM"
 		(shape input)
@@
 		(mirror y)
 		(unit 1)
-		(exclude_from_sim no)
-		(in_bom yes)
-		(on_board yes)
-		(dnp no)
+		(exclude_from_sim yes)
+		(in_bom no)
+		(on_board no)
+		(dnp yes)
 		(fields_autoplaced yes)
 		(property "Reference" "J14"
@@
 			)
 		)
-		(property "Footprint" ""
+		(property "Footprint" "Connector_PinHeader_2.54mm:PinHeader_1x04_P2.54mm_Vertical"
 			(at 170.18 26.67 0)
 			(effects
@@
 		(unit 1)
 		(exclude_from_sim no)
-		(in_bom yes)
+		(in_bom no)
 		(on_board yes)
 		(dnp no)
@@
 		(at 123.19 91.44 0)
 		(unit 1)
-		(exclude_from_sim no)
-		(in_bom yes)
-		(on_board yes)
-		(dnp no)
+		(exclude_from_sim yes)
+		(in_bom no)
+		(on_board no)
+		(dnp yes)
 		(fields_autoplaced yes)
 		(property "Reference" "R19"
@@
 			)
 		)
-		(property "Value" "R"
+		(property "Value" "20kR"
 			(at 125.73 92.7099 0)
 			(effects
@@
 			)
 		)
-		(property "Footprint" ""
+		(property "Footprint" "Resistor_SMD:R_0402_1005Metric"
 			(at 121.412 91.44 90)
 			(effects
@@
 			)
 		)
-		(property "Footprint" ""
+		(property "Footprint" "Resistor_SMD:R_0402_1005Metric"
 			(at 31.75 100.838 90)
 			(effects
@@
 		(unit 1)
 		(exclude_from_sim no)
-		(in_bom yes)
+		(in_bom no)
 		(on_board yes)
 		(dnp no)
@@
 			)
 		)
-		(property "Footprint" ""
+		(property "Footprint" "Connector_PinHeader_2.54mm:PinHeader_1x02_P2.54mm_Vertical"
 			(at 77.47 96.52 0)
 			(effects
@@
 			)
 		)
-		(property "Footprint" ""
+		(property "Footprint" "A1_SMD_THB:sot23f"
 			(at 114.3 86.36 0)
 			(effects
@@
 			)
 		)
-		(property "Footprint" ""
+		(property "Footprint" "Resistor_SMD:R_0402_1005Metric"
 			(at 41.91 52.578 90)
 			(effects
@@
 			)
 		)
-		(property "Footprint" ""
+		(property "Footprint" "Resistor_SMD:R_0402_1005Metric"
 			(at 133.35 53.848 90)
 			(effects
@@
 		(at 123.19 82.55 270)
 		(unit 1)
-		(exclude_from_sim no)
-		(in_bom yes)
-		(on_board yes)
-		(dnp no)
+		(exclude_from_sim yes)
+		(in_bom no)
+		(on_board no)
+		(dnp yes)
 		(fields_autoplaced yes)
 		(property "Reference" "D1"
@@
 			)
 		)
-		(property "Footprint" ""
+		(property "Footprint" "Resistor_SMD:R_0402_1005Metric"
 			(at 96.52 53.848 90)
 			(effects
@@
 			)
 		)
-		(property "Footprint" ""
+		(property "Footprint" "Resistor_SMD:R_0402_1005Metric"
 			(at 99.06 97.028 90)
 			(effects
@@
 		(unit 1)
 		(exclude_from_sim no)
-		(in_bom yes)
+		(in_bom no)
 		(on_board yes)
 		(dnp no)
@@
 			)
 		)
-		(property "Footprint" ""
+		(property "Footprint" "Connector_JST:JST_XH_B4B-XH-A_1x04_P2.50mm_Vertical"
 			(at 132.08 26.67 0)
 			(effects
@@
 		(unit 1)
 		(exclude_from_sim no)
-		(in_bom yes)
+		(in_bom no)
 		(on_board yes)
 		(dnp no)
@@
 			)
 		)
-		(property "Footprint" "Connector_JST:JST_XH_B3B-XH-A_1x03_P2.50mm_Vertical"
+		(property "Footprint" "Connector_PinHeader_2.54mm:PinHeader_1x03_P2.54mm_Vertical"
 			(at 180.34 92.71 0)
 			(effects
@@
 		(unit 1)
 		(exclude_from_sim no)
-		(in_bom yes)
+		(in_bom no)
 		(on_board yes)
 		(dnp no)
@@
 			)
 		)
-		(property "Footprint" "Connector_JST:JST_XH_B2B-XH-A_1x02_P2.50mm_Vertical"
+		(property "Footprint" "Connector_PinHeader_2.54mm:PinHeader_1x02_P2.54mm_Vertical"
 			(at 180.34 82.55 0)
 			(effects
@@
 		(unit 1)
 		(exclude_from_sim no)
-		(in_bom yes)
+		(in_bom no)
 		(on_board yes)
 		(dnp no)
@@
 			)
 		)
-		(property "Footprint" ""
+		(property "Footprint" "Connector_JST:JST_XH_B5B-XH-A_1x05_P2.50mm_Vertical"
 			(at 95.25 26.67 0)
 			(effects
@@
 			)
 		)
-		(property "Footprint" ""
+		(property "Footprint" "Resistor_SMD:R_0402_1005Metric"
 			(at 33.782 40.64 90)
 			(effects
@@
 			)
 		)
-		(property "Footprint" ""
+		(property "Footprint" "Resistor_SMD:R_0402_1005Metric"
 			(at 133.35 43.688 90)
 			(effects
@@
 			)
 		)
-		(property "Footprint" ""
+		(property "Footprint" "Resistor_SMD:R_0402_1005Metric"
 			(at 31.75 122.428 90)
 			(effects
@@
 			)
 		)
-		(property "Footprint" ""
+		(property "Footprint" "Resistor_SMD:R_0402_1005Metric"
 			(at 55.88 52.578 90)
 			(effects
@@
 			)
 		)
-		(property "Footprint" ""
+		(property "Footprint" "Resistor_SMD:R_0402_1005Metric"
 			(at 41.91 100.838 90)
 			(effects
@@
 		(at 46.99 95.25 0)
 		(unit 1)
-		(exclude_from_sim no)
-		(in_bom yes)
-		(on_board yes)
-		(dnp no)
+		(exclude_from_sim yes)
+		(in_bom no)
+		(on_board no)
+		(dnp yes)
 		(fields_autoplaced yes)
 		(property "Reference" "R29"
@@
 		(at 186.69 26.67 90)
 		(unit 1)
-		(exclude_from_sim no)
-		(in_bom yes)
-		(on_board yes)
-		(dnp no)
+		(exclude_from_sim yes)
+		(in_bom no)
+		(on_board no)
+		(dnp yes)
 		(fields_autoplaced yes)
 		(property "Reference" "D3"
@@
 			)
 		)
-		(property "Footprint" ""
+		(property "Footprint" "Resistor_SMD:R_0402_1005Metric"
 			(at 96.52 43.688 90)
 			(effects
@@
 		(at 171.45 41.91 90)
 		(unit 1)
-		(exclude_from_sim no)
-		(in_bom yes)
-		(on_board yes)
-		(dnp no)
+		(exclude_from_sim yes)
+		(in_bom no)
+		(on_board no)
+		(dnp yes)
 		(fields_autoplaced yes)
 		(property "Reference" "R23"
@@
 			)
 		)
-		(property "Footprint" ""
+		(property "Footprint" "Resistor_SMD:R_0402_1005Metric"
 			(at 171.45 43.688 90)
 			(effects
@@
 		(unit 1)
 		(exclude_from_sim no)
-		(in_bom yes)
+		(in_bom no)
 		(on_board yes)
 		(dnp no)
@@
 		(at 171.45 52.07 90)
 		(unit 1)
-		(exclude_from_sim no)
-		(in_bom yes)
-		(on_board yes)
-		(dnp no)
+		(exclude_from_sim yes)
+		(in_bom no)
+		(on_board no)
+		(dnp yes)
 		(fields_autoplaced yes)
 		(property "Reference" "R24"
@@
 			)
 		)
-		(property "Footprint" ""
+		(property "Footprint" "Resistor_SMD:R_0402_1005Metric"
 			(at 171.45 53.848 90)
 			(effects
@@
 		(at 46.99 116.84 0)
 		(unit 1)
-		(exclude_from_sim no)
-		(in_bom yes)
-		(on_board yes)
-		(dnp no)
+		(exclude_from_sim yes)
+		(in_bom no)
+		(on_board no)
+		(dnp yes)
 		(fields_autoplaced yes)
 		(property "Reference" "R30"
@@
 		(unit 1)
 		(exclude_from_sim no)
-		(in_bom yes)
+		(in_bom no)
 		(on_board yes)
 		(dnp no)
@@
 			)
 		)
-		(property "Footprint" ""
+		(property "Footprint" "Connector_PinHeader_2.54mm:PinHeader_1x02_P2.54mm_Vertical"
 			(at 74.93 118.11 0)
 			(effects
@@
 			)
 		)
-		(property "Footprint" ""
+		(property "Footprint" "Resistor_SMD:R_0402_1005Metric"
 			(at 41.91 122.428 90)
 			(effects
@@
 			)
 		)
-		(property "Footprint" ""
+		(property "Footprint" "Resistor_SMD:R_0402_1005Metric"
 			(at 99.06 90.678 90)
 			(effects

Commit message: e
e
Parts:
- renumbered C28 to C119, C29 to C120, C30 to C121, D5 to D101, D4 to D102, D1 to D103, D2 to D104, D3 to D105, J6 to J104, J12 to J105, J11 to J106, J3 to J107, J7 to J108, J13 to J109, J14 to J110, J8 to J111, J9 to J112, Q1 to Q101, R14 to R108, R15 to R109, R27 to R110, R20 to R111, R13 to R112, R16 to R113, R30 to R114, R31 to R115, R29 to R116, R28 to R117, R25 to R118, R26 to R119, R17 to R120, R18 to R121, R19 to R122, R21 to R123, R22 to R124, R23 to R125, R24 to R126
Other:
- note added: "DO NOT PLACE"
- note added: "Filtering"
- note removed: "WILL DO YOURSELF"
- moved on the sheet: D103, J108, J111, J112, Q101, R115, R116, R120, R121, R122

Commit message: e
e
Parts:
- removed D102, D104, D105: schotty, symbol Device:D_Schottky_Dual_CommonAnode_AKK_Split
- removed J104: THO, Connector_JST:JST_XH_B2B-XH-A_1x02_P2.50mm_Vertical, symbol Connector_Generic:Conn_01x02
- removed J107: EXF, Connector_JST:JST_XH_B5B-XH-A_1x05_P2.50mm_Vertical, symbol Connector_Generic:Conn_01x05
- removed J108: HE, Connector_JST:JST_XH_B2B-XH-A_1x02_P2.50mm_Vertical, symbol Connector_Generic:Conn_01x02
- removed J110: SP_FAN, Connector_PinHeader_2.54mm:PinHeader_1x04_P2.54mm_Vertical, symbol Connector_Generic:Conn_01x04
- removed R118: 10k, Resistor_SMD:R_0402_1005Metric, symbol Device:R
- removed R119: 100, Resistor_SMD:R_0402_1005Metric, symbol Device:R
- added C122, C123: 10uF 50V, symbol Device:C
- added D103, D104: D, symbol Device:D
- added J104: SGDBM-08-020P-H40, A1KLibrary:Mezzanine Connector, symbol Connector_Generic:Conn_02x10_Counter_Clockwise
- added J110: EXF, Connector_JST:JST_XH_B5B-XH-A_1x05_P2.50mm_Vertical, symbol Connector_Generic:Conn_01x05
- added R121, R122: 10k, Resistor_SMD:R_0402_1005Metric, symbol Device:R
- J105: renamed from J111; footprint Connector_PinHeader_2.54mm:PinHeader_1x02_P2.54mm_Vertical -> Connector_JST:JST_PH_B2B-PH-K_1x02_P2.00mm_Vertical
- J106: renamed from J112; footprint Connector_PinHeader_2.54mm:PinHeader_1x03_P2.54mm_Vertical -> Connector_JST:JST_PH_B3B-PH-K_1x03_P2.00mm_Vertical
- J107: renamed from J105; footprint Connector_PinHeader_2.54mm:PinHeader_1x02_P2.54mm_Vertical -> Connector_JST:JST_PH_B2B-PH-K_1x02_P2.00mm_Vertical
- J108: renamed from J106; footprint Connector_PinHeader_2.54mm:PinHeader_1x02_P2.54mm_Vertical -> Connector_JST:JST_PH_B2B-PH-K_1x02_P2.00mm_Vertical
- Q101: footprint A1_SMD_THB:sot23f -> A1KLibrary:PPAK-8L 5x6 Mosfet
- R119: renamed from R115; now not fitted; now left out of the parts list
- R123: value 10k -> 4.7k
- R124: value 100 -> 10k
- R125: now fitted; now in the parts list
- R126: value 100 -> 4.7k; now fitted; now in the parts list
- renumbered C121 to C119, C119 to C121, D103 to D102, R117 to R108, R111 to R109, R120 to R111, R121 to R112, R122 to R113, R109 to R114, R108 to R115, R113 to R116, R112 to R117, R114 to R118, R116 to R120
Connections:
- net SPARE_FAN_PWM is gone; now on net EXF_PWM: R126.1
- net SPARE_FAN_TACH is gone; now on net +24V: R125.1
- net +24V: now also C122.1, C123.1, D103.1 (K), D104.1 (K), J104.1 (Pin_1), J104.18 (Pin_18), J104.19 (Pin_19), J104.2 (Pin_2), J104.20 (Pin_20), J104.3 (Pin_3), J110.2 (Pin_2), R122.1
- net EXF_PWM: now also J110.4 (Pin_4)
- net EXF_TACH: now also R124.1
- net GND: now also J108.1 (Pin_1), R123.2, R126.2, C122.2, C123.2, D103.2 (A), D104.2 (A), J104.14 (Pin_14), J104.15 (Pin_15), J104.6 (Pin_6), J104.7 (Pin_7), J110.3 (Pin_3)
- net HE_SIG: no longer Q101.2 (G), R111.2
- net PCF_PWM: now also J109.3 (Pin_3), R123.1; no longer R124.1
- net PCF_TACH: now also R121.1; no longer R123.1
- net at R125.2: now also R124.2, J110.5 (Pin_5)
- net at R109.1, R110.2: now also J104.16 (Pin_16), J104.17 (Pin_17), J104.4 (Pin_4), J104.5 (Pin_5)
- net at D102.1 (K), Q101.1 (D): now also J104.10 (Pin_10), J104.11 (Pin_11), J104.12 (Pin_12), J104.13 (Pin_13), J104.8 (Pin_8), J104.9 (Pin_9)
- net at J109.4 (Pin_4): now also R121.2, R122.2; no longer R123.2
- new net: Q101.2 (G), R111.2
- no-connect marks 0 -> 1
Other:
- moved on the sheet: C119, C120, C121, D101, D102, J105, J106, J107, J108, Q101, R108, R109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
