File: KicadProjects/A1_SMD_THB/mcu_stm32.kicad_sch (KiCad schematic)
At the start: 19 parts, among them J114 RUNJMP, J115 BOOT, U105 STM32G474RBTx, Y102 Crystal_GND24

Commit message: e
e
Parts:
- added P102: USB_C_Plug, symbol Connector:USB_C_Plug
- C134: renamed from C132; footprint (none) -> Capacitor_SMD:C_0402_1005Metric
- C137: renamed from C135; footprint (none) -> Capacitor_SMD:C_0402_1005Metric
- C138: renamed from C136; value 10uF -> 100nF
- C140: renamed from C138; footprint (none) -> Package_DFN_QFN:W-PDFN-8-1EP_6x5mm_P1.27mm_EP3x3mm
- FB101: footprint (none) -> Capacitor_SMD:C_0603_1608Metric
- J112: renamed from J114; footprint (none) -> Connector_PinHeader_2.54mm:PinHeader_1x02_P2.54mm_Vertical
- J113: renamed from J115; footprint (none) -> Connector_PinHeader_2.54mm:PinHeader_1x03_P2.54mm_Vertical
- R137: footprint (none) -> Resistor_SMD:R_0402_1005Metric
- Y102: footprint (none) -> Crystal:Crystal_SMD_3225-4Pin_3.2x2.5mm
- renumbered C6 to C132, C5 to C133, C4 to C135, C3 to C136, C2 to C139, C1 to C141, C7 to C142, C8 to C143, C9 to C144
Connections:
- net USB_D+: now also P102.A6 (D+)
- net USB_D-: now also P102.A7 (D-)
- new net: P102.A1 (GND), P102.A12 (GND), P102.B1 (GND), P102.B12 (GND)
- new net: P102.A4 (VBUS), P102.A9 (VBUS), P102.B4 (VBUS), P102.B9 (VBUS)
Other:
- note added: "C14709"
