File: KicadProjects/A1_SMD_THB/stepstick.kicad_sch (KiCad schematic)
At the start: 18 parts, among them M1 StepperMotor, U3 TMC2209-LA

Commit message: e
e
Other:
- moved on the sheet: C19, C21, C22, C23, C24, C25, C26, C27, EXM1, EXM2, R10, R11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

Commit message: e
e
Parts:
- added R32, R33, R34, R35: 100o, Resistor_SMD:R_0402_1005Metric, symbol Device:R
- EXM2: now left out of the parts list
- R10, R11, R12: footprint Capacitor_SMD:C_0201_0603Metric -> Resistor_SMD:R_0402_1005Metric
- U3: footprint A1_SMD_THB:QFN50P500X500X90-29N -> A1_SMD_THB:TMC2209-LA
Connections:
- net DIAG: now also R35.2
- net DIR: now also R33.1; no longer U3.19 (DIR)
- net EN: now also R34.1; no longer R12.2, U3.2 (~{EN})
- net STEP: now also R32.1; no longer U3.16 (STEP)
- net at EXM2.2 (Pin_2): now also U3.26 (OB1); no longer U3.21 (OA2)
- net at EXM2.3 (Pin_3): now also U3.24 (OA1); no longer U3.26 (OB1)
- net at EXM2.4 (Pin_4): now also U3.21 (OA2); no longer U3.24 (OA1)
- net at U3.11 (DIAG): now also R35.1
- new net: R12.2, R34.2, U3.2 (~{EN})
- new net: R33.2, U3.19 (DIR)
- new net: R32.2, U3.16 (STEP)
Other:
- note added: "WILL DO YOURSELF"
- moved on the sheet: EXM2

Commit message: e
e
Parts:
- U104: renamed from U3; footprint A1_SMD_THB:TMC2209-LA -> OpenA1K:TMC2209 Footprint
- renumbered C21 to C122, C27 to C123, C26 to C124, C25 to C125, C24 to C126, C23 to C127, C22 to C128, C19 to C129, EXM2 to EXM101, EXM1 to EXM102, M1 to M101, R11 to R127, R10 to R128, R12 to R129, R32 to R130, R33 to R131, R34 to R132, R8 to R133, R9 to R134, R35 to R135, R7 to R136
Connections:
- net at EXM101.2 (Pin_2): now also U104.21 (OA2); no longer U104.26 (OB1)
- net at EXM101.3 (Pin_3): now also U104.26 (OB1); no longer U104.24 (OA1)
- net at EXM101.4 (Pin_4): now also U104.24 (OA1); no longer U104.21 (OA2)
Other:
- note added: "Add lots of vias and ground pour for thermal transfer"
- note added: "Adress 0"
- note added: "Directly to ground plane"
- note added: "High Watt dissapation"
- note added: "Need to confirm pins"
- note added: "Uart split into tx and rx through 1k ohm resistor"

Commit message: e
e
Parts:
- U104: footprint OpenA1K:TMC2209 Footprint -> A1KLibrary:TMC2209-LA-FOOTPRINT
- renumbered C122 to C124, C123 to C125, C124 to C126, C125 to C127, C126 to C128, C127 to C129, C128 to C130, C129 to C131
Connections:
- net at EXM101.2 (Pin_2): now also U104.26 (OB1); no longer U104.21 (OA2)
- net at EXM101.3 (Pin_3): now also U104.24 (OA1); no longer U104.26 (OB1)
- net at EXM101.4 (Pin_4): now also U104.21 (OA2); no longer U104.24 (OA1)
