File: KicadProjects/A1_SMD_MB/motor.kicad_sch (KiCad schematic)
At the start: 20 parts, among them J15 Sensorless, J19 Endstop, U3 TMC2209-LA

Commit message: e
e
Parts:
- renumbered C21 to C42, C27 to C43, C26 to C44, C25 to C45, C24 to C46, C23 to C47, C22 to C48, EXM2 to EXM5, J15 to J18, J19 to J22, R11 to R23, R10 to R24, R12 to R25, R8 to R26, R9 to R27, R32 to R44, R33 to R45, R34 to R46, R35 to R47, U3 to U6
