File: KicadProjects/A1_SMD_MB/motors.kicad_sch (KiCad schematic)
At the start: 0 parts

Commit message: e
e
Other:
- note added: "A MOTOR"
- note added: "B MOTOR"
- note added: "C MOTOR"
- note added: "D MOTOR"
- note removed: "SMOTOR"
- note removed: "XMOTOR"
- note removed: "YMOTOR"
- note removed: "ZMOTOR"
Changed lines of the file:
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@@
 	(generator_version "9.0")
 	(paper "A4")
-	(text "SMOTOR\n"
+	(text "D MOTOR"
 		(exclude_from_sim no)
 		(at 156.21 42.418 0)
@@
 		)
 	)
-	(text "ZMOTOR\n"
+	(text "C MOTOR"
 		(exclude_from_sim no)
 		(at 127 42.418 0)
@@
 		)
 	)
-	(text "YMOTOR\n"
+	(text "B MOTOR"
 		(exclude_from_sim no)
 		(at 88.9 42.418 0)
@@
 		)
 	)
-	(text "XMOTOR"
+	(text "A MOTOR"
 		(exclude_from_sim no)
 		(at 50.8 42.418 0)
@@
 	(wire
 		(pts
-			(xy 132.715 52.07) (xy 138.43 52.07)
+			(xy 133.35 58.42) (xy 133.35 54.61)
 		)
 		(stroke
@@
 	(wire
 		(pts
-			(xy 132.715 54.61) (xy 135.255 54.61)
+			(xy 132.715 52.07) (xy 138.43 52.07)
+		)
+		(stroke
+			(width 0)
+			(type default)
+		)
+	)
+	(wire
+		(pts
+			(xy 133.35 54.61) (xy 132.715 54.61)
+		)
+		(stroke
+			(width 0)
+			(type default)
+		)
+	)
+	(wire
+		(pts
+			(xy 133.35 58.42) (xy 135.89 58.42)
 		)
 		(stroke
@@
 		)
 	)
-	(hierarchical_label "MZ_DIAG"
+	(hierarchical_label "MC_DIAG"
 		(shape input)
 		(at 119.38 57.15 180)
@@
 		)
 	)
-	(hierarchical_label "MZ_EN"
+	(hierarchical_label "MC_EN"
 		(shape input)
 		(at 119.38 49.53 180)
@@
 		)
 	)
-	(hierarchical_label "MY_EN"
+	(hierarchical_label "MB_EN"
 		(shape input)
 		(at 81.28 49.53 180)
@@
 		)
 	)
-	(hierarchical_label "MS_EN"
+	(hierarchical_label "MD_EN"
 		(shape input)
 		(at 157.48 49.53 180)
@@
 		)
 	)
-	(hierarchical_label "MS_DIAG"
+	(hierarchical_label "MD_DIAG"
 		(shape input)
 		(at 157.48 57.15 180)
@@
 		)
 	)
-	(hierarchical_label "MY_DIAG"
+	(hierarchical_label "MB_DIAG"
 		(shape input)
 		(at 81.28 57.15 180)
@@
 		)
 	)
-	(hierarchical_label "MS_STEP"
+	(hierarchical_label "MD_STEP"
 		(shape input)
 		(at 157.48 52.07 180)
@@
 		)
 	)
-	(hierarchical_label "MX_DIR"
+	(hierarchical_label "MA_DIR"
 		(shape input)
 		(at 43.18 54.61 180)
@@
 		)
 	)
-	(hierarchical_label "MY_DIR"
+	(hierarchical_label "MB_DIR"
 		(shape input)
 		(at 81.28 54.61 180)
@@
 		)
 	)
-	(hierarchical_label "MZ_DIR"
+	(hierarchical_label "MC_DIR"
 		(shape input)
 		(at 119.38 54.61 180)
@@
 		)
 	)
-	(hierarchical_label "MX_EN"
+	(hierarchical_label "MA_EN"
 		(shape input)
 		(at 43.18 49.53 180)
@@
 		)
 	)
-	(hierarchical_label "MY_STEP"
+	(hierarchical_label "MB_STEP"
 		(shape input)
 		(at 81.28 52.07 180)
@@
 		)
 	)
-	(hierarchical_label "MZ_STEP"
+	(hierarchical_label "MC_STEP"
 		(shape input)
 		(at 119.38 52.07 180)
@@
 		)
 	)
-	(hierarchical_label "MS_DIR"
+	(hierarchical_label "MD_DIR"
 		(shape input)
 		(at 157.48 54.61 180)
@@
 		)
 	)
-	(hierarchical_label "MX_STEP"
+	(hierarchical_label "MA_STEP"
 		(shape input)
 		(at 43.18 52.07 180)
@@
 		)
 	)
-	(hierarchical_label "MX_DIAG"
+	(hierarchical_label "MA_DIAG"
 		(shape input)
 		(at 43.18 57.15 180)
@@
 		)
 		(instances
-			(project "A1_MB_V2"
-				(path "/a288b6e0-7c74-4cd9-8c53-d587802da1e5/dd78447b-7ded-4c2d-bbee-1d2f5fbfdbd7"
+			(project "A1_SMD_MB"
+				(path "/a288b6e0-7c74-4cd9-8c53-d587802da1e5/55a65d08-43ee-456e-9750-5e9df50d0c33"
+					(reference "#PWR0138")
+					(unit 1)
+				)
+				(path "/a288b6e0-7c74-4cd9-8c53-d587802da1e5/a00a7ee4-471c-4552-bc8c-cbcb57c96fdf"
 					(reference "#PWR021")
 					(unit 1)
@@
 	(symbol
 		(lib_id "power:+3V3")
-		(at 135.255 54.61 0)
+		(at 135.89 58.42 0)
 		(unit 1)
 		(exclude_from_sim no)
@@
 		(fields_autoplaced yes)
 		(property "Reference" "#PWR023"
-			(at 135.255 58.42 0)
+			(at 135.89 62.23 0)
 			(effects
 				(font
@@
 		)
 		(property "Value" "+3V3"
-			(at 135.255 49.53 0)
+			(at 135.89 53.34 0)
 			(effects
 				(font
@@
 		)
 		(property "Footprint" ""
-			(at 135.255 54.61 0)
+			(at 135.89 58.42 0)
 			(effects
 				(font
@@
 		)
 		(property "Datasheet" ""
-			(at 135.255 54.61 0)
+			(at 135.89 58.42 0)
 			(effects
 				(font
@@
 		)
 		(property "Description" "Power symbol creates a global label with name \"+3V3\""
-			(at 135.255 54.61 0)
+			(at 135.89 58.42 0)
 			(effects
 				(font
@@
 		)
 		(instances
-			(project "A1_MB_V2"
-				(path "/a288b6e0-7c74-4cd9-8c53-d587802da1e5/dd78447b-7ded-4c2d-bbee-1d2f5fbfdbd7"
+			(project "A1_SMD_MB"
+				(path "/a288b6e0-7c74-4cd9-8c53-d587802da1e5/55a65d08-43ee-456e-9750-5e9df50d0c33"
+					(reference "#PWR0140")
+					(unit 1)
+				)
+				(path "/a288b6e0-7c74-4cd9-8c53-d587802da1e5/a00a7ee4-471c-4552-bc8c-cbcb57c96fdf"
 					(reference "#PWR023")
 					(unit 1)
@@
 		)
 		(instances
-			(project "A1_MB_V2"
-				(path "/a288b6e0-7c74-4cd9-8c53-d587802da1e5/dd78447b-7ded-4c2d-bbee-1d2f5fbfdbd7"
+			(project "A1_SMD_MB"
+				(path "/a288b6e0-7c74-4cd9-8c53-d587802da1e5/55a65d08-43ee-456e-9750-5e9df50d0c33"
+					(reference "#PWR0142")
+					(unit 1)
+				)
+				(path "/a288b6e0-7c74-4cd9-8c53-d587802da1e5/a00a7ee4-471c-4552-bc8c-cbcb57c96fdf"
 					(reference "#PWR025")
 					(unit 1)
@@
 		)
 		(instances
-			(project "A1_MB_V2"
-				(path "/a288b6e0-7c74-4cd9-8c53-d587802da1e5/dd78447b-7ded-4c2d-bbee-1d2f5fbfdbd7"
+			(project "A1_SMD_MB"
+				(path "/a288b6e0-7c74-4cd9-8c53-d587802da1e5/55a65d08-43ee-456e-9750-5e9df50d0c33"
+					(reference "#PWR0143")
+					(unit 1)
+				)
+				(path "/a288b6e0-7c74-4cd9-8c53-d587802da1e5/a00a7ee4-471c-4552-bc8c-cbcb57c96fdf"
 					(reference "#PWR027")
 					(unit 1)
@@
 		)
 		(instances
-			(project "A1_MB_V2"
-				(path "/a288b6e0-7c74-4cd9-8c53-d587802da1e5/dd78447b-7ded-4c2d-bbee-1d2f5fbfdbd7"
+			(project "A1_SMD_MB"
+				(path "/a288b6e0-7c74-4cd9-8c53-d587802da1e5/55a65d08-43ee-456e-9750-5e9df50d0c33"
+					(reference "#PWR0139")
+					(unit 1)
+				)
+				(path "/a288b6e0-7c74-4cd9-8c53-d587802da1e5/a00a7ee4-471c-4552-bc8c-cbcb57c96fdf"
 					(reference "#PWR022")
 					(unit 1)
@@
 		)
 		(instances
-			(project "A1_MB_V2"
-				(path "/a288b6e0-7c74-4cd9-8c53-d587802da1e5/dd78447b-7ded-4c2d-bbee-1d2f5fbfdbd7"
+			(project "A1_SMD_MB"
+				(path "/a288b6e0-7c74-4cd9-8c53-d587802da1e5/55a65d08-43ee-456e-9750-5e9df50d0c33"
+					(reference "#PWR0141")
+					(unit 1)
+				)
+				(path "/a288b6e0-7c74-4cd9-8c53-d587802da1e5/a00a7ee4-471c-4552-bc8c-cbcb57c96fdf"
 					(reference "#PWR024")
 					(unit 1)
@@
 		)
 		(instances
-			(project ""
-				(path "/a288b6e0-7c74-4cd9-8c53-d587802da1e5/dd78447b-7ded-4c2d-bbee-1d2f5fbfdbd7"
+			(project "A1_SMD_MB"
+				(path "/a288b6e0-7c74-4cd9-8c53-d587802da1e5/55a65d08-43ee-456e-9750-5e9df50d0c33"
+					(reference "#PWR0136")
+					(unit 1)
+				)
+				(path "/a288b6e0-7c74-4cd9-8c53-d587802da1e5/a00a7ee4-471c-4552-bc8c-cbcb57c96fdf"
 					(reference "#PWR019")
 					(unit 1)
@@
 		)
 		(instances
-			(project "A1_MB_V2"
-				(path "/a288b6e0-7c74-4cd9-8c53-d587802da1e5/dd78447b-7ded-4c2d-bbee-1d2f5fbfdbd7"
+			(project "A1_SMD_MB"
+				(path "/a288b6e0-7c74-4cd9-8c53-d587802da1e5/55a65d08-43ee-456e-9750-5e9df50d0c33"
+					(reference "#PWR0137")
+					(unit 1)
+				)
+				(path "/a288b6e0-7c74-4cd9-8c53-d587802da1e5/a00a7ee4-471c-4552-bc8c-cbcb57c96fdf"
 					(reference "#PWR020")
 					(unit 1)
@@
 		)
 		(instances
-			(project "A1_MB_V2"
-				(path "/a288b6e0-7c74-4cd9-8c53-d587802da1e5/dd78447b-7ded-4c2d-bbee-1d2f5fbfdbd7"
+			(project "A1_SMD_MB"
+				(path "/a288b6e0-7c74-4cd9-8c53-d587802da1e5/a00a7ee4-471c-4552-bc8c-cbcb57c96fdf"
 					(page "5")
+				)
+				(path "/a288b6e0-7c74-4cd9-8c53-d587802da1e5/55a65d08-43ee-456e-9750-5e9df50d0c33"
+					(page "15")
 				)
 			)
@@
 		)
 		(instances
-			(project "A1_MB_V2"
-				(path "/a288b6e0-7c74-4cd9-8c53-d587802da1e5/dd78447b-7ded-4c2d-bbee-1d2f5fbfdbd7"
-					(page "7")
+			(project "A1_SMD_MB"
+				(path "/a288b6e0-7c74-4cd9-8c53-d587802da1e5/a00a7ee4-471c-4552-bc8c-cbcb57c96fdf"
+					(page "4")
+				)
+				(path "/a288b6e0-7c74-4cd9-8c53-d587802da1e5/55a65d08-43ee-456e-9750-5e9df50d0c33"
+					(page "17")
 				)
 			)
@@
 		)
 		(instances
-			(project "A1_MB_V2"
-				(path "/a288b6e0-7c74-4cd9-8c53-d587802da1e5/dd78447b-7ded-4c2d-bbee-1d2f5fbfdbd7"
-					(page "4")
+			(project "A1_SMD_MB"
+				(path "/a288b6e0-7c74-4cd9-8c53-d587802da1e5/a00a7ee4-471c-4552-bc8c-cbcb57c96fdf"
+					(page "6")
+				)
+				(path "/a288b6e0-7c74-4cd9-8c53-d587802da1e5/55a65d08-43ee-456e-9750-5e9df50d0c33"
+					(page "16")
 				)
 			)
@@
 		)
 		(instances
-			(project "A1_MB_V2"
-				(path "/a288b6e0-7c74-4cd9-8c53-d587802da1e5/dd78447b-7ded-4c2d-bbee-1d2f5fbfdbd7"
-					(page "6")
-				)
-			)
+			(project "A1_SMD_MB"
+				(path "/a288b6e0-7c74-4cd9-8c53-d587802da1e5/a00a7ee4-471c-4552-bc8c-cbcb57c96fdf"
+					(page "7")
+				)
+				(path "/a288b6e0-7c74-4cd9-8c53-d587802da1e5/55a65d08-43ee-456e-9750-5e9df50d0c33"
+					(page "18")
+				)
+			)
