File: A1-Main-Board/A1-Main-Board.kicad_sch (KiCad schematic)
At the start: 3 parts

Commit message: e
e
Parts:
- removed R22, R24: 1k, symbol Device:R
Other:
- added sheet computeboard (computeboard.kicad_sch)
- added sheet fan (fan.kicad_sch)
- added sheet heated-bed (heated-bed.kicad_sch)
- added sheet power (power.kicad_sch)
- added sheet spare (spare.kicad_sch)
- sheet communications-toolhead ports: added UART_RX, UART_TX, USB_D+, USB_D-; removed none
- sheet mcu ports: added BED_THERM1, BED_THERM2, FAN0_PWM, FAN0_TACH, FAN1_PWM, FAN1_TACH, HEATED_BED_PWM, UART_RX, UART_TX, USB_D+, USB_D-, gpioPB11, gpioPB12, gpioPB13, gpioPB15, gpioPB3, gpioPB4, gpioPB5, gpioPB6, gpioPB7, gpioPC13, gpioPC14, gpioPC15; removed none
- moved on the sheet: R20
