File: A1-Main-Board/comms-toolhead.kicad_sch (KiCad schematic)
At the start: 3 parts, among them J4 UART_PINS, J5 USB_PINS, P1 USB_C_Plug

Commit message: e
e
Other:
- note added: "BACKUP TO CM4"
- note added: "BACKUP TO RPZ2"
- note added: "TO CM4"
- note added: "TO RPZ2"
- note added: "Toolhead Incoming"
Changed lines of the file:
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@@
 	(generator_version "9.0")
 	(paper "A4")
+	(text "Toolhead Incoming"
+		(exclude_from_sim no)
+		(at 119.634 39.878 0)
+		(effects
+			(font
+				(size 2.54 2.54)
+				(thickness 0.3175)
+			)
+		)
+	)
+	(text "BACKUP TO RPZ2"
+		(exclude_from_sim no)
+		(at 197.358 85.598 0)
+		(effects
+			(font
+				(size 1.27 1.27)
+				(thickness 0.254)
+				(bold yes)
+			)
+		)
+	)
+	(text "BACKUP TO CM4"
+		(exclude_from_sim no)
+		(at 196.85 94.234 0)
+		(effects
+			(font
+				(size 1.27 1.27)
+				(thickness 0.254)
+				(bold yes)
+			)
+		)
+	)
+	(text "TO CM4"
+		(exclude_from_sim no)
+		(at 192.278 69.088 0)
+		(effects
+			(font
+				(size 1.27 1.27)
+				(thickness 0.254)
+				(bold yes)
+			)
+		)
+	)
 	(text "RECIEVE = UART"
 		(exclude_from_sim no)
@@
 		(effects
 			(font
+				(size 1.27 1.27)
+				(thickness 0.254)
+				(bold yes)
+			)
+		)
+	)
+	(text "TO RPZ2"
+		(exclude_from_sim no)
+		(at 193.294 56.134 0)
+		(effects
+			(font
