File: A1-Main-Board/drivers.kicad_sch (KiCad schematic)
At the start: 0 parts

Commit message: e
e
Other:
- sheet stepstick ports: added MS1, MS2; removed none
- sheet stepstick1 ports: added MS1, MS2; removed none
- sheet stepstick2 ports: added MS1, MS2; removed none
