File: A1-Main-Board/mcu.kicad_sch (KiCad schematic)
At the start: 19 parts, among them J115 BOOT, SW101 SW_SPST, U105 STM32G431RBT3, Y103 Crystal_GND24

Commit message: e
e
Connections:
- net MZ_DIR: now reaches U105.10 (PC2)
- net MZ_STEP: now reaches U105.11 (PC3)
- net MY_DIAG: now reaches U105.13 (PA1)
- net MY_EN: now reaches U105.14 (PA2)
- net MY_DIR: now reaches U105.17 (PA3)
- net MY_STEP: now reaches U105.18 (PA4)
- net MX_DIAG: now reaches U105.19 (PA5)
- net MX_EN: now reaches U105.20 (PA6)
- net MX_DIR: now reaches U105.21 (PA7)
- net MT_UART_TX: now reaches U105.22 (PC4)
- net MT_UART_RX: now reaches U105.23 (PC5)
- net MX_STEP: now reaches U105.24 (PB0)
- net at U105.61 (PB8): now also R138.2
- net MZ_DIAG: now reaches U105.8 (PC0)
- net MZ_EN: now reaches U105.9 (PC1)
Other:
- moved on the sheet: C145, C146, C147, C148, C149, C150, C151, C152, C153, C154, C155, C156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

Commit message: e
e
Parts:
- added J6: MB_UART, symbol Connector_Generic:Conn_01x02
- added J7: MB_USB, symbol Connector_Generic:Conn_01x02
Connections:
- net +3V3A: now also U105.28 (VREF+)
- net GND: now also U105.15 (VSS), U105.27 (VSSA), U105.31 (VSS), U105.47 (VSS), U105.63 (VSS)
- net gpioPC13: now reaches U105.2 (PC13)
- net gpioPC14: now reaches U105.3 (PC14)
- net gpioPB11: now reaches U105.33 (PB11)
- net gpioPB12: now reaches U105.34 (PB12)
- net gpioPB13: now reaches U105.35 (PB13)
- net BED_THERM2: now reaches U105.36 (PB14)
- net gpioPB15: now reaches U105.37 (PB15)
- net HEATED_BED_PWM: now reaches U105.38 (PC6)
- net FAN0_PWM: now reaches U105.39 (PC7)
- net gpioPC15: now reaches U105.4 (PC15)
- net FAN0_TACH: now reaches U105.40 (PC8)
- net FAN1_PWM: now reaches U105.41 (PC9)
- net I2C_SCL: now reaches U105.42 (PA8)
- net BED_THERM1: now reaches U105.43 (PA9)
- net FAN1_TACH: now reaches U105.44 (PA10)
- net USB_D-: now reaches U105.45 (PA11)
- net USB_D-: now also J7.1 (Pin_1)
- net USB_D+: now reaches U105.46 (PA12)
- net USB_D+: now also J7.2 (Pin_2)
- net UART_TX: now reaches U105.50 (PA14)
- net UART_TX: now also J6.1 (Pin_1)
- net UART_RX: now reaches U105.51 (PA15)
- net UART_RX: now also J6.2 (Pin_2)
- net I2C_SDA: now reaches U105.53 (PC11)
- net gpioPB3: now reaches U105.56 (PB3)
- net gpioPB4: now reaches U105.57 (PB4)
- net gpioPB5: now reaches U105.58 (PB5)
- net gpioPB6: now reaches U105.59 (PB6)
- net gpioPB7: now reaches U105.60 (PB7)
- no-connect marks 0 -> 9
Other:
- note added: "BACKUP TO CM4"
- note added: "BACKUP TO RPZ2"
- note added: "Do i add jumpers between the cm4 thing, to disable the on board slots. Will this stop reflectivity of singals. idk i only know stuff similar to this with ddr dimm."
- note added: "Jumper or Switch"
- note added: "TO CM4"
- note added: "TO RPZ2"
